File: projects/LabBenchPsu/Arduino.sch (KiCad schematic (older format))
At the start: 0 parts

Commit message: LabBenchPsu updated
Parts:
- added C? (x2): 100nF, symbol C
- added IC?: ATMEGA168A-P, DIL28, symbol ATMEGA168A-P
- added P?: CONN_3X2, symbol CONN_3X2
- added P?: CONN_6, symbol CONN_6
Connections:
- net 3V3_reg: now also C?.1, C?.1, IC?.20 (AVCC), IC?.7 (VCC)
- net ENCONV: now also IC?.26 ((PCINT11/ADC3)PC3)
- net SCL: now also IC?.28 ((PCINT14/SCL/ADC5)PC5)
- net SDA: now also IC?.27 ((PCINT12/SDA/ADC4)PC4)
- new net ADC-VOUT: IC?.23 ((PCINT8/ADC0)PC0)
- new net GND: C?.2, C?.2, IC?.22 (GND), IC?.8 (GND)
- new net V_REF: IC?.21 (AREF)
Changed lines of the file:
@@
 Comment4 ""
 $EndDescr
-Text HLabel 1775 1600 0    60   Input ~ 0
+Text HLabel 1950 2150 0    60   Input ~ 0
 3V3_reg
-Text HLabel 9000 2575 2    60   Output ~ 0
+Text HLabel 4250 3700 2    60   Output ~ 0
 SDA
-Text HLabel 9000 2800 2    60   Output ~ 0
+Text HLabel 4250 3800 2    60   Output ~ 0
 SCL
-Text HLabel 9050 3625 2    60   Output ~ 0
+Text HLabel 4250 3600 2    60   Output ~ 0
 ENCONV
+Text HLabel 2050 3050 0    60   Input ~ 0
+V_REF
+$Comp
+L ATMEGA168A-P IC?
+U 1 1 54A0D87B
+P 3050 3550
+F 0 "IC?" H 2300 4800 40  0000 L BNN
+F 1 "ATMEGA168A-P" H 3450 2150 40  0000 L BNN
+F 2 "DIL28" H 3050 3550 30  0000 C CIN
+F 3 "" H 3050 3550 60  0000 C CNN
+	1    3050 3550
+	1    0    0    -1
+$EndComp
+$Comp
+L C C?
+U 1 1 54A0D89B
+P 1850 2650
+F 0 "C?" H 1850 2750 40  0000 L CNN
+F 1 "100nF" H 1856 2565 40  0000 L CNN
+F 2 "" H 1888 2500 30  0000 C CNN
+F 3 "" H 1850 2650 60  0000 C CNN
+	1    1850 2650
+	1    0    0    -1
+$EndComp
+$Comp
+L C C?
+U 1 1 54A0D8B2
+P 1550 2650
+F 0 "C?" H 1550 2750 40  0000 L CNN
+F 1 "100nF" H 1556 2565 40  0000 L CNN
+F 2 "" H 1588 2500 30  0000 C CNN
+F 3 "" H 1550 2650 60  0000 C CNN
+	1    1550 2650
+	1    0    0    -1
+$EndComp
+$Comp
+L GND #PWR?
+U 1 1 54A0DA7C
+P 1550 2950
+F 0 "#PWR?" H 1550 2950 30  0001 C CNN
+F 1 "GND" H 1550 2880 30  0001 C CNN
+F 2 "" H 1550 2950 60  0000 C CNN
+F 3 "" H 1550 2950 60  0000 C CNN
+	1    1550 2950
+	1    0    0    -1
+$EndComp
+$Comp
+L GND #PWR?
+U 1 1 54A0DA8E
+P 2150 4900
+F 0 "#PWR?" H 2150 4900 30  0001 C CNN
+F 1 "GND" H 2150 4830 30  0001 C CNN
+F 2 "" H 2150 4900 60  0000 C CNN
+F 3 "" H 2150 4900 60  0000 C CNN
+	1    2150 4900
+	1    0    0    -1
+$EndComp
+Wire Wire Line
+	2050 3050 2150 3050
+Wire Wire Line
+	2150 2150 2150 2750
+Wire Wire Line
+	1550 2450 2150 2450
+Connection ~ 1850 2450
+Wire Wire Line
+	1850 2850 1550 2850
+Wire Wire Line
+	1550 2850 1550 2950
+Wire Wire Line
+	1950 2150 2150 2150
+Connection ~ 2150 2450
+Wire Wire Line
+	2150 4650 2150 4900
+Connection ~ 2150 4750
+Wire Wire Line
+	4050 3600 4250 3600
+Wire Wire Line
+	4050 3700 4250 3700
+Wire Wire Line
+	4050 3800 4250 3800
+$Comp
+L CONN_3X2 P?
+U 1 1 54A0ECAA
+P 6225 4625
+F 0 "P?" H 6225 4875 50  0000 C CNN
+F 1 "CONN_3X2" V 6225 4675 40  0000 C CNN
+F 2 "" H 6225 4625 60  0000 C CNN
+F 3 "" H 6225 4625 60  0000 C CNN
+	1    6225 4625
+	1    0    0    -1
+$EndComp
+$Comp
+L CONN_6 P?
+U 1 1 54A0ECBE
+P 6275 3650
+F 0 "P?" V 6225 3650 60  0000 C CNN
+F 1 "CONN_6" V 6325 3650 60  0000 C CNN
+F 2 "" H 6275 3650 60  0000 C CNN
+F 3 "" H 6275 3650 60  0000 C CNN
+	1    6275 3650
+	1    0    0    -1
+$EndComp
+Text HLabel 4250 3300 2    60   Input ~ 0
+ADC-VOUT
+Wire Wire Line
+	4250 3300 4050 3300
 $EndSCHEMATC

Commit message: LabBenchPsu updated
Parts:
- added C? (x2): 100nF, symbol C
- added ENC? (x2): RotaryEncoder, symbol RotaryEncoder
- added P?: CONN_4, symbol CONN_4
- added R?: 10K, symbol R
- added S? (x6): TAC_SWITCH, TACTILE, symbol TAC_SWITCH
- added U?: MCP23008, symbol MCP23008
- added X?: Resonator, symbol Resonator
Connections:
- net 3V3_reg: now also P?.2, P?.4, C?.1, P?.1 (P1), R?.1, U?.18 (VDD)
- net GND: now also P?.5, P?.6, P?.6, C?.2, ENC?.2 (COM), ENC?.2 (COM), P?.4 (P4), S?.3, S?.3, S?.3, S?.3, S?.3, S?.3, S?.4, S?.4, S?.4, S?.4, S?.4, S?.4, U?.3 (A2), U?.4 (A1), U?.5 (A0), U?.9 (VSS), X?.2 (GND)
- net SCL: now also P?.3 (P3), U?.1 (SCL)
- net SDA: now also P?.2 (P2), U?.2 (SDA)
- net RESET: now reaches IC?.1 ((PCINT14/~RESET~)PC6)
- net RESET: now also P?.5, C?.1, R?.2, S?.1, S?.2, U?.6 (!RESET)
- net X2: now reaches IC?.10 ((PCINT7/XTAL2/TOSC2)PB7)
- net X2: now also X?.3 (X2)
- net ENC2B: now reaches IC?.11 ((PCINT21/OC0B/T1)PD5)
- net ENC2B: now also ENC?.3 (B)
- net CLIM: now reaches IC?.13 ((PCINT23/AIN1)PD7)
- net INT: now reaches IC?.14 ((PCINT0/CLKO/ICP1)PB0)
- net INT: now also U?.8 (INT)
- net ISET: now reaches IC?.15 ((PCINT1/OC1A)PB1)
- net MOSI: now reaches IC?.17 ((PCINT3/OC2A/MOSI)PB3)
- net MOSI: now also P?.4
- net MISO: now reaches IC?.18 ((PCINT4/MISO)PB4)
- net MISO: now also P?.1
- net SCK: now reaches IC?.19 ((PCINT5/SCK)PB5)
- net SCK: now also P?.3
- net RXD: now reaches IC?.2 ((PCINT16/RXD)PD0)
- net RXD: now also P?.3
- net ADC-IOUT: now reaches IC?.25 ((PCINT10/ADC2)PC2)
- net TXD: now reaches IC?.3 ((PCINT17/TXD)PD1)
- net TXD: now also P?.2
- net ENC1A: now reaches IC?.4 ((PCINT18/INT0)PD2)
- net ENC1A: now also ENC?.1 (A)
- net ENC1B: now reaches IC?.5 ((PCINT19/OC2B/INT1)PD3)
- net ENC1B: now also ENC?.3 (B)
- net ENC2A: now reaches IC?.6 ((PCINT20/XCK/T0)PD4)
- net ENC2A: now also ENC?.1 (A)
- net X1: now reaches IC?.9 ((PCINT6/XTAL1/TOSC1)PB6)
- net X1: now also X?.1 (X1)
- net at P?.1: now also C?.2
- new net: S?.1, S?.2, U?.10 (GP0)
- new net: S?.1, S?.2, U?.11 (GP1)
- new net: S?.1, S?.2, U?.12 (GP2)
- new net: S?.1, S?.2, U?.13 (GP3)
- new net: S?.1, S?.2, U?.14 (GP4)
- no-connect marks 0 -> 3
Other:
- moved on the sheet: P?

Commit message: LabBenchPsu updated
Parts:
- removed C? (x4): 100nF, symbol C
- removed IC?: ATMEGA168A-P, DIL28, symbol ATMEGA168A-P
- removed P?: CONN_3X2, symbol CONN_3X2
- removed P?: CONN_6, symbol CONN_6
- removed R?: 10K, symbol R
- removed S? (x2): TAC_SWITCH, TACTILE, symbol TAC_SWITCH
- removed U?: MCP23008, symbol MCP23008
- added C? (x3): 100nF, symbol C
- added CON?: USB-MINI-B, symbol USB-MINI-B
- added D?: DIODE, symbol DIODE
- added F?: FUSE, symbol FUSE
- added P?: CONN_3X2, symbol CONN_3X2
- added R? (x2): 33R, symbol R
- added R? (x2): 10K, symbol R
- added R? (x3): 4K7, symbol R
- added R? (x2): 2K2, symbol R
- added S?: Reset, TACTILE, symbol TAC_SWITCH
- added U?: ATMEGA32U4, MODULE, symbol ATMEGA32U4
- added U?: 24AA04, symbol 24AA04
- added X?: OLED-2004, OLED2004, symbol OLED-2004
- S?: value TAC_SWITCH -> PB1
- S?: value TAC_SWITCH -> PB2
- S?: value TAC_SWITCH -> PB3
- S?: value TAC_SWITCH -> PB4
Connections:
- net 3V3_reg: now also C?.1, C?.1, R?.1, R?.1, R?.2, U?.14 (VCC), U?.2 (UVcc:), U?.24 (AVCC), U?.34 (VCC), U?.4 (Vcc), U?.44 (AVCC), X?.18 (BS1), X?.2 (VDD)
- net GND: now also C?.2, C?.2, C?.2, CON?.5 (GND), CON?.6 (SHELL1), CON?.7 (SHELL2), CON?.8 (SHELL3), CON?.9 (SHELL4), P?.6, R?.2, S?.3, S?.4, U?.15 (GND), U?.2 (Vss), U?.23 (GND), U?.35 (GND), U?.43 (GND), U?.5 (UGnd), U?.5 (WP), X?.1 (VSS), X?.10 (NC), X?.11 (NC), X?.12 (NC), X?.13 (NC), X?.14 (NC), X?.15 (NC), X?.17 (BS0), X?.19 (BS2), X?.20 (VSS), X?.4 (SA0), X?.5 (NC), X?.6 (NC)
- net MISO: now also R?.2, U?.11 ((PDO/PCINT3/MISO)PB3)
- net MOSI: now also R?.1, U?.10 ((PDI/PCINT2/MOSI)PB2)
- net SCK: now also R?.2, U?.9 ((PCINT1/SCLK)PB1)
- net SCL: now also R?.2, U?.1 (SCL), U?.18 ((OC0B/SCL/INT0)PD0), X?.7 (SCL)
- net SDA: now also R?.1, U?.19 ((SDA/INT1)PD1), U?.3 (SDA), X?.8 (SDA_in), X?.9 (SDA_out)
- net V_REF: now also U?.42 (AREF)
- net X1: now also U?.17 (XTAL1)
- net X2: now also U?.16 (XTAL2)
- net PB4: now reaches S?.1, S?.2
- net PB3: now reaches S?.1, S?.2
- net PB2: now reaches S?.1, S?.2
- net PB1: now reaches S?.1, S?.2
- new net: R?.2, U?.3 (D-)
- new net: R?.1, U?.33 (PE2(^HWB))
- new net: R?.2, U?.4 (D+)
- new net: C?.1, U?.6 (UCap)
- new net: CON?.1 (VBUS), F?.1
- new net: CON?.2 (D-), R?.1
- new net: CON?.3 (D+), R?.1
- new net: P?.1, R?.1
- new net: P?.3, R?.1
- new net: P?.4, R?.2
- new net: D?.2 (K), P?.5
- new net Reset: D?.1 (A), R?.2, S?.1, S?.2, U?.13 (^RESET), X?.16 (!Reset)
- new net VBUS: F?.2, U?.7 (VBus)
- no-connect marks 3 -> 9
Other:
- note added: "# 16bit-PWM"
- note added: "4K EEPROM"
- note added: "I2C"
- note added: "ICSP"
- note added: "Place near ATMEGA"
- note added: "Save settings\nand calibration"
- note added: "i2c configuration:\nbs0-2 = 010 for i2c\nslave address:\n011110 SA0=0 R/W"
- moved on the sheet: ENC?, P?, S?, X?

Commit message: update LabBenchPsu
Parts:
- added D?: CLimit, symbol LED
- added D?: Load on, symbol LED
- added R? (x2): 100R, symbol R
- F?: value FUSE -> FUSE 500mA
- X?: value Resonator -> Resonator 16MHz
Connections:
- net GND: now also D?.2 (K), D?.2 (K)
- new net: D?.1 (A), R?.1 (x2)
Other:
- note added: "USB boot enable"
- note added: "i2c configuration:\nbs0-2 = 010 for i2c\nslave address:\n011110 SA0=0 R/W\nRead: 0x79\nWrite: 0x78"
- note added: "i2c configuration:\nslave address:\n1010 xx B0 R/W\nBlockselect: xxB0\n0xA..."
- note removed: "Save settings\nand calibration"
- note removed: "i2c configuration:\nbs0-2 = 010 for i2c\nslave address:\n011110 SA0=0 R/W"
- moved on the sheet: C?, CON?, D?, ENC?, F?, P?, R?, S?, U?, X?
