File: projects/LabBenchPsu/LabBenchPsu.sch (KiCad schematic (older format))
At the start: 32 parts

Commit message: LabBenchPsu update
Other:
- moved on the sheet: D?, F?, P?, R?, S?

Commit message: LabBenchPsu updated
Other:
- moved on the sheet: D?, F?, P?, R?, S?

Commit message: LabBenchPsu updated
Changed lines of the file:
@@
 F6 "OUT+" I R 9225 3600 60
 F7 "ISET" I L 7925 4275 60
-F8 "CLIM" I R 9225 3950 60
+F8 "CLIM" I R 9225 3800 60
 F9 "ADC-VOUT" O R 9225 4050 60
 F10 "V_REF" O R 9225 4250 60
+F11 "ADC-IOUT" O R 9225 3950 60
 $EndSheet
 $Sheet
@@
 F6 "V_REF" I R 7175 5350 60
 F7 "ADC-VOUT" I R 7175 5475 60
+F8 "ADC-IOUT" I R 7175 5600 60
+F9 "CLIM" I R 7175 5725 60
+F10 "ISET" O R 7175 5225 60
 $EndSheet
 Wire Wire Line
@@
 Wire Wire Line
 	9550 5475 7175 5475
+Wire Wire Line
+	9225 3950 9650 3950
+Wire Wire Line
+	9650 3950 9650 5600
+Wire Wire Line
+	9650 5600 7175 5600
+Wire Wire Line
+	9225 3800 9750 3800
+Wire Wire Line
+	9750 3800 9750 5725
+Wire Wire Line
+	9750 5725 7175 5725
+Wire Wire Line
+	7175 5225 7550 5225
+Wire Wire Line
+	7550 5225 7550 4275
+Wire Wire Line
+	7550 4275 7925 4275
 $EndSCHEMATC

Commit message: LabBenchPsu updated
Changed lines of the file:
@@
 F1 "Charging.sch" 50
 F2 "5V_direct" I R 3425 3550 60
+F3 "SDA" I R 3425 3825 60
+F4 "SCL" I R 3425 3925 60
+F5 "3V3_reg" I R 3425 3725 60
+F6 "Reset" I R 3425 4025 60
 $EndSheet
 $Sheet
-S 7925 3425 1300 975
+S 7925 3650 1300 975
 U 54A01D2E
 F0 "PSU" 50
@@
 F3 "SCL" I L 7925 4175 60
 F4 "3V3_reg" I L 7925 3875 60
-F5 "V+" I L 7925 3550 60
-F6 "OUT+" I R 9225 3600 60
+F5 "V+" I L 7925 3775 60
+F6 "OUT+" I R 9225 4450 60
 F7 "ISET" I L 7925 4275 60
 F8 "CLIM" I R 9225 3800 60
@@
 F3 "SDA" O R 7175 5025 60
 F4 "SCL" O R 7175 5125 60
-F5 "ENCONV" O L 5450 4825 60
+F5 "ENCONV" O R 7175 5850 60
 F6 "V_REF" I R 7175 5350 60
 F7 "ADC-VOUT" I R 7175 5475 60
@@
 F9 "CLIM" I R 7175 5725 60
 F10 "ISET" O R 7175 5225 60
+F11 "Reset" O L 5450 4825 60
 $EndSheet
 Wire Wire Line
@@
 Wire Wire Line
 	5100 2075 5100 1725
-Wire Wire Line
-	4775 1725 4775 3550
 Connection ~ 4775 3550
 Wire Wire Line
@@
 F2 "5V_direct" I L 5450 3550 60
 F3 "3V3_reg" O R 7025 3875 60
-F4 "V+" O R 7025 3550 60
+F4 "V+" O R 7025 3775 60
 F5 "SCL" I R 7025 4175 60
 F6 "SDA" I R 7025 4075 60
-F7 "ENCONV" I L 5450 4150 60
-$EndSheet
-Wire Wire Line
-	7025 3550 7925 3550
+F7 "ENCONV" I R 7025 3550 60
+$EndSheet
 Wire Wire Line
 	7025 3875 7925 3875
@@
 Connection ~ 7450 4175
 Wire Wire Line
-	5450 4825 5325 4825
-Wire Wire Line
-	5325 4825 5325 4150
-Wire Wire Line
-	5325 4150 5450 4150
-Wire Wire Line
 	9225 4250 9450 4250
 Wire Wire Line
@@
 Wire Wire Line
 	7550 4275 7925 4275
+Wire Wire Line
+	4775 1725 4775 3550
+Wire Wire Line
+	7025 3775 7925 3775
+Wire Wire Line
+	7175 5850 9850 5850
+Wire Wire Line
+	9850 5850 9850 3550
+Wire Wire Line
+	9850 3550 7025 3550
+Wire Wire Line
+	7250 4400 4250 4400
+Wire Wire Line
+	4250 4400 4250 3725
+Wire Wire Line
+	4250 3725 3425 3725
+Connection ~ 7250 4400
+Wire Wire Line
+	7350 4500 4150 4500
+Wire Wire Line
+	4150 4500 4150 3825
+Wire Wire Line
+	4150 3825 3425 3825
+Connection ~ 7350 4500
+Wire Wire Line
+	7450 4600 4050 4600
+Wire Wire Line
+	4050 4600 4050 3925
+Wire Wire Line
+	4050 3925 3425 3925
+Connection ~ 7450 4600
+Wire Wire Line
+	5450 4825 3950 4825
+Wire Wire Line
+	3950 4825 3950 4025
+Wire Wire Line
+	3950 4025 3425 4025
 $EndSCHEMATC

Commit message: update LabBenchPsu
Parts:
- removed F? (x4): FUSE, symbol FUSE
- removed P? (x9): CONN_1, symbol CONN_1
- removed S?: SWITCH, switch, symbol SWITCH-SPSTPTH2
- added F? (x4): FUSE 1A, symbol FUSE
- added P? (x10): CONN_1, symbol CONN_1
- added P? (x2): ED2823-ND, symbol CONN_6
- F?: value FUSE -> FUSE 1A
- R? (x2): value 330R -> 270R
Connections:
- net +12V: now also F?.2
- net +3.3V: now also F?.2
- net -12V: now also F?.2
- net -5V: now also F?.2
- net Charging/5V_direct: now also P?.5, P?.6; no longer F?.1
- net GND: now also P?.1, P?.1, P?.1, P?.4, P?.6
- net PSU/OUT+: now also P?.1
- net at D?.1 (A): now also P?.1
- net at D?.1 (A): now also P?.2
- net at P?.1: now also P?.3
- new net: F?.1, P?.1
- new net: F?.1, P?.2
- new net: F?.1, P?.3
- new net: F?.1, P?.4
- new net: F?.1, P?.5
- no-connect marks 1 -> 12
Other:
- note added: "1: +5V (red)\n2: +12V (yellow)\n3: -5V (white)\n4: -12V (blue)\n5: +3V3 (orange)\n6: GND (black)"
- note added: "1: PGS (gray)\n2: +5vSB (purple)\n3: on-off (green)\n4: GND (black)\n5: +5V (red)\n6: +5V (red)"
- note added: "solder wires directly to switch"
- note added: "wires \nfrom \nPSU"
- note removed: "+12V (yellow)"
- note removed: "+3V3 (orange)"
- note removed: "+5V (red)"
- note removed: "+5vSB (purple)"
- note removed: "-12V (blue)"
- note removed: "-5V (white)"
- note removed: "GND (black)"
- note removed: "PGS (gray)"
- note removed: "on-off (green)"
- moved on the sheet: D?, F?, P?, R?
