File: projects/LabBenchPsu/PSU.sch (KiCad schematic (older format))
At the start: 0 parts

Commit message: LabBenchPsu update
Parts:
- added C? (x9): 100nF, symbol C
- added C? (x2): 2u2, symbol C
- added C?: 22uF, symbol C
- added D? (x2): DIODESCH, symbol DIODESCH
- added IC? (x4): OPAMP-DUALU, SparkFun-SO08, symbol OPAMP-DUALU
- added Q? (x2): 2N3904, TO92, symbol 2N3904
- added R? (x12): 10R, symbol R
- added R? (x8): 18K 0.1%, symbol R
- added R? (x2): 100R, symbol R
- added R? (x2): 1K 0.1%, symbol R
- added R? (x2): 1K, symbol R
- added R? (x4): 10K, symbol R
- added R?: 4K7, symbol R
- added U?: INA219, symbol INA219
- added U?: ISL21070, symbol ISL21070
- added U?: MCP4716, symbol MCP4716
- added U?: LT3083, symbol LT3083
- added U?: LM334Z, symbol LM334Z
Connections:
- new net: C?.2, R?.2, U?.7 (Vin-)
- new net: C?.1, R?.2, U?.8 (Vin+)
- new net: U?.2 (OUT), U?.6 (VREF)
- new net: IC?.3 (+IN), U?.1 (VOUT)
- new net: IC?.1 (OUT), IC?.2 (-IN), R?.2
- new net: C?.1, D?.2 (K), IC?.3 (+IN), R?.1, R?.1, R?.1, R?.1, R?.1, R?.1, R?.1, R?.1, R?.1, R?.1, R?.1, U?.5 (IN)
- new net: IC?.5 (+IN), R?.2, R?.2
- new net: IC?.6 (-IN), R?.1, R?.2
- new net: IC?.7 (OUT), R?.1, R?.1
- new net: IC?.1 (OUT), R?.1
- new net: IC?.2 (-IN), R?.1, R?.1, R?.2
- new net: C?.1, IC?.5 (+IN), R?.2
- new net: C?.1, IC?.6 (-IN), R?.2
- new net: IC?.7 (OUT), R?.1
- new net: C?.1, R?.2, R?.2, R?.2, U?.2 (SET)
- new net: R?.2, U?.2 (R)
- new net: C?.2, C?.2, R?.1, U?.~ (V-)
- new net: R?.1, R?.1, R?.2, R?.2, R?.2, R?.2, R?.2, R?.2, R?.2, R?.2, R?.2, R?.2
- new net: Q?.2 (C), R?.1, R?.2
- new net: Q?.3 (B), R?.2 (x2)
- new net: C?.1, R?.1, R?.1, R?.2
- new net 3V3_reg: C?.1, C?.1, U?.1 (IN), U?.3 (VDD), U?.5 (Vs)
- new net ADC-VOUT: C?.1, R?.1, R?.1, R?.2
- new net CLIM: Q?.2 (C)
- new net GND: C?.1, C?.2, C?.2, C?.2, C?.2, C?.2, C?.2, C?.2, C?.2, D?.1 (A), IC?.4 (V-), IC?.4 (V-), Q?.1 (E), R?.1, R?.1, R?.1, R?.2, U?.1 (A1), U?.2 (A0), U?.2 (VSS), U?.3 (GND), U?.6 (GND)
- new net ISET: R?.1
- new net OUT+: C?.1, D?.1 (A), D?.2 (K), R?.2, R?.2, U?.3 (OUT), U?.~ (V-)
- new net SCL: U?.4 (SCL), U?.5 (SCL)
- new net SDA: U?.3 (SDA), U?.4 (SDA)
- new net V+: C?.1, C?.2, IC?.8 (V+), IC?.8 (V+), U?.4 (VC)
Other:
- note added: "DAC"
- note added: "Voltage reference: \n2.048V"

Commit message: LabBenchPsu updated
Connections:
- net V_REF: now reaches U?.2 (OUT), U?.6 (VREF)
Changed lines of the file:
@@
 Text HLabel 9775 3000 0    60   Input ~ 0
 ADC-VOUT
+Text HLabel 2450 3900 2    60   Output ~ 0
+V_REF
+Wire Wire Line
+	2350 4075 2350 3900
+Wire Wire Line
+	2350 3900 2450 3900
 $EndSCHEMATC

Commit message: LabBenchPsu updated
Connections:
- net ADC-IOUT: now reaches C?.1, IC?.5 (+IN), R?.2
Changed lines of the file:
@@
 Wire Wire Line
 	2350 3900 2450 3900
+Text HLabel 7075 5550 2    60   Output ~ 0
+ADC-IOUT
+Wire Wire Line
+	7075 5550 7000 5550
+Wire Wire Line
+	7000 5550 7000 5650
 $EndSCHEMATC

Commit message: update LabBenchPsu
Parts:
- added P? (x4): CONN_1, symbol CONN_1
Connections:
- net GND: now also Q?.1 (E), P?.1
- net OUT+: now also P?.1; no longer C?.1, D?.1 (A), D?.2 (K), U?.3 (OUT), U?.~ (V-)
- net at IC?.7 (OUT), R?.1: now also R?.1
- new net: C?.1, D?.1 (A), D?.2 (K), P?.1, U?.3 (OUT), U?.~ (V-)
- new net LOAD_ON: P?.1
Other:
- note added: "Loadswitch"
- note added: "i2c configuration:\n1000000 R/W\nRead: 0x81\nWrite: 0x80"
- note added: "i2c configuration:\n1100000 R/W\nRead: 0xC1\nWrite: 0xC0"
- moved on the sheet: C?, D?, R?, U?
