File: projects/LabBenchPsu/Regulation.sch (KiCad schematic (older format))
At the start: 20 parts

Commit message: LabBenchPsu updated
Other:
- note added: "=> V_Out = 5V\n=> V_Out = 22V"
- note added: "R: 4470\nR: 28"
Changed lines of the file:
@@
 	1    0    0    -1
 $EndComp
-Text Notes 4900 4525 0    60   ~ 0
+Text Notes 4900 4475 0    60   ~ 0
 DC-DC
 $Comp
@@
 Text Notes 7450 4950 0    60   ~ 0
 EPOT\n5K 128 Tap
-Text Notes 6475 5175 0    60   ~ 0
+Text Notes 6325 5175 0    60   ~ 0
 R = [584R ... 3K6]
 Wire Notes Line
 	7350 5050 6325 5050
-Text Notes 4850 5525 0    60   ~ 0
+Text Notes 4850 5500 0    60   ~ 0
 V_OUT = [4.8V ... 22.9V]
+Text Notes 6325 5500 0    60   ~ 0
+R: 4470\nR: 28
+Text Notes 6725 5500 0    60   ~ 0
+=> V_Out = 5V\n=> V_Out = 22V
 $EndSCHEMATC

Commit message: update LabBenchPsu
Parts:
- C? (x2): value 470uF -> 47uF
Other:
- note added: "i2c configuration:\n0101100 R/W\nRead: 0x5F\nWrite: 0x5E"
Changed lines of the file:
@@
 Comment2 ""
 Comment3 ""
-Comment4 ""
+Comment4 "- Voltage preregulation with boost converter"
 $EndDescr
 Text HLabel 3000 2425 0    60   Input ~ 0
@@
 P 3300 3775
 F 0 "C?" H 3350 3875 50  0000 L CNN
-F 1 "470uF" H 3350 3675 50  0000 L CNN
+F 1 "47uF" H 3350 3675 50  0000 L CNN
 F 2 "" H 3300 3775 60  0000 C CNN
 F 3 "" H 3300 3775 60  0000 C CNN
@@
 P 7000 3775
 F 0 "C?" H 7050 3875 50  0000 L CNN
-F 1 "470uF" H 7050 3675 50  0000 L CNN
+F 1 "47uF" H 7050 3675 50  0000 L CNN
 F 2 "" H 7000 3775 60  0000 C CNN
 F 3 "" H 7000 3775 60  0000 C CNN
@@
 Text Notes 6725 5500 0    60   ~ 0
 => V_Out = 5V\n=> V_Out = 22V
+Text Notes 7525 4150 0    79   ~ 0
+i2c configuration:\n0101100 R/W\nRead: 0x5F\nWrite: 0x5E
 $EndSCHEMATC
