File: projects/ArduinoController/ArduinoController.kicad_pcb (KiCad board)
At the start: 2 copper layers, 106 parts, among them CN1 DCBARREL, CON1 USB-MICRO, IC1 TMP36, IC2 LM358, J1 Joystick, P1 CONN_4, P2 CONN_4, P3 CONN_3X2, P4 CONN_4, P5 CONN_4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

Commit message: small changes
Parts:
- moved CN1 429.4 mm to (-161.5, 59.2)
- moved IC2 335.9 mm to (-140.7, 71.9)
- moved S6 332.0 mm to (-169.9, 48.0)
- moved R21 315.0 mm to (-163.8, 64.0)
- moved LDR1 311.0 mm to (-161.3, 77.5)
- moved R19 310.8 mm to (-161.5, 84.1)
- moved D4 309.7 mm to (-158.5, 64.3)
- moved C29 305.2 mm to (-156.7, 102.6)
- moved R7 303.3 mm to (-152.7, 140.7)
- moved U7 302.8 mm to (-153.4, 127.5)
- moved R6 301.9 mm to (-151.6, 137.2)
- moved C28 300.7 mm to (-152.1, 110.5)
- moved P8 298.9 mm to (-150.1, 91.7)
- moved C17 295.9 mm to (-147.3, 97.5)
- moved Q2 295.7 mm to (-145.3, 138.9)
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Other:
- board outline added: 227.1 x 265 mm
