File: projects/PowerBox/PowerBox.sch (KiCad schematic (older format))
At the start: 12 parts

Commit message: update PowerBox
Parts:
- added CON?: USB-MICRO, symbol USB-MICRO
- added P? (x2): CONN_2, symbol CONN_2
- added PB?: PowerBoost, symbol PowerBoost
- added S?: Lipo Select, symbol SPDT
- added S? (x2): Load on/off, symbol SPDT
Connections:
- net labels added: V_LOAD, V_MP
- wire segments 19 -> 30
- no-connect marks 1 -> 4
Other:
- note added: "Powerinput"

Commit message: powerbox updated
Parts:
- added CON?: USB-MICRO, symbol USB-MICRO
- added P?: CONN_3X2, symbol CONN_3X2
- R?: value 10K 1% -> 24K 1%
Connections:
- net labels added: I_MEASURE, RESET, SELECT
- net labels removed: V_LOAD
- wire segments 30 -> 36
- no-connect marks 4 -> 7
Other:
- note added: "Is = (Vout * 1k) / (R_shunt * R_L)"
- note added: "Poweroutput"
- note added: "R_L"
- note added: "R_shunt\n1% 0.1W+"
- note removed: "R shunt\n1% 0.1W+"
- moved on the sheet: R?, S?, U?

Commit message: automatic poweroff with LBO signal
Parts:
- removed PB?: PowerBoost, symbol PowerBoost
- added D1: Low Battery, symbol LED
- added D2: Power Load, symbol LED
- added IC1: OPAMP-DUALU, SparkFun-SO08, symbol OPAMP-DUALU
- added P3, P4, P5, P6: CONN_1, symbol CONN_1
- added PB1: PowerBoost, symbol PowerBoost
- added R1, R4: 330R, symbol R
- added R10: 43K 1%, symbol R
- added R11, R8: 49.9K 1%, symbol R
- added R2, R3: 1K, symbol R
- added R9: 78.7K 1%, symbol R
- S3: renamed from S?; value Load on/off -> Attiny on/off
- gave numbers to parts that had none: 19
Connections:
- net labels added: LBO, VS
- wire segments 36 -> 48
- no-connect marks 7 -> 17
Other:
- note added: ""apple resistors":\nD- : 49.9 / (43 + 49.9) * 5.2 = 2.79\nD+: 49.9 / (49.9 + 79) * 5.2 = 2.01"
- note added: "Mounting holes"
- moved on the sheet: C2, CON1, CON2, IC2, P1, P2, P7, R5, R6, R7, S1, S2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

Commit message: update schematic
Parts:
- added R8: 300R 1%, symbol R
- R2, R3: value 1K -> 10K
- renumbered R9 to R10, R10 to R11, R11 to R12, R8 to R9
Other:
- note added: ""apple resistors":\nD-: 49.9 / (49.9 + 43) * 5.2 = 2.79\nD+: 49.9 / (49.9 + 78.7+0.3) * 5.2 = 2.00\n\nidentifies device as wall adapter,\nwhich can deliver charge current of 1A"
- note added: "LBO is HIGH when Batterie is ok"
- note removed: ""apple resistors":\nD- : 49.9 / (43 + 49.9) * 5.2 = 2.79\nD+: 49.9 / (49.9 + 79) * 5.2 = 2.01"
- moved on the sheet: CON2, D1, IC1A, IC1B, R1
Changed lines of the file:
@@
 L USB-MICRO CON2
 U 1 1 5581E5BD
-P 9000 4800
-F 0 "CON2" H 8750 5250 60  0000 C CNN
-F 1 "USB-MICRO" H 8950 4300 60  0000 C CNN
-F 2 "" H 9000 4800 60  0000 C CNN
-F 3 "" H 9000 4800 60  0000 C CNN
-	1    9000 4800
+P 9100 4800
+F 0 "CON2" H 8850 5250 60  0000 C CNN
+F 1 "USB-MICRO" H 9050 4300 60  0000 C CNN
+F 2 "" H 9100 4800 60  0000 C CNN
+F 3 "" H 9100 4800 60  0000 C CNN
+	1    9100 4800
 	1    0    0    -1
 $EndComp
@@
 L GND #PWR024
 U 1 1 5581E5DC
-P 8450 5100
-F 0 "#PWR024" H 8450 5100 30  0001 C CNN
-F 1 "GND" H 8450 5030 30  0001 C CNN
-F 2 "" H 8450 5100 60  0000 C CNN
-F 3 "" H 8450 5100 60  0000 C CNN
-	1    8450 5100
-	0    1    1    0
-$EndComp
-NoConn ~ 8450 4950
+P 8550 5100
+F 0 "#PWR024" H 8550 5100 30  0001 C CNN
+F 1 "GND" H 8550 5030 30  0001 C CNN
+F 2 "" H 8550 5100 60  0000 C CNN
+F 3 "" H 8550 5100 60  0000 C CNN
+	1    8550 5100
+	0    1    1    0
+$EndComp
+NoConn ~ 8550 4950
 Text GLabel 7350 3950 2    47   Input ~ 0
 V_MP
@@
 NoConn ~ 1950 4600
 NoConn ~ 1950 4750
-NoConn ~ 9550 4500
-NoConn ~ 9550 4650
-NoConn ~ 9550 4950
-NoConn ~ 9550 5100
+NoConn ~ 9650 4500
+NoConn ~ 9650 4650
+NoConn ~ 9650 4950
+NoConn ~ 9650 5100
 Wire Wire Line
 	5200 4150 5200 5700
@@
 Connection ~ 5200 4150
 $Comp
-L R R10
+L R R11
 U 1 1 55833755
 P 8300 4400
-F 0 "R10" V 8380 4400 40  0000 C CNN
+F 0 "R11" V 8380 4400 40  0000 C CNN
 F 1 "43K 1%" V 8307 4401 40  0000 C CNN
 F 2 "" V 8230 4400 30  0000 C CNN
@@
 $EndComp
 $Comp
-L R R9
+L R R10
 U 1 1 55833774
 P 8050 4800
-F 0 "R9" V 8130 4800 40  0000 C CNN
+F 0 "R10" V 8130 4800 40  0000 C CNN
 F 1 "78.7K 1%" V 8057 4801 40  0000 C CNN
 F 2 "" V 7980 4800 30  0000 C CNN
@@
 $EndComp
 $Comp
-L R R11
+L R R12
 U 1 1 55833789
 P 8300 5050
-F 0 "R11" V 8380 5050 40  0000 C CNN
+F 0 "R12" V 8380 5050 40  0000 C CNN
 F 1 "49.9K 1%" V 8307 5051 40  0000 C CNN
 F 2 "" V 8230 5050 30  0000 C CNN
@@
 $EndComp
 $Comp
-L R R8
+L R R9
 U 1 1 55833794
 P 8050 4650
-F 0 "R8" V 8130 4650 40  0000 C CNN
+F 0 "R9" V 8130 4650 40  0000 C CNN
 F 1 "49.9K 1%" V 8057 4651 40  0000 C CNN
 F 2 "" V 7980 4650 30  0000 C CNN
@@
 $EndComp
 Wire Wire Line
-	8450 4800 8300 4800
-Wire Wire Line
-	8450 4650 8300 4650
-Wire Wire Line
-	8450 4150 8450 4500
-Wire Wire Line
-	7350 4150 8450 4150
+	8300 4800 8550 4800
+Wire Wire Line
+	8300 4650 8550 4650
+Wire Wire Line
+	7350 4150 8550 4150
 Connection ~ 8300 4150
 Wire Wire Line
 	7800 4800 7650 4800
-Wire Wire Line
-	7650 4800 7650 4150
 Connection ~ 7650 4150
 $Comp
@@
 Text Notes 5825 7000 0    60   ~ 0
 Mounting holes
-Text Notes 7825 3975 0    60   ~ 0
-"apple resistors":\nD- : 49.9 / (43 + 49.9) * 5.2 = 2.79\nD+: 49.9 / (49.9 + 79) * 5.2 = 2.01
+Text Notes 7525 6375 0    60   ~ 0
+"apple resistors":\nD-: 49.9 / (49.9 + 43) * 5.2 = 2.79\nD+: 49.9 / (49.9 + 78.7+0.3) * 5.2 = 2.00\n\nidentifies device as wall adapter,\nwhich can deliver charge current of 1A
 $Comp
 L OPAMP-DUALU IC1
 U 1 1 5583A310
-P 3900 6950
-F 0 "IC1" H 4100 6725 50  0000 R TNN
-F 1 "OPAMP-DUALU" H 4100 7150 50  0000 R TNN
-F 2 "SparkFun-SO08" H 3900 7100 50  0001 C CNN
-F 3 "" H 3900 6950 60  0000 C CNN
-	1    3900 6950
+P 3900 7150
+F 0 "IC1" H 4100 6925 50  0000 R TNN
+F 1 "OPAMP-DUALU" H 4100 7350 50  0000 R TNN
+F 2 "SparkFun-SO08" H 3900 7300 50  0001 C CNN
+F 3 "" H 3900 7150 60  0000 C CNN
+	1    3900 7150
 	1    0    0    -1
 $EndComp
@@
 L OPAMP-DUALU IC1
 U 2 1 5583A324
-P 2700 6950
-F 0 "IC1" H 2900 6725 50  0000 R TNN
-F 1 "OPAMP-DUALU" H 2900 7150 50  0000 R TNN
-F 2 "SparkFun-SO08" H 2700 7100 50  0001 C CNN
-F 3 "" H 2700 6950 60  0000 C CNN
-	2    2700 6950
+P 2700 7150
+F 0 "IC1" H 2900 6925 50  0000 R TNN
+F 1 "OPAMP-DUALU" H 2900 7350 50  0000 R TNN
+F 2 "SparkFun-SO08" H 2700 7300 50  0001 C CNN
+F 3 "" H 2700 7150 60  0000 C CNN
+	2    2700 7150
 	-1   0    0    1
 $EndComp
@@
 Wire Wire Line
 	4000 4250 4000 4150
-Text GLabel 3700 6850 0    47   Input ~ 0
+Text GLabel 3700 7250 0    47   Input ~ 0
 LBO
 Text GLabel 3700 4150 3    47   Output ~ 0
@@
 L GND #PWR027
 U 1 1 55845A65
-P 3900 7250
-F 0 "#PWR027" H 3900 7250 30  0001 C CNN
-F 1 "GND" H 3900 7180 30  0001 C CNN
-F 2 "" H 3900 7250 60  0000 C CNN
-F 3 "" H 3900 7250 60  0000 C CNN
-	1    3900 7250
+P 3900 7450
+F 0 "#PWR027" H 3900 7450 30  0001 C CNN
+F 1 "GND" H 3900 7380 30  0001 C CNN
+F 2 "" H 3900 7450 60  0000 C CNN
+F 3 "" H 3900 7450 60  0000 C CNN
+	1    3900 7450
 	-1   0    0    -1
 $EndComp
@@
 P 3350 6800
 F 0 "R2" V 3430 6800 40  0000 C CNN
-F 1 "1K" V 3357 6801 40  0000 C CNN
+F 1 "10K" V 3357 6801 40  0000 C CNN
 F 2 "" V 3280 6800 30  0000 C CNN
 F 3 "" H 3350 6800 30  0000 C CNN
@@
 P 3350 7300
 F 0 "R3" V 3430 7300 40  0000 C CNN
-F 1 "1K" V 3357 7301 40  0000 C CNN
+F 1 "10K" V 3357 7301 40  0000 C CNN
 F 2 "" V 3280 7300 30  0000 C CNN
 F 3 "" H 3350 7300 30  0000 C CNN
@@
 $EndComp
 Wire Wire Line
-	3900 6550 3900 6650
+	3900 6550 3900 6850
 Wire Wire Line
 	3000 7050 3700 7050
 Wire Wire Line
-	4300 6950 4500 6950
-Wire Wire Line
-	4500 6950 4500 5700
+	4500 5700 4500 7150
 Wire Wire Line
 	3350 6450 3350 6550
 Wire Wire Line
 	3350 6550 3900 6550
-Text GLabel 3000 6850 2    47   Input ~ 0
+Text GLabel 3000 7250 2    47   Input ~ 0
 LBO
 Connection ~ 3350 7050
@@
 L R R1
 U 1 1 55846585
-P 2150 6950
-F 0 "R1" V 2230 6950 40  0000 C CNN
-F 1 "330R" V 2157 6951 40  0000 C CNN
-F 2 "" V 2080 6950 30  0000 C CNN
-F 3 "" H 2150 6950 30  0000 C CNN
-	1    2150 6950
+P 2150 7150
+F 0 "R1" V 2230 7150 40  0000 C CNN
+F 1 "330R" V 2157 7151 40  0000 C CNN
+F 2 "" V 2080 7150 30  0000 C CNN
+F 3 "" H 2150 7150 30  0000 C CNN
+	1    2150 7150
 	0    -1   -1   0
 $EndComp
@@
 L LED D1
 U 1 1 55846747
-P 1700 6950
-F 0 "D1" H 1700 7050 50  0000 C CNN
-F 1 "Low Battery" H 1700 6850 50  0000 C CNN
-F 2 "" H 1700 6950 60  0000 C CNN
-F 3 "" H 1700 6950 60  0000 C CNN
-	1    1700 6950
+P 1700 7150
+F 0 "D1" H 1700 7250 50  0000 C CNN
+F 1 "Low Battery" H 1700 7050 50  0000 C CNN
+F 2 "" H 1700 7150 60  0000 C CNN
+F 3 "" H 1700 7150 60  0000 C CNN
+	1    1700 7150
 	-1   0    0    1
 $EndComp
@@
 L GND #PWR029
 U 1 1 5584676D
-P 1500 6950
-F 0 "#PWR029" H 1500 6950 30  0001 C CNN
-F 1 "GND" H 1500 6880 30  0001 C CNN
-F 2 "" H 1500 6950 60  0000 C CNN
-F 3 "" H 1500 6950 60  0000 C CNN
-	1    1500 6950
+P 1500 7150
+F 0 "#PWR029" H 1500 7150 30  0001 C CNN
+F 1 "GND" H 1500 7080 30  0001 C CNN
+F 2 "" H 1500 7150 60  0000 C CNN
+F 3 "" H 1500 7150 60  0000 C CNN
+	1    1500 7150
 	0    1    -1   0
 $EndComp
@@
 Wire Wire Line
 	5350 7050 5350 7250
+$Comp
+L R R8
+U 1 1 5586A13E
+P 7650 4400
+F 0 "R8" V 7730 4400 40  0000 C CNN
+F 1 "300R 1%" V 7657 4401 40  0000 C CNN
+F 2 "" V 7580 4400 30  0000 C CNN
+F 3 "" H 7650 4400 30  0000 C CNN
+	1    7650 4400
+	-1   0    0    1
+$EndComp
+Wire Wire Line
+	7650 4800 7650 4650
+Text Notes 1625 6725 0    60   ~ 0
+LBO is HIGH when Batterie is ok
+Wire Wire Line
+	8550 4150 8550 4500
+Wire Bus Line
+	7500 4050 8400 4050
+Wire Bus Line
+	8400 4050 8400 5750
+Wire Bus Line
+	8400 5750 7500 5750
+Wire Bus Line
+	7500 5750 7500 4050
+Wire Wire Line
+	4500 7150 4300 7150
 $EndSCHEMATC

Commit message: new display driver with 74HC595
Parts:
- removed C1: 10uF, symbol CP1
- removed C2: 100nF, symbol C
- removed SEG1: 4_x_7Segment, symbol 4_x_7Segment
- removed U1: MAX7219, symbol MAX7219
- added JP1: JUMPER, symbol JUMPER
- added R1, R2, R3, R4, R7, R8, R9: 300R, symbol R
- added U1, U2: 74HC595, symbol 74HC595
- R6: value 12K -> 300R
- renumbered R2 to R10, R3 to R11, R4 to R12, R5 to R13, R7 to R14, R8 to R15, R9 to R16, R10 to R17, R11 to R18, R12 to R19, R1 to R5, SEG2 to SEG1, U2 to U3
Connections:
- net labels removed: D4, D5, D6, D7
- wire segments 48 -> 50
- no-connect marks 17 -> 21
Other:
- note added: "Jumper for current measurement"
- moved on the sheet: CON1, CON2, D1, D2, IC1A, IC1B, P1, P2, P3, P4, P5, P6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

Commit message: new footprints added
Parts:
- added C1: 1uF, symbol C
- added C2: 100nF, symbol C
- R1, R2, R3, R4, R6, R7, R8, R9: value 300R -> 220R
Connections:
- net GND: now also C1.2, C2.2
- net LBO: now also IC1.6 (-IN); no longer IC1.5 (+IN)
- net VCC: now also C1.1, C2.1
- net at IC1.2 (-IN), R10.1, R11.2: now also IC1.5 (+IN); no longer IC1.6 (-IN)
Other:
- note added: "+ -"
- moved on the sheet: D1, IC1B, IC2, R5, S5
Changed lines of the file:
@@
 LIBS:valves
 LIBS:frep
+LIBS:PowerBox-cache
 EELAYER 24 0
 EELAYER END
@@
 L ATTINY85-S IC2
 U 1 1 55806C90
-P 9175 1450
-F 0 "IC2" H 8125 1850 60  0000 C CNN
-F 1 "ATTINY85-S" H 10025 1050 60  0000 C CNN
-F 2 "SO8-200" H 8275 1050 60  0001 C CNN
-F 3 "" H 9175 1450 60  0000 C CNN
-	1    9175 1450
-	1    0    0    -1
-$EndComp
-Text GLabel 7825 1600 0    47   Input ~ 0
+P 8750 1450
+F 0 "IC2" H 7700 1850 60  0000 C CNN
+F 1 "ATTINY85-S" H 9600 1050 60  0000 C CNN
+F 2 "SO8-200" H 7850 1050 60  0001 C CNN
+F 3 "" H 8750 1450 60  0000 C CNN
+	1    8750 1450
+	1    0    0    -1
+$EndComp
+Text GLabel 7400 1600 0    47   Input ~ 0
 LOAD
-Text GLabel 7825 1500 0    47   Input ~ 0
+Text GLabel 7400 1500 0    47   Input ~ 0
 CLK
-Text GLabel 7825 1200 0    47   Input ~ 0
+Text GLabel 7400 1200 0    47   Input ~ 0
 DIN
 Wire Wire Line
@@
 L TAC_SWITCH S5
 U 1 1 558071DB
-P 8475 2725
-F 0 "S5" H 8450 2925 50  0000 L BNN
-F 1 "RESET" H 8375 2500 50  0000 L BNN
-F 2 "TACTILE" H 8475 2875 50  0001 C CNN
-F 3 "" H 8475 2725 60  0000 C CNN
-	1    8475 2725
+P 8500 2750
+F 0 "S5" H 8475 2950 50  0000 L BNN
+F 1 "RESET" H 8400 2525 50  0000 L BNN
+F 2 "TACTILE" H 8500 2900 50  0001 C CNN
+F 3 "" H 8500 2750 60  0000 C CNN
+	1    8500 2750
 	0    -1   -1   0
 $EndComp
@@
 L GND #PWR03
 U 1 1 55807293
-P 8575 3025
-F 0 "#PWR03" H 8575 3025 30  0001 C CNN
-F 1 "GND" H 8575 2955 30  0001 C CNN
-F 2 "" H 8575 3025 60  0000 C CNN
-F 3 "" H 8575 3025 60  0000 C CNN
-	1    8575 3025
+P 8600 3050
+F 0 "#PWR03" H 8600 3050 30  0001 C CNN
+F 1 "GND" H 8600 2980 30  0001 C CNN
+F 2 "" H 8600 3050 60  0000 C CNN
+F 3 "" H 8600 3050 60  0000 C CNN
+	1    8600 3050
 	-1   0    0    -1
 $EndComp
@@
 L GND #PWR05
 U 1 1 55808163
-P 10525 1700
-F 0 "#PWR05" H 10525 1700 30  0001 C CNN
-F 1 "GND" H 10525 1630 30  0001 C CNN
-F 2 "" H 10525 1700 60  0000 C CNN
-F 3 "" H 10525 1700 60  0000 C CNN
-	1    10525 1700
+P 10100 1700
+F 0 "#PWR05" H 10100 1700 30  0001 C CNN
+F 1 "GND" H 10100 1630 30  0001 C CNN
+F 2 "" H 10100 1700 60  0000 C CNN
+F 3 "" H 10100 1700 60  0000 C CNN
+	1    10100 1700
 	0    -1   1    0
 $EndComp
 Wire Wire Line
-	8575 2525 8475 2525
-Wire Wire Line
-	8575 2925 8475 2925
+	8600 2550 8500 2550
+Wire Wire Line
+	8600 2950 8500 2950
 $Comp
 L USB-MICRO CON1
@@
 Wire Wire Line
 	5800 3750 5700 3750
-Text GLabel 7825 1400 0    47   Input ~ 0
+Text GLabel 7400 1400 0    47   Input ~ 0
 I_MEASURE
-Text GLabel 10525 1200 2    47   Input ~ 0
+Text GLabel 10650 1200 2    47   Input ~ 0
 V_MP
 $Comp
@@
 	1    0    0    -1
 $EndComp
-Text GLabel 7825 1300 0    47   Input ~ 0
+Text GLabel 7400 1300 0    47   Input ~ 0
 SELECT
-Text GLabel 7825 1700 0    47   Input ~ 0
+Text GLabel 7400 1700 0    47   Input ~ 0
 RESET
 Wire Wire Line
-	8575 3025 8575 2925
+	8600 3050 8600 2950
 Text GLabel 7950 2450 1    47   Output ~ 0
 SELECT
 Wire Wire Line
 	7950 2550 7950 2450
-Text GLabel 8575 2425 1    47   Output ~ 0
+Text GLabel 8600 2450 1    47   Output ~ 0
 RESET
 Wire Wire Line
-	8575 2425 8575 2525
+	8600 2450 8600 2550
 Text GLabel 9500 2600 0    47   Input ~ 0
 SELECT
@@
 L OPAMP-DUALU IC1
 U 2 1 5583A324
-P 2350 7150
-F 0 "IC1" H 2550 6925 50  0000 R TNN
-F 1 "OPAMP-DUALU" H 2550 7350 50  0000 R TNN
-F 2 "SparkFun-SO08" H 2350 7300 50  0001 C CNN
-F 3 "" H 2350 7150 60  0000 C CNN
-	2    2350 7150
+P 2350 6950
+F 0 "IC1" H 2550 6725 50  0000 R TNN
+F 1 "OPAMP-DUALU" H 2550 7150 50  0000 R TNN
+F 2 "SparkFun-SO08" H 2350 7100 50  0001 C CNN
+F 3 "" H 2350 6950 60  0000 C CNN
+	2    2350 6950
 	-1   0    0    1
 $EndComp
@@
 Wire Wire Line
 	3000 6550 3550 6550
-Text GLabel 2650 7250 2    47   Input ~ 0
+Text GLabel 2650 6850 2    47   Input ~ 0
 LBO
 Connection ~ 3000 7050
@@
 L R R5
 U 1 1 55846585
-P 1800 7150
-F 0 "R5" V 1880 7150 40  0000 C CNN
-F 1 "330R" V 1807 7151 40  0000 C CNN
-F 2 "" V 1730 7150 30  0000 C CNN
-F 3 "" H 1800 7150 30  0000 C CNN
-	1    1800 7150
+P 1800 6950
+F 0 "R5" V 1880 6950 40  0000 C CNN
+F 1 "330R" V 1807 6951 40  0000 C CNN
+F 2 "" V 1730 6950 30  0000 C CNN
+F 3 "" H 1800 6950 30  0000 C CNN
+	1    1800 6950
 	0    -1   -1   0
 $EndComp
@@
 L LED D1
 U 1 1 55846747
-P 1350 7150
-F 0 "D1" H 1350 7250 50  0000 C CNN
-F 1 "Low Battery" H 1350 7050 50  0000 C CNN
-F 2 "" H 1350 7150 60  0000 C CNN
-F 3 "" H 1350 7150 60  0000 C CNN
-	1    1350 7150
+P 1350 6950
+F 0 "D1" H 1350 7050 50  0000 C CNN
+F 1 "Low Battery" H 1350 6850 50  0000 C CNN
+F 2 "" H 1350 6950 60  0000 C CNN
+F 3 "" H 1350 6950 60  0000 C CNN
+	1    1350 6950
 	-1   0    0    1
 $EndComp
@@
 L GND #PWR025
 U 1 1 5584676D
-P 1150 7150
-F 0 "#PWR025" H 1150 7150 30  0001 C CNN
-F 1 "GND" H 1150 7080 30  0001 C CNN
-F 2 "" H 1150 7150 60  0000 C CNN
-F 3 "" H 1150 7150 60  0000 C CNN
-	1    1150 7150
+P 1150 6950
+F 0 "#PWR025" H 1150 6950 30  0001 C CNN
+F 1 "GND" H 1150 6880 30  0001 C CNN
+F 2 "" H 1150 6950 60  0000 C CNN
+F 3 "" H 1150 6950 60  0000 C CNN
+	1    1150 6950
 	0    1    -1   0
 $EndComp
@@
 Wire Wire Line
 	8000 4800 8000 4650
-Text Notes 1275 6725 0    60   ~ 0
+Text Notes 1150 7375 0    60   ~ 0
 LBO is HIGH when Batterie is ok
 Wire Wire Line
@@
 Wire Wire Line
 	7750 4150 8900 4150
-Text Notes 7475 5850 1    60   ~ 0
+Text Notes 7500 5975 1    60   ~ 0
 Jumper for current measurement
 $Comp
@@
 P 1850 2600
 F 0 "R6" V 1930 2600 40  0000 C CNN
-F 1 "300R" V 1857 2601 40  0000 C CNN
+F 1 "220R" V 1857 2601 40  0000 C CNN
 F 2 "" V 1780 2600 30  0000 C CNN
 F 3 "" H 1850 2600 30  0000 C CNN
@@
 P 2000 2600
 F 0 "R7" V 2080 2600 40  0000 C CNN
-F 1 "300R" V 2007 2601 40  0000 C CNN
+F 1 "220R" V 2007 2601 40  0000 C CNN
 F 2 "" V 1930 2600 30  0000 C CNN
 F 3 "" H 2000 2600 30  0000 C CNN
@@
 P 2150 2600
 F 0 "R8" V 2230 2600 40  0000 C CNN
-F 1 "300R" V 2157 2601 40  0000 C CNN
+F 1 "220R" V 2157 2601 40  0000 C CNN
 F 2 "" V 2080 2600 30  0000 C CNN
 F 3 "" H 2150 2600 30  0000 C CNN
@@
 P 2300 2600
 F 0 "R9" V 2380 2600 40  0000 C CNN
-F 1 "300R" V 2307 2601 40  0000 C CNN
+F 1 "220R" V 2307 2601 40  0000 C CNN
 F 2 "" V 2230 2600 30  0000 C CNN
 F 3 "" H 2300 2600 30  0000 C CNN
@@
 P 1250 2600
 F 0 "R1" V 1330 2600 40  0000 C CNN
-F 1 "300R" V 1257 2601 40  0000 C CNN
+F 1 "220R" V 1257 2601 40  0000 C CNN
 F 2 "" V 1180 2600 30  0000 C CNN
 F 3 "" H 1250 2600 30  0000 C CNN
@@
 P 1400 2600
 F 0 "R2" V 1480 2600 40  0000 C CNN
-F 1 "300R" V 1407 2601 40  0000 C CNN
+F 1 "220R" V 1407 2601 40  0000 C CNN
 F 2 "" V 1330 2600 30  0000 C CNN
 F 3 "" H 1400 2600 30  0000 C CNN
@@
 P 1550 2600
 F 0 "R3" V 1630 2600 40  0000 C CNN
-F 1 "300R" V 1557 2601 40  0000 C CNN
+F 1 "220R" V 1557 2601 40  0000 C CNN
 F 2 "" V 1480 2600 30  0000 C CNN
 F 3 "" H 1550 2600 30  0000 C CNN
@@
 P 1700 2600
 F 0 "R4" V 1780 2600 40  0000 C CNN
-F 1 "300R" V 1707 2601 40  0000 C CNN
+F 1 "220R" V 1707 2601 40  0000 C CNN
 F 2 "" V 1630 2600 30  0000 C CNN
 F 3 "" H 1700 2600 30  0000 C CNN
@@
 	-1   0    0    1
 $EndComp
+Text Notes 7300 4325 0    60   ~ 0
++   -
+$Comp
+L C C1
+U 1 1 558C175F
+P 10250 1400
+F 0 "C1" H 10250 1500 40  0000 L CNN
+F 1 "1uF" H 10256 1315 40  0000 L CNN
+F 2 "" H 10288 1250 30  0000 C CNN
+F 3 "" H 10250 1400 60  0000 C CNN
+	1    10250 1400
+	1    0    0    -1
+$EndComp
+$Comp
+L C C2
+U 1 1 558C177B
+P 10500 1400
+F 0 "C2" H 10500 1500 40  0000 L CNN
+F 1 "100nF" H 10506 1315 40  0000 L CNN
+F 2 "" H 10538 1250 30  0000 C CNN
+F 3 "" H 10500 1400 60  0000 C CNN
+	1    10500 1400
+	1    0    0    -1
+$EndComp
+$Comp
+L GND #PWR035
+U 1 1 558C178E
+P 10250 1600
+F 0 "#PWR035" H 10250 1600 30  0001 C CNN
+F 1 "GND" H 10250 1530 30  0001 C CNN
+F 2 "" H 10250 1600 60  0000 C CNN
+F 3 "" H 10250 1600 60  0000 C CNN
+	1    10250 1600
+	-1   0    0    -1
+$EndComp
+$Comp
+L GND #PWR036
+U 1 1 558C1799
+P 10500 1600
+F 0 "#PWR036" H 10500 1600 30  0001 C CNN
+F 1 "GND" H 10500 1530 30  0001 C CNN
+F 2 "" H 10500 1600 60  0000 C CNN
+F 3 "" H 10500 1600 60  0000 C CNN
+	1    10500 1600
+	-1   0    0    -1
+$EndComp
+Wire Wire Line
+	10100 1200 10650 1200
+Connection ~ 10500 1200
+Connection ~ 10250 1200
 $EndSCHEMATC
