File: projects/PowerBox/PowerBox.sch (KiCad schematic (older format))
At the start: 60 parts, among them CON1 USB-MICRO, CON2 USB-A-Jack, IC1 LM358, IC2 LM358, P1 CONN_2, P2 CONN_2, P3 CONN_1, P4 CONN_1, P5 CONN_1, P6 CONN_1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

Commit message: layout in progress
Parts:
- JP2: value JUMPER -> + -
Other:
- note removed: "+ -"
Changed lines of the file:
@@
 P 6750 3900
 F 0 "JP2" H 6750 4050 60  0000 C CNN
-F 1 "JUMPER" H 6750 3820 40  0000 C CNN
+F 1 "+ -" H 6750 3820 40  0000 C CNN
 F 2 "frep:Pin_Proto_Straight_1x02" H 6750 3900 60  0001 C CNN
 F 3 "" H 6750 3900 60  0000 C CNN
@@
 Text Notes 8100 3650 2    60   ~ 0
 Jumper for current measurement
-Text Notes 6600 4075 0    60   ~ 0
-+   -
 $Sheet
 S 6600 2050 1450 1300

Commit message: pcb layout still in progress
Connections:
- net VCC: now also U1.10 (SRCLR), U3.10 (SRCLR)
- net V_MP: no longer U1.10 (SRCLR), U3.10 (SRCLR)
Changed lines of the file:
@@
 Text GLabel 3200 2200 2    47   Output ~ 0
 SEGDP
-Text GLabel 1800 1800 0    47   Input ~ 0
-V_MP
-Text GLabel 4000 1800 0    47   Input ~ 0
-V_MP
 $Comp
 L GND #PWR025
@@
 Text GLabel 4400 1300 1    47   Input ~ 0
 VREG_in
+Text GLabel 1800 1800 0    47   Input ~ 0
+VREG_in
+Text GLabel 4000 1800 0    47   Input ~ 0
+VREG_in
 $EndSCHEMATC

Commit message: arduino pins labled
Parts:
- D6: value V_bat -> V bat
- D7: value V_load -> V load
- D8: value i_load -> I load
- D9: value P_load -> P load
Changed lines of the file:
@@
 P 7500 800
 F 0 "D6" H 7500 900 50  0000 C CNN
-F 1 "V_bat" H 7500 700 50  0000 C CNN
+F 1 "V bat" H 7500 700 50  0000 C CNN
 F 2 "frep:LED-0805" H 7500 800 60  0001 C CNN
 F 3 "" H 7500 800 60  0000 C CNN
@@
 P 7500 1100
 F 0 "D7" H 7500 1200 50  0000 C CNN
-F 1 "V_load" H 7500 1000 50  0000 C CNN
+F 1 "V load" H 7500 1000 50  0000 C CNN
 F 2 "frep:LED-0805" H 7500 1100 60  0001 C CNN
 F 3 "" H 7500 1100 60  0000 C CNN
@@
 P 7500 1400
 F 0 "D8" H 7500 1500 50  0000 C CNN
-F 1 "i_load" H 7500 1300 50  0000 C CNN
+F 1 "I load" H 7500 1300 50  0000 C CNN
 F 2 "frep:LED-0805" H 7500 1400 60  0001 C CNN
 F 3 "" H 7500 1400 60  0000 C CNN
@@
 P 7500 1700
 F 0 "D9" H 7500 1800 50  0000 C CNN
-F 1 "P_load" H 7500 1600 50  0000 C CNN
+F 1 "P load" H 7500 1600 50  0000 C CNN
 F 2 "frep:LED-0805" H 7500 1700 60  0001 C CNN
 F 3 "" H 7500 1700 60  0000 C CNN

Commit message: digikey partnumbers in schematic added
Parts:
- D10, D2: DK (none) -> 568-6472-1-ND
- D3, D4: DK (none) -> SDM40E20LC-7DICT-ND
- IC1, IC2: DK (none) -> LM358MXFSCT-ND
- P1, P2: DK (none) -> 455-1704-ND
- Q1, Q2, Q3: DK (none) -> DMG3415UDICT-ND
- R11: DK (none) -> P300CCT-ND
- R12, R15: DK (none) -> P49.9KCCT-ND
- R13: DK (none) -> P78.7KCCT-ND
- R14: DK (none) -> P43.0KCCT-ND
- R16, R17, R18, R19, R20, R21, R22, R23, R4, R5: DK (none) -> P220CCT-ND
- S1, S2, S3: DK (none) -> CKN9565-ND
- U1, U3: DK (none) -> 296-14858-1-ND
- U2: DK (none) -> ICL7660AIBAZA-ND
Changed lines of the file:
@@
 F 2 "frep:Switch_SPDT" H 6000 5500 60  0001 C CNN
 F 3 "" H 6000 5500 60  0000 C CNN
+F 4 "CKN9565-ND" H 6000 5500 60  0001 C CNN "DK"
 	1    6000 5500
 	0    1    1    0
@@
 F 2 "frep:JST-PH-2-THM" H 3150 6200 60  0001 C CNN
 F 3 "" H 3150 6200 60  0000 C CNN
+F 4 "455-1704-ND" V 3150 6200 60  0001 C CNN "DK"
 	1    3150 6200
 	-1   0    0    1
@@
 F 2 "frep:JST-PH-2-THM" H 4650 6200 60  0001 C CNN
 F 3 "" H 4650 6200 60  0000 C CNN
+F 4 "455-1704-ND" V 4650 6200 60  0001 C CNN "DK"
 	1    4650 6200
 	1    0    0    1
@@
 F 2 "frep:Switch_SPDT" H 6700 5500 60  0001 C CNN
 F 3 "" H 6700 5500 60  0000 C CNN
+F 4 "CKN9565-ND" H 6700 5500 60  0001 C CNN "DK"
 	1    6700 5500
 	0    1    1    0
@@
 F 2 "frep:Switch_SPDT" H 7400 5500 60  0001 C CNN
 F 3 "" H 7400 5500 60  0000 C CNN
+F 4 "CKN9565-ND" H 7400 5500 60  0001 C CNN "DK"
 	1    7400 5500
 	0    1    1    0
@@
 F 2 "frep:R0805" V 8880 4150 30  0001 C CNN
 F 3 "" H 8950 4150 30  0000 C CNN
+F 4 "P43.0KCCT-ND" V 8950 4150 60  0001 C CNN "DK"
 	1    8950 4150
 	-1   0    0    1
@@
 F 2 "frep:R0805" V 8630 4550 30  0001 C CNN
 F 3 "" H 8700 4550 30  0000 C CNN
+F 4 "P78.7KCCT-ND" V 8700 4550 60  0001 C CNN "DK"
 	1    8700 4550
 	0    -1   -1   0
@@
 F 2 "frep:R0805" V 8880 4800 30  0001 C CNN
 F 3 "" H 8950 4800 30  0000 C CNN
+F 4 "P49.9KCCT-ND" V 8950 4800 60  0001 C CNN "DK"
 	1    8950 4800
 	-1   0    0    1
@@
 F 2 "frep:R0805" V 8630 4400 30  0001 C CNN
 F 3 "" H 8700 4400 30  0000 C CNN
+F 4 "P49.9KCCT-ND" V 8700 4400 60  0001 C CNN "DK"
 	1    8700 4400
 	0    -1   -1   0
@@
 F 2 "frep:SOIC8" H 1600 6150 50  0001 C CNN
 F 3 "" H 1600 6000 60  0000 C CNN
+F 4 "LM358MXFSCT-ND" H 1600 6000 60  0001 C CNN "DK"
 	1    1600 6000
 	1    0    0    -1
@@
 F 2 "frep:SOIC8" H 1700 6750 50  0001 C CNN
 F 3 "" H 1700 6600 60  0000 C CNN
+F 4 "LM358MXFSCT-ND" H 1700 6600 60  0001 C CNN "DK"
 	2    1700 6600
 	1    0    0    -1
@@
 F 2 "frep:R0805" V 2080 6850 30  0001 C CNN
 F 3 "" H 2150 6850 30  0000 C CNN
+F 4 "P220CCT-ND" V 2150 6850 60  0001 C CNN "DK"
 	1    2150 6850
 	-1   0    0    1
@@
 F 2 "frep:R0805" V 5080 3650 30  0001 C CNN
 F 3 "" H 5150 3650 30  0000 C CNN
+F 4 "P220CCT-ND" V 5150 3650 60  0001 C CNN "DK"
 	1    5150 3650
 	0    1    1    0
@@
 F 2 "frep:R0805" V 8230 4150 30  0001 C CNN
 F 3 "" H 8300 4150 30  0000 C CNN
+F 4 "P300CCT-ND" V 8300 4150 60  0001 C CNN "DK"
 	1    8300 4150
 	-1   0    0    1
@@
 F 2 "frep:SO16" H 2500 1950 60  0001 C CNN
 F 3 "" H 2500 1950 60  0000 C CNN
+F 4 "296-14858-1-ND" H 2500 1950 60  0001 C CNN "DK"
 	1    2500 1950
 	1    0    0    -1
@@
 F 2 "frep:SO16" H 4700 1950 60  0001 C CNN
 F 3 "" H 4700 1950 60  0000 C CNN
+F 4 "296-14858-1-ND" H 4700 1950 60  0001 C CNN "DK"
 	1    4700 1950
 	1    0    0    -1
@@
 F 2 "frep:R0805" V 8980 2700 30  0001 C CNN
 F 3 "" H 9050 2700 30  0000 C CNN
+F 4 "P220CCT-ND" V 9050 2700 60  0001 C CNN "DK"
 	1    9050 2700
 	1    0    0    -1
@@
 F 2 "frep:R0805" V 9130 2700 30  0001 C CNN
 F 3 "" H 9200 2700 30  0000 C CNN
+F 4 "P220CCT-ND" V 9200 2700 60  0001 C CNN "DK"
 	1    9200 2700
 	1    0    0    -1
@@
 F 2 "frep:R0805" V 9280 2700 30  0001 C CNN
 F 3 "" H 9350 2700 30  0000 C CNN
+F 4 "P220CCT-ND" V 9350 2700 60  0001 C CNN "DK"
 	1    9350 2700
 	1    0    0    -1
@@
 F 2 "frep:R0805" V 9430 2700 30  0001 C CNN
 F 3 "" H 9500 2700 30  0000 C CNN
+F 4 "P220CCT-ND" V 9500 2700 60  0001 C CNN "DK"
 	1    9500 2700
 	1    0    0    -1
@@
 F 2 "frep:R0805" V 9580 2700 30  0001 C CNN
 F 3 "" H 9650 2700 30  0000 C CNN
+F 4 "P220CCT-ND" V 9650 2700 60  0001 C CNN "DK"
 	1    9650 2700
 	1    0    0    -1
@@
 F 2 "frep:R0805" V 9730 2700 30  0001 C CNN
 F 3 "" H 9800 2700 30  0000 C CNN
+F 4 "P220CCT-ND" V 9800 2700 60  0001 C CNN "DK"
 	1    9800 2700
 	1    0    0    -1
@@
 F 2 "frep:R0805" V 9880 2700 30  0001 C CNN
 F 3 "" H 9950 2700 30  0000 C CNN
+F 4 "P220CCT-ND" V 9950 2700 60  0001 C CNN "DK"
 	1    9950 2700
 	1    0    0    -1
@@
 F 2 "frep:R0805" V 10030 2700 30  0001 C CNN
 F 3 "" H 10100 2700 30  0000 C CNN
+F 4 "P220CCT-ND" V 10100 2700 60  0001 C CNN "DK"
 	1    10100 2700
 	1    0    0    -1
@@
 F 2 "frep:SOT23" V 5750 2850 50  0001 C CNN
 F 3 "" V 5600 2850 60  0000 C CNN
+F 4 "DMG3415UDICT-ND" H 5600 2850 60  0001 C CNN "DK"
 	1    5600 2850
 	1    0    0    1
@@
 F 2 "frep:SOIC8" H 2800 5600 50  0001 C CNN
 F 3 "" H 2800 5450 60  0000 C CNN
+F 4 "LM358MXFSCT-ND" H 2800 5450 60  0001 C CNN "DK"
 	1    2800 5450
 	1    0    0    -1
@@
 F 2 "frep:SOIC8" H 4900 5600 50  0001 C CNN
 F 3 "" H 4900 5450 60  0000 C CNN
+F 4 "LM358MXFSCT-ND" H 4900 5450 60  0001 C CNN "DK"
 	2    4900 5450
 	-1   0    0    -1
@@
 F 2 "frep:SOT23" V 3650 5450 50  0001 C CNN
 F 3 "" V 3500 5450 60  0000 C CNN
+F 4 "DMG3415UDICT-ND" H 3500 5450 60  0001 C CNN "DK"
 	1    3500 5450
 	0    -1   -1   0
@@
 F 2 "frep:SOT23" V 4450 5450 50  0001 C CNN
 F 3 "" V 4300 5450 60  0000 C CNN
+F 4 "DMG3415UDICT-ND" H 4300 5450 60  0001 C CNN "DK"
 	1    4300 5450
 	0    1    -1   0
@@
 F 2 "frep:SOT23" H 3300 4300 60  0001 C CNN
 F 3 "" H 3300 4300 60  0000 C CNN
+F 4 "SDM40E20LC-7DICT-ND" H 3300 4300 60  0001 C CNN "DK"
 	1    3300 4300
 	0    1    1    0
@@
 F 2 "frep:SOT23" H 3900 6100 60  0001 C CNN
 F 3 "" H 3900 6100 60  0000 C CNN
+F 4 "SDM40E20LC-7DICT-ND" H 3900 6100 60  0001 C CNN "DK"
 	1    3900 6100
 	1    0    0    -1
@@
 F 2 "frep:SOT23" H 2650 4100 60  0001 C CNN
 F 3 "" H 2650 4100 60  0000 C CNN
+F 4 "568-6472-1-ND" H 2650 4100 60  0001 C CNN "DK"
 	1    2650 4100
 	0    -1   -1   0
@@
 F 2 "frep:SOT23" H 7700 4100 60  0001 C CNN
 F 3 "" H 7700 4100 60  0000 C CNN
+F 4 "568-6472-1-ND" H 7700 4100 60  0001 C CNN "DK"
 	1    7700 4100
 	0    -1   -1   0
@@
 F 2 "frep:SOIC8" H 3950 6950 60  0001 C CNN
 F 3 "" H 3950 6950 60  0000 C CNN
+F 4 "ICL7660AIBAZA-ND" H 3950 6950 60  0001 C CNN "DK"
 	1    3950 6950
 	1    0    0    -1

Commit message: footprints changed and tracks adjusted
Parts:
- U1, U3: footprint frep:SO16 -> frep:SO-16-L
Changed lines of the file:
@@
 F 0 "U1" H 2650 2550 70  0000 C CNN
 F 1 "74HC595" H 2500 1350 70  0000 C CNN
-F 2 "frep:SO16" H 2500 1950 60  0001 C CNN
+F 2 "frep:SO-16-L" H 2500 1950 60  0001 C CNN
 F 3 "" H 2500 1950 60  0000 C CNN
 F 4 "296-14858-1-ND" H 2500 1950 60  0001 C CNN "DK"
@@
 F 0 "U3" H 4850 2550 70  0000 C CNN
 F 1 "74HC595" H 4700 1350 70  0000 C CNN
-F 2 "frep:SO16" H 4700 1950 60  0001 C CNN
+F 2 "frep:SO-16-L" H 4700 1950 60  0001 C CNN
 F 3 "" H 4700 1950 60  0000 C CNN
 F 4 "296-14858-1-ND" H 4700 1950 60  0001 C CNN "DK"
