File: projects/PowerBox/PowerBox.kicad_pcb (KiCad board)
At the start: 2 copper layers, 0 parts

Commit message: pcb layout started
Parts:
- added C1: 10uF, frep:C0805, F.Cu at (76.2, 121.9)
- added C10: 10uF, frep:C0805, F.Cu at (219.7, 105.4)
- added C11: 1uF, frep:C0805, F.Cu at (144.8, 151.1)
- added C12: 1uF, frep:C0805, F.Cu at (153.7, 152.4)
- added C13: 100nF, frep:C0805, F.Cu at (157.5, 95.2)
- added C14: 100nF, frep:C0805, F.Cu at (170.2, 95.2)
- added C15: 100nF, frep:C0805, F.Cu at (157.5, 102.9)
- added C16: 100nF, frep:C0805, F.Cu at (135.9, 161.3)
- added C17: 100nF, frep:C0805, F.Cu at (170.2, 102.9)
- added C18: 1uF, frep:C0805, F.Cu at (152.4, 161.3)
- added C2: 10uF, frep:C0805, F.Cu at (113.0, 167.6)
- added C3: 10uF, frep:C0805, F.Cu at (113.0, 154.9)
- added C4: 10uF, frep:C0805, F.Cu at (257.8, 94.0)
- added C5: 18pF, frep:C0805, F.Cu at (153.7, 134.6)
- added C6: 100NF, frep:C0805, F.Cu at (153.7, 141.0)
- added C7: 18pF, frep:C0805, F.Cu at (134.6, 146.1)
- added C8: 100nF, frep:C0805, F.Cu at (219.7, 102.9)
- added C9: 1uF, frep:C0805, F.Cu at (153.7, 147.3)
- added CON1: USB-MICRO, frep:USB_Micro, F.Cu at (68.6, 124.5)
- added CON2: USB-A-Jack, frep:USB-A-Jack, F.Cu at (273.1, 92.7)
- added CON3: USB-MINI-B-Vert, frep:Vertical_USB_Mini_B, F.Cu at (204.5, 100.3)
- added D1: Low Battery, frep:LED-0805, F.Cu at (101.6, 147.3)
- added D10: 5.3V Zener, frep:SOT23, F.Cu at (257.8, 88.9)
- added D11: DL4148, frep:Diode-MiniMELF_Handsoldering, F.Cu at (123.2, 127.0)
- added D12: 5.3V Zener, frep:SOT23, F.Cu at (219.7, 96.5)
- added D13: RX, frep:LED-0805, F.Cu at (213.4, 161.3)
- added D14: TX, frep:LED-0805, F.Cu at (199.4, 162.6)
- added D15: Power, frep:LED-0805, F.Cu at (213.4, 157.5)
- added D16: IO13, frep:LED-0805, F.Cu at (213.4, 153.7)
- added D2: 5.3V Zener, frep:SOT23, F.Cu at (76.2, 127.0)
- added D3: SDM40E20LC, frep:SOT23, F.Cu at (82.5, 125.7)
- added D4: SDM40E20LC, frep:SOT23, F.Cu at (101.6, 158.8)
- added D5: Power Load, frep:LED-0805, F.Cu at (199.4, 153.7)
- added D6: V_bat, frep:LED-0805, F.Cu at (224.8, 49.5)
- added D7: V_load, frep:LED-0805, F.Cu at (224.8, 53.3)
- added D8: i_load, frep:LED-0805, F.Cu at (224.8, 57.1)
- added D9: P_load, frep:LED-0805, F.Cu at (224.8, 61.0)
- added F1: FUSE, frep:C1812, F.Cu at (213.4, 96.5)
- added IC1: LM358, frep:SOIC8, F.Cu at (95.2, 147.3)
- added IC2: LM358, frep:SOIC8, F.Cu at (95.2, 156.2)
- added IC3: LM358, frep:SOIC8, F.Cu at (200.7, 134.6)
- added JP1: JUMPER3, frep:Pin_Proto_Straight_1x03, F.Cu at (190.5, 71.1)
- added JP2: JUMPER, frep:Pin_Proto_Straight_1x02, F.Cu at (257.8, 97.8)
- added JP3: JUMPER, frep:Pin_Proto_Straight_1x02, F.Cu at (163.8, 87.6)
- added JP4: JUMPER, frep:Pin_Proto_Straight_1x02, F.Cu at (275.6, 135.9)
- added JP5: JUMPER, frep:Pin_Proto_Straight_1x02, F.Cu at (104.1, 71.1)
- added L1: Ferrit bead, frep:R0805, F.Cu at (269.2, 154.9)
- added N1: Neopixel, frep:Neopixel, F.Cu at (163.8, 95.2)
- added N2: Neopixel, frep:Neopixel, F.Cu at (176.5, 95.2)
- added N3: Neopixel, frep:Neopixel, F.Cu at (163.8, 102.9)
- added N4: Neopixel, frep:Neopixel, F.Cu at (176.5, 102.9)
- added P1: CONN_2, frep:JST-PH-2-THM, F.Cu at (92.7, 166.4)
- added P10: CONN_4, frep:grove_con_straight, F.Cu at (73.7, 96.5)
- added P11: CONN_10, frep:Pin_Header_Straight_1x10, F.Cu at (88.9, 41.9)
- added P12: CONN_8, frep:Pin_Header_Straight_1x08, F.Cu at (114.3, 41.9)
- added P13: CONN_8, frep:Pin_Header_Straight_1x08, F.Cu at (95.2, 35.6)
- added P14: CONN_6, frep:Pin_Header_Straight_1x06, F.Cu at (116.8, 35.6)
- added P15: CONN_4, frep:grove_con_straight, F.Cu at (73.7, 102.9)
- added P2: CONN_2, frep:JST-PH-2-THM-RA, F.Cu at (104.1, 165.1)
- added P3: CONN_1, frep:MountingHole_3mm, F.Cu at (71.1, 153.7)
- added P4: CONN_1, frep:MountingHole_3mm, F.Cu at (77.5, 160.0)
- added P5: CONN_1, frep:MountingHole_3mm, F.Cu at (77.5, 153.7)
- added P6: CONN_1, frep:MountingHole_3mm, F.Cu at (71.1, 160.0)
- added P7: CONN_3X2, frep:Pin_Proto_Straight_2x03, F.Cu at (153.7, 123.2)
- added P8: CONN_4, frep:grove_con_straight, F.Cu at (73.7, 83.8)
- added P9: CONN_4, frep:grove_con_straight, F.Cu at (73.7, 90.2)
- added PB1: PowerBoost, frep:Powerboost1000C, F.Cu at (106.7, 101.6)
- added Q1: DMG3415U, frep:SOT23, F.Cu at (101.6, 153.7)
- added Q2: DMG3415U, frep:SOT23, F.Cu at (108.0, 153.7)
- added Q3: DMG3415U, frep:SOT23, F.Cu at (166.4, 128.3)
- added Q4: DMG3415U, frep:SOT23, F.Cu at (184.2, 154.9)
- added Q5: DMG3415U, frep:SOT23, F.Cu at (185.4, 161.3)
- added R1: 10K, frep:R0805, F.Cu at (90.2, 154.9)
- added R10: 220R, frep:R0805, F.Cu at (231.1, 61.0)
- added R11: 300R 1%, frep:R0805, F.Cu at (264.2, 87.6)
- added R12: 49.9K 1%, frep:R0805, F.Cu at (264.2, 90.2)
- added R13: 78.7K 1%, frep:R0805, F.Cu at (264.2, 92.7)
- added R14: 43K 1%, frep:R0805, F.Cu at (264.2, 95.2)
- added R15: 49.9K 1%, frep:R0805, F.Cu at (264.2, 97.8)
- added R16: 220R, frep:R0805, F.Cu at (196.8, 44.5)
- added R17: 220R, frep:R0805, F.Cu at (199.4, 44.5)
- added R18: 220R, frep:R0805, F.Cu at (201.9, 44.5)
- added R19: 220R, frep:R0805, F.Cu at (204.5, 44.5)
- added R2: 10K, frep:R0805, F.Cu at (90.2, 148.6)
- added R20: 220R, frep:R0805, F.Cu at (207.0, 44.5)
- added R21: 220R, frep:R0805, F.Cu at (209.6, 44.5)
- added R22: 220R, frep:R0805, F.Cu at (212.1, 44.5)
- added R23: 220R, frep:R0805, F.Cu at (214.6, 44.5)
- added R24: 10K, frep:R0805, F.Cu at (137.2, 62.2)
- added R25: 10K, frep:R0805, F.Cu at (137.2, 66.0)
- added R26: 1M, frep:R0805, F.Cu at (251.5, 156.2)
- added R27: 10K, frep:R0805, F.Cu at (127.0, 127.0)
- added R28: 0.1R 1%, frep:R1206, F.Cu at (147.3, 63.5)
- added R29: 22R, frep:R0805, F.Cu at (241.3, 143.5)
- added R3: 10K, frep:R0805, F.Cu at (190.5, 64.8)
- added R30: 22R, frep:R0805, F.Cu at (251.5, 137.2)
- added R31: 220R, frep:R0805, F.Cu at (243.8, 135.9)
- added R32: 220R, frep:R0805, F.Cu at (251.5, 129.5)
- added R33: 220R, frep:R0805, F.Cu at (232.4, 149.9)
- added R34: 220R, frep:R0805, F.Cu at (259.1, 156.2)
- added R35: 1K, frep:R0805, F.Cu at (260.4, 151.1)
- added R36: 10K, frep:R0805, F.Cu at (104.1, 59.7)
- added R4: 220R, frep:R0805, F.Cu at (101.6, 144.8)
- added R5: 220R, frep:R0805, F.Cu at (233.7, 156.2)
- added R6: 10K, frep:R0805, F.Cu at (226.1, 156.2)
- added R7: 220R, frep:R0805, F.Cu at (231.1, 49.5)
- added R8: 220R, frep:R0805, F.Cu at (231.1, 53.3)
- added R9: 220R, frep:R0805, F.Cu at (231.1, 57.1)
- added S1: Lipo Select, frep:Switch_SPDT, F.Cu at (265.4, 45.7)
- added S2: Load on/off, frep:Switch_SPDT, F.Cu at (270.5, 45.7)
- added S3: Arduino on/off, frep:Switch_SPDT, F.Cu at (275.6, 45.7)
- added S4: Reset, frep:TACTILE-PTH, F.Cu at (115.6, 127.0)
- added S5: Select, frep:TACTILE-PTH, F.Cu at (104.1, 64.8)
- added SEG1: 4_x_7Segment, frep:4digit7segment, F.Cu at (204.5, 55.9)
- added U1: 74HC595, frep:SO16, F.Cu at (214.6, 69.8)
- added U2: ICL7660, frep:SOIC8, F.Cu at (111.8, 161.3)
- added U3: 74HC595, frep:SO16, F.Cu at (200.7, 69.8)
- added U4: INA219, frep:SOIC8, F.Cu at (142.2, 63.5)
- added U5: AP7333, frep:SOT23, F.Cu at (240.0, 118.1)
- added U6: ATMEGA32U4, frep:TQFP44, F.Cu at (171.4, 141.0)
- added VR1: VR, frep:R0805, F.Cu at (213.4, 102.9)
- added VR2: VR, frep:R0805, F.Cu at (213.4, 105.4)
- added X1: 16MHz, frep:HC49UP, F.Cu at (171.4, 153.7)

Commit message: basic part placement
Parts:
- C1, C11, C16, C18, C5, C7, D11, D2, D3, F1, L1, P2, PB1, R10, R11, R12, R13, R14, R15, R16, R17, R18, R19, R20, R21, R22, R23, R26, R27, R3, R31, R32, R33, R34, R35, R36, R5, R7, R8, R9, U1, U3, X1: moved to B.Cu
- P10: value CONN_4 -> Analog
- P15: value CONN_4 -> Digital
- P8: value CONN_4 -> Serial
- P9: value CONN_4 -> I2C
- moved S1 144.3 mm to (137.2, 111.8)
- moved S2 142.0 mm to (144.8, 111.8)
- moved R34 140.7 mm to (142.9, 76.8), turned to 180 degrees
- moved S3 139.8 mm to (152.4, 111.8)
- moved P5 129.5 mm to (180.3, 74.9)
- moved P8 125.8 mm to (199.4, 78.7)
- moved P9 125.8 mm to (199.4, 86.4)
- moved P10 125.8 mm to (199.4, 94.0)
- moved P15 125.7 mm to (199.4, 101.6)
- moved R7 121.2 mm to (113.0, 76.8), turned to 180 degrees
- moved JP4 120.3 mm to (157.5, 113.0), turned to 90 degrees
- moved P6 117.5 mm to (180.3, 116.6)
- moved D6 115.0 mm to (113.0, 76.8)
- moved R35 114.8 mm to (158.8, 97.8), turned to 180 degrees
- moved N2 114.6 mm to (64.8, 69.8), turned to 180 degrees
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Other:
- board outline added: 91.4 x 56.9 mm

Commit message: routing started
Parts:
- D4, IC1, R1, R2, R4: moved to B.Cu
- moved U4 56.1 mm to (90.2, 80.3)
- moved JP4 56.0 mm to (101.6, 109.2)
- moved R28 55.9 mm to (90.4, 84.8)
- moved C2 21.3 mm to (125.5, 100.6), turned to 90 degrees
- moved IC1 19.9 mm to (110.7, 88.9), turned to 180 degrees
- moved C3 19.5 mm to (125.5, 96.5)
- moved U2 17.2 mm to (121.7, 98.6)
- moved R16 16.8 mm to (136.1, 82.3), turned to 0 degrees
- moved C9 16.1 mm to (131.3, 109.0)
- moved S1 16.0 mm to (121.4, 114.8), turned to 180 degrees
- moved R17 14.9 mm to (136.1, 96.5), turned to 0 degrees
- moved IC3 14.5 mm to (133.1, 101.9)
- moved R1 14.5 mm to (115.3, 86.9), turned to 90 degrees
- moved IC2 14.2 mm to (115.3, 98.6), turned to 180 degrees
- moved Q1 14.1 mm to (110.2, 96.3), turned to 180 degrees
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Connections:
- R3 pad 1: V_MP -> VREG_in
- U1 pad 16: V_MP -> VREG_in
- U3 pad 16: V_MP -> VREG_in
Routing:
- net A2: track 0.00 -> 71.8 mm
- net Enable: track 0.00 -> 52.1 mm, vias 0 -> 1
- net En: track 0.00 -> 47.0 mm, vias 0 -> 1
- net V-: track 0.00 -> 40.0 mm, vias 0 -> 2
- net DIG1: track 0.00 -> 39.7 mm
- net V+: track 0.00 -> 37.5 mm, vias 0 -> 1
- net DIG4: track 0.00 -> 31.9 mm, vias 0 -> 1
- net LipoSwitch: track 0.00 -> 26.7 mm, vias 0 -> 1
- net SEGA: track 0.00 -> 25.4 mm
- net DIG2: track 0.00 -> 24.7 mm
- net DIG3: track 0.00 -> 21.5 mm
- net V_BATT: track 0.00 -> 20.7 mm
- net Net-(C1-Pad1): track 0.00 -> 20.6 mm, vias 0 -> 1
- net Net-(R20-Pad1): track 0.00 -> 18.9 mm
- net Net-(R17-Pad1): track 0.00 -> 18.8 mm, vias 0 -> 1
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
Commit message: layout in progress
Parts:
- C10, C8, D12, Q4, R29, R30, VR1, VR2: moved to B.Cu
- C11, C16, C18, C5, C7, L1, R26, R31, R32, R35, X1: moved to F.Cu
- P2: footprint frep:JST-PH-2-THM-RA -> frep:JST-PH-2-THM
- moved R24 70.0 mm to (83.8, 80.0)
- moved R25 70.0 mm to (83.8, 85.1)
- moved D15 63.9 mm to (101.6, 80.0), turned to 0 degrees
- moved R33 63.9 mm to (101.6, 80.0), turned to 0 degrees
- moved D5 59.0 mm to (101.6, 83.8), turned to 0 degrees
- moved R5 59.0 mm to (101.6, 83.8), turned to 0 degrees
- moved D12 47.6 mm to (128.3, 104.4), turned to 90 degrees
- moved C8 44.5 mm to (128.3, 109.2), turned to 180 degrees
- moved C10 41.9 mm to (128.3, 107.2), turned to 180 degrees
- moved CON3 41.4 mm to (124.5, 119.4)
- moved F1 41.0 mm to (128.3, 113.5), turned to 270 degrees
- moved VR1 30.6 mm to (136.1, 112.5)
- moved VR2 25.9 mm to (136.1, 116.3), turned to 270 degrees
- moved R30 23.7 mm to (139.4, 113.3), turned to 180 degrees
- moved R6 19.9 mm to (133.3, 98.6), turned to 90 degrees
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Routing:
- net /Arduino/Vin+: track 0.00 -> 124.8 mm
- net DIG1: track 39.7 -> 0.00 mm
- net Net-(D4-Pad1): track 4.59 -> 41.3 mm
- net DIG4: track 31.9 -> 0.00 mm, vias 1 -> 0
- net GND: track 7.77 -> 36.0 mm
- net SEGA: track 25.4 -> 0.00 mm
- net DIG2: track 24.7 -> 0.00 mm
- net Enable: track 52.1 -> 28.3 mm, vias 1 -> 0
- net DIG3: track 21.5 -> 0.00 mm
- net /Arduino/VCC: track 0.00 -> 19.5 mm
- net Net-(R20-Pad1): track 18.9 -> 0.00 mm
- net Net-(R17-Pad1): track 18.8 -> 0.00 mm, vias 1 -> 0
- net Net-(R21-Pad1): track 18.5 -> 0.00 mm, vias 1 -> 0
- net V_MP: track 0.00 -> 17.8 mm, vias 0 -> 1
- net En: track 47.0 -> 29.5 mm, vias 1 -> 0
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
Commit message: layout in progress
Parts:
- removed P10: Analog, frep:grove_con_straight
- removed P15: Digital, frep:grove_con_straight
- removed P8: Serial, frep:grove_con_straight
- removed P9: I2C, frep:grove_con_straight
- C16: moved to B.Cu
- JP2: value JUMPER -> + -
- moved R32 37.3 mm to (151.8, 81.3)
- moved D13 37.3 mm to (144.8, 81.3)
- moved D14 37.3 mm to (148.6, 81.3)
- moved R31 37.3 mm to (142.2, 81.3)
- moved L1 14.8 mm to (170.2, 111.3)
- moved C18 14.8 mm to (172.2, 111.3)
- moved C6 7.40 mm to (156.5, 112.0), turned to 270 degrees
- moved R35 6.71 mm to (153.4, 112.0), turned to 90 degrees
- moved C16 6.16 mm to (164.1, 114.0)
- moved C7 5.78 mm to (157.2, 95.2)
- moved R26 5.78 mm to (162.9, 95.2)
- moved X1 5.78 mm to (162.9, 90.8)
- moved C5 5.78 mm to (168.7, 95.2), turned to 0 degrees
- moved U6 5.72 mm to (162.6, 104.8)
- moved C11 4.89 mm to (172.2, 105.8)
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Connections:
- net D5 renamed Data
- net D6 renamed Clock
- net D7 renamed Latch
Routing:
- net VREG_in: track 11.3 -> 58.5 mm, vias 2 -> 5
- net RESET: track 0.00 -> 30.1 mm
- net MOSI: track 0.00 -> 27.4 mm
- net SCK: track 0.00 -> 26.1 mm
- net MISO: track 0.00 -> 22.4 mm
- net GND: track 36.0 -> 55.7 mm, vias 3 -> 6
- net A5: track 0.00 -> 16.2 mm
- net A4: track 0.00 -> 14.4 mm
- net Net-(JP5-Pad2): track 0.00 -> 14.1 mm
- net A3: track 0.00 -> 12.4 mm
- net XTAL1: track 0.00 -> 12.3 mm
- net XTAL2: track 0.00 -> 12.3 mm
- net A2: track 68.8 -> 79.2 mm
- net A0: track 0.00 -> 9.88 mm
- net A1: track 0.00 -> 9.64 mm
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
Commit message: layout in progress
Parts:
- C4, C5, C7, D10, R26, R31, R32: moved to B.Cu
- D15: value Power -> Power Ard.
- moved R32 6.07 mm to (148.1, 76.5), turned to 90 degrees
- moved D11 5.47 mm to (173.2, 80.0)
- moved R31 5.34 mm to (144.5, 76.5), turned to 90 degrees
- moved D14 4.85 mm to (148.1, 76.5)
- moved D13 4.83 mm to (144.5, 76.5)
- moved C11 3.81 mm to (172.2, 102.0)
- moved C16 3.81 mm to (164.1, 110.2)
- moved C18 3.81 mm to (172.2, 107.4)
- moved C5 3.81 mm to (168.7, 91.4)
- moved C6 3.81 mm to (156.5, 108.2)
- moved C7 3.81 mm to (157.2, 91.4)
- moved L1 3.81 mm to (170.2, 107.4)
- moved R26 3.81 mm to (162.9, 91.4)
- moved R35 3.81 mm to (153.4, 108.2)
- moved U6 3.81 mm to (162.6, 101.0)
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Connections:
- net Clock renamed D6
- net Data renamed D5
- JP3 pad 1: IO_10 -> Latch
- P11 pad 3: IO_10 -> Latch
- P12 pad 8: Latch -> D7
- U6 pad 1: Latch -> D7
- U6 pad 30: IO_10 -> Latch
Routing:
- net D0/RX: track 0.00 -> 30.6 mm, vias 0 -> 1
- net D1/TX: track 0.00 -> 28.7 mm, vias 0 -> 1
- net D3/SCL: track 0.00 -> 28.5 mm, vias 0 -> 2
- net D2/SDA: track 0.00 -> 27.6 mm, vias 0 -> 2
- net IO_11: track 0.00 -> 27.2 mm, vias 0 -> 2
- net MOSI: track 27.4 -> 0.25 mm
- net SCK: track 26.1 -> 0.00 mm
- net IO_12: track 0.00 -> 22.7 mm, vias 0 -> 2
- net MISO: track 22.4 -> 0.00 mm
- net D7: track 0.00 -> 21.5 mm, vias 0 -> 2
- net RESET: track 30.1 -> 11.7 mm, vias 0 -> 1
- net Net-(C4-Pad1): track 8.99 -> 27.2 mm
- net A5: track 16.2 -> 0.00 mm
- net IO_13: track 0.00 -> 14.9 mm
- net A4: track 14.4 -> 0.00 mm
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
Commit message: layout in progress
Parts:
- moved JP5 22.6 mm to (174.5, 75.4)
- moved D11 3.56 mm to (173.2, 83.6)
- moved U1 2.29 mm to (146.6, 101.1)
- moved U3 1.02 mm to (146.6, 88.1)
- moved P7 0.51 mm to (179.1, 82.0)
Connections:
- JP3 pad 1: Latch -> IO_10
- P11 pad 3: Latch -> IO_10
- P11 pad 4: IO_11 -> Latch
- U1 pad 11: D6 -> D7
- U1 pad 14: D5 -> IO_12
- U3 pad 11: D6 -> D7
- U6 pad 12: IO_11 -> Latch
- U6 pad 30: Latch -> IO_10
Routing:
- net D4: track 2.78 -> 50.7 mm
- net D5: track 10.8 -> 40.5 mm
- net D6: track 5.56 -> 35.1 mm
- net IO_11: track 27.2 -> 0.00 mm, vias 2 -> 0
- net D7: track 21.5 -> 48.2 mm
- net Net-(JP5-Pad2): track 0.00 -> 24.5 mm, vias 0 -> 1
- net IO_13: track 14.9 -> 5.62 mm
- net IO_12: track 22.7 -> 13.5 mm
- net VREG_in: track 65.2 -> 57.7 mm
- net Latch: track 10.6 -> 17.8 mm, vias 0 -> 2
- net IO_10: track 0.00 -> 6.58 mm
- net IO_9: track 9.40 -> 5.59 mm
- net (no net): track 0.98 -> 3.22 mm
- net RESET: track 11.7 -> 10.3 mm

Commit message: pcb layout in progress
Parts:
- moved R24 77.1 mm to (152.8, 114.6), turned to 270 degrees
- moved R25 72.8 mm to (150.4, 114.7)
- moved U4 63.2 mm to (146.1, 109.7)
- moved R28 61.4 mm to (144.3, 114.3)
- moved VR2 37.2 mm to (173.2, 113.3), turned to 0 degrees
- moved R29 33.2 mm to (172.2, 110.2), turned to 90 degrees
- moved VR1 33.0 mm to (169.2, 113.3), turned to 180 degrees
- moved R30 30.9 mm to (170.2, 110.2), turned to 270 degrees
- moved C11 1.91 mm to (172.2, 100.1), turned to 90 degrees
- moved U3 1.02 mm to (146.6, 87.1)
- moved S1 0.51 mm to (116.8, 109.7)
- moved S2 0.51 mm to (124.5, 109.7)
- moved S3 0.51 mm to (132.1, 109.7)
- turned D16 to 90 degrees
- turned R34 to 90 degrees
Routing:
- net RESET: track 10.3 -> 109.3 mm, vias 1 -> 2
- net /Arduino/Vin+: track 124.8 -> 45.8 mm, vias 0 -> 2
- net AREF: track 4.75 -> 71.4 mm, vias 1 -> 2
- net VREG_in: track 57.7 -> 111.4 mm
- net Net-(CON3-Pad2): track 0.00 -> 53.4 mm, vias 0 -> 1
- net Latch: track 17.8 -> 64.7 mm
- net IO_12: track 13.5 -> 59.5 mm
- net Net-(CON3-Pad3): track 7.25 -> 51.4 mm, vias 0 -> 1
- net IO_13: track 5.62 -> 48.1 mm, vias 0 -> 1
- net 3V3: track 0.00 -> 37.2 mm
- net IO_10: track 6.58 -> 39.8 mm
- net IO_9: track 5.59 -> 37.8 mm
- net GND: track 47.5 -> 74.7 mm, vias 10 -> 22
- net IO_8: track 8.22 -> 35.1 mm
- net MOSI: track 0.00 -> 22.0 mm
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