File: projects/Sepic/Sepic.sch (KiCad schematic (older format))
At the start: 1 part

Commit message: sepic schematic first draw
Parts:
- added C?: CP1, symbol CP1
- added C? (x4): C, symbol C
- added D?: DIODESCH, symbol DIODESCH
- added L? (x2): InductorsCoupled, symbol InductorsCoupled
- added P? (x7): CONN_1, symbol CONN_1
- added P? (x2): CONN_2, symbol CONN_2
- added R? (x3): R, symbol R
Connections:
- net labels added: GND
- wire segments 0 -> 27
- no-connect marks 0 -> 1

Commit message: schematic finished
Parts:
- added JP1: JUMPER, symbol JUMPER
- gave numbers to parts that had none: 20
Connections:
- wire segments 27 -> 30
Other:
- moved on the sheet: C1, P1, P2, P3, P4

Commit message: working on sepic
Parts:
- C2: value C -> 470nF
- C3: value C -> 4n7F
- D1: value DIODESCH -> V8PAN50-M3; footprint (none) -> frep:DO-221BC
- JP1: footprint (none) -> bytelabs:S_JUMPER_2
- L1: footprint (none) -> frep:InductorsCoupled
- P1: value CONN_1 -> V_in+; footprint (none) -> frep:Pin_Proto_Straight_1x01
- P2: value CONN_1 -> V_in-; footprint (none) -> frep:Pin_Proto_Straight_1x01
- P3: value CONN_2 -> JST_In; footprint (none) -> frep:JST-PH-2-THM
- P4: value CONN_1 -> En; footprint (none) -> frep:Pin_Proto_Straight_1x01
- P5: value CONN_1 -> R+; footprint (none) -> frep:Pin_Proto_Straight_1x01
- P6: value CONN_1 -> R-; footprint (none) -> frep:Pin_Proto_Straight_1x01
- P7: value CONN_2 -> JST_Out; footprint (none) -> frep:JST-PH-2-THM
- P8: value CONN_1 -> V_out+; footprint (none) -> frep:Pin_Proto_Straight_1x01
- P9: value CONN_1 -> V_out-; footprint (none) -> frep:Pin_Proto_Straight_1x01
- R1: value R -> 2K; footprint (none) -> frep:R0805
- R2, R3: footprint (none) -> frep:R0805
- U1: footprint (none) -> frep:TO-263-7
Connections:
- net GND: now also U1.4 (GND), U1.8 (pad)
Other:
- note added: "Dmax = (Vout,max + Vd) / (Vin,min + Vout,max + Vd)\nPout,max = Vout,max*Iout,max\nPin,max=Pout,max/eff (eff about 0.85)\nIin,max=Pin,max/Vin,min"
- note added: "Enable signal (S/S) \nfrom input with \nsolder jumper or \nexternal from P4"
- note added: "R2 can be \nreplaced by \nan external \nresistor or \n(dig.) pot."
- note added: "Vd"
- moved on the sheet: C5, P5, P6, P7, P8, P9

Commit message: still working on sepic
Parts:
- removed C5: C, symbol C
- removed P5: R+, frep:Pin_Proto_Straight_1x01, symbol CONN_1
- removed P6: R-, frep:Pin_Proto_Straight_1x01, symbol CONN_1
- added C5: 100uF, symbol CP1
- added RV1: POT, frep:Trimmer, symbol POT
- C1: value CP1 -> 100uF; DK (none) -> 493-13627-1-ND
- C2: footprint (none) -> frep:C0805; DK (none) -> 445-2276-1-ND
- C3: footprint (none) -> frep:C0805
- C4: value C -> 4u7F; footprint (none) -> frep:R1206; DK (none) -> 478-8718-1-ND
- D1: DK (none) -> V8PAN50-M3/ICT-ND
- L1: value InductorsCoupled -> 22uH; DK (none) -> SRF1280-220MCT-ND
- L1: value InductorsCoupled -> 22uH
- P3, P7: DK (none) -> 455-1704-ND
- R1: DK (none) -> P2.00KCCT-ND
- R3: value R -> 1K
- U1: DK (none) -> LT1370HVCR#PBF-ND
Connections:
- net GND: now also C5.2
- net at C4.2, L1.1, P7.2 (PM)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: now also C5.1
- net at D1.2 (K), R2.1: now also RV1.1
- net at R2.2, R3.1, U1.2 (FB+): now also RV1.2
- no-connect marks 1 -> 2
Other:
- note removed: "Dmax = (Vout,max + Vd) / (Vin,min + Vout,max + Vd)\nPout,max = Vout,max*Iout,max\nPin,max=Pout,max/eff (eff about 0.85)\nIin,max=Pin,max/Vin,min"
Changed lines of the file:
@@
 P 3400 2900
 F 0 "C1" H 3450 3000 50  0000 L CNN
-F 1 "CP1" H 3450 2800 50  0000 L CNN
+F 1 "100uF" H 3450 2800 50  0000 L CNN
 F 2 "" H 3400 2900 60  0001 C CNN
 F 3 "" H 3400 2900 60  0000 C CNN
+F 4 "493-13627-1-ND" H 3400 2900 60  0001 C CNN "DK"
 	1    3400 2900
 	1    0    0    -1
@@
 F 0 "C2" H 5550 4400 40  0000 L CNN
 F 1 "470nF" H 5556 4215 40  0000 L CNN
-F 2 "" H 5588 4150 30  0001 C CNN
+F 2 "frep:C0805" H 5588 4150 30  0001 C CNN
 F 3 "" H 5550 4300 60  0000 C CNN
+F 4 "445-2276-1-ND" H 5550 4300 60  0001 C CNN "DK"
 	1    5550 4300
 	1    0    0    -1
@@
 P 6500 2650
 F 0 "C4" H 6500 2750 40  0000 L CNN
-F 1 "C" H 6506 2565 40  0000 L CNN
-F 2 "" H 6538 2500 30  0001 C CNN
+F 1 "4u7F" H 6506 2565 40  0000 L CNN
+F 2 "frep:R1206" H 6538 2500 30  0001 C CNN
 F 3 "" H 6500 2650 60  0000 C CNN
+F 4 "478-8718-1-ND" H 6500 2650 60  0001 C CNN "DK"
 	1    6500 2650
 	0    1    1    0
-$EndComp
-$Comp
-L C C5
-U 1 1 55E5C1B0
-P 8300 2900
-F 0 "C5" H 8300 3000 40  0000 L CNN
-F 1 "C" H 8306 2815 40  0000 L CNN
-F 2 "" H 8338 2750 30  0001 C CNN
-F 3 "" H 8300 2900 60  0000 C CNN
-	1    8300 2900
-	1    0    0    -1
 $EndComp
 $Comp
@@
 F 0 "C3" H 5900 4400 40  0000 L CNN
 F 1 "4n7F" H 5906 4215 40  0000 L CNN
-F 2 "" H 5938 4150 30  0001 C CNN
+F 2 "frep:C0805" H 5938 4150 30  0001 C CNN
 F 3 "" H 5900 4300 60  0000 C CNN
 	1    5900 4300
@@
 F 2 "frep:R0805" V 5480 3850 30  0001 C CNN
 F 3 "" H 5550 3850 30  0000 C CNN
+F 4 "P2.00KCCT-ND" V 5550 3850 60  0001 C CNN "DK"
 	1    5550 3850
 	1    0    0    -1
@@
 P 7250 3400
 F 0 "R3" V 7330 3400 40  0000 C CNN
-F 1 "R" V 7257 3401 40  0000 C CNN
+F 1 "1K" V 7257 3401 40  0000 C CNN
 F 2 "frep:R0805" V 7180 3400 30  0001 C CNN
 F 3 "" H 7250 3400 30  0000 C CNN
@@
 F 2 "frep:DO-221BC" H 7000 2650 60  0001 C CNN
 F 3 "" H 7000 2650 60  0000 C CNN
+F 4 "V8PAN50-M3/ICT-ND" H 7000 2650 60  0001 C CNN "DK"
 	1    7000 2650
 	1    0    0    1
@@
 F 2 "frep:JST-PH-2-THM" H 2750 2900 60  0001 C CNN
 F 3 "" H 2750 2900 60  0000 C CNN
+F 4 "455-1704-ND" V 2750 2900 60  0001 C CNN "DK"
 	1    2750 2900
 	-1   0    0    1
@@
 F 2 "frep:JST-PH-2-THM" H 8950 2900 60  0001 C CNN
 F 3 "" H 8950 2900 60  0000 C CNN
+F 4 "455-1704-ND" V 8950 2900 60  0001 C CNN "DK"
 	1    8950 2900
 	1    0    0    1
@@
 P 5900 2050
 F 0 "L1" H 5900 1950 60  0000 C CNN
-F 1 "InductorsCoupled" H 5900 2250 60  0000 C CNN
+F 1 "22uH" H 5900 2250 60  0000 C CNN
 F 2 "frep:InductorsCoupled" H 5900 2050 60  0001 C CNN
 F 3 "" H 5900 2050 60  0000 C CNN
+F 4 "SRF1280-220MCT-ND" H 5900 2050 60  0001 C CNN "DK"
 	1    5900 2050
 	1    0    0    -1
@@
 P 6750 3700
 F 0 "L1" H 6750 3600 60  0000 C CNN
-F 1 "InductorsCoupled" H 6750 3900 60  0000 C CNN
+F 1 "22uH" H 6750 3900 60  0000 C CNN
 F 2 "frep:InductorsCoupled" H 6750 3700 60  0001 C CNN
 F 3 "" H 6750 3700 60  0000 C CNN
@@
 	5050 3600 5050 4500
 Wire Wire Line
-	6300 3150 7400 3150
+	6300 3150 7550 3150
 Connection ~ 7250 3150
 Wire Wire Line
-	7200 2650 7400 2650
+	7200 2650 7700 2650
 Wire Wire Line
 	6700 2650 6800 2650
@@
 Connection ~ 8300 2050
 $Comp
-L CONN_1 P5
-U 1 1 55E87807
-P 7550 2650
-F 0 "P5" H 7630 2650 40  0000 L CNN
-F 1 "R+" H 7550 2550 60  0000 C CNN
-F 2 "frep:Pin_Proto_Straight_1x01" H 7550 2650 60  0001 C CNN
-F 3 "" H 7550 2650 60  0000 C CNN
-	1    7550 2650
-	1    0    0    -1
-$EndComp
-$Comp
-L CONN_1 P6
-U 1 1 55E87861
-P 7550 3150
-F 0 "P6" H 7630 3150 40  0000 L CNN
-F 1 "R-" H 7550 3250 60  0000 C CNN
-F 2 "frep:Pin_Proto_Straight_1x01" H 7550 3150 60  0001 C CNN
-F 3 "" H 7550 3150 60  0000 C CNN
-	1    7550 3150
-	1    0    0    -1
-$EndComp
-$Comp
 L JUMPER JP1
 U 1 1 55E94E7E
@@
 Wire Notes Line
 	3750 2200 4250 2200
-Text Notes 3700 3850 0    60   ~ 0
+Text Notes 3600 3850 0    60   ~ 0
 Enable signal (S/S) \nfrom input with \nsolder jumper or \nexternal from P4
-Wire Notes Line
-	7450 2500 7450 3300
-Wire Notes Line
-	7450 3300 7800 3300
-Wire Notes Line
-	7800 3300 7800 2500
-Wire Notes Line
-	7800 2500 7450 2500
-Text Notes 7500 3850 0    60   ~ 0
+Text Notes 7500 4050 0    60   ~ 0
 R2 can be \nreplaced by \nan external \nresistor or \n(dig.) pot.
-Text Notes 2250 5150 0    60   ~ 0
-Dmax = (Vout,max + Vd) / (Vin,min + Vout,max + Vd)\nPout,max = Vout,max*Iout,max\nPin,max=Pout,max/eff  (eff about 0.85)\nIin,max=Pin,max/Vin,min
 $Comp
 L LT1370 U1
@@
 F 2 "frep:TO-263-7" H 5300 2900 60  0001 C CNN
 F 3 "" H 5300 2900 60  0000 C CNN
+F 4 "LT1370HVCR#PBF-ND" H 5300 2900 60  0001 C CNN "DK"
 	1    5300 2900
 	1    0    0    -1
@@
 Wire Wire Line
 	5300 3600 5300 4500
+$Comp
+L POT RV1
+U 1 1 55EA1D69
+P 7700 3150
+F 0 "RV1" H 7700 3050 50  0000 C CNN
+F 1 "POT" H 7700 3150 50  0000 C CNN
+F 2 "frep:Trimmer" H 7700 3150 60  0001 C CNN
+F 3 "" H 7700 3150 60  0000 C CNN
+	1    7700 3150
+	0    -1   1    0
+$EndComp
+NoConn ~ 7700 3400
+Wire Wire Line
+	7700 2650 7700 2900
+Wire Notes Line
+	7500 2600 7500 3550
+Wire Notes Line
+	7500 3550 7950 3550
+Wire Notes Line
+	7950 3550 7950 2600
+Wire Notes Line
+	7950 2600 7500 2600
+$Comp
+L CP1 C5
+U 1 1 55EA3021
+P 8300 2900
+F 0 "C5" H 8350 3000 50  0000 L CNN
+F 1 "100uF" H 8350 2800 50  0000 L CNN
+F 2 "" H 8300 2900 60  0001 C CNN
+F 3 "" H 8300 2900 60  0000 C CNN
+F 4 "493-13627-1-ND" H 8300 2900 60  0001 C CNN "DK"
+	1    8300 2900
+	1    0    0    -1
+$EndComp
 $EndSCHEMATC

Commit message: layout started
Parts:
- added P10: V_out+, frep:Pin_Proto_Straight_1x01, symbol CONN_1
- added P11: V_out-, frep:Pin_Proto_Straight_1x01, symbol CONN_1
- added P5: V_in+, frep:Pin_Proto_Straight_1x01, symbol CONN_1
- added P6: V_in-, frep:Pin_Proto_Straight_1x01, symbol CONN_1
- added R4, R5: 0R, frep:R1206, symbol R
- C1, C5: footprint (none) -> frep:Cap_Nichicon
- P2: value V_in- -> GND
- P9: value V_out- -> GND
- R3: value 1K -> 10K; DK (none) -> P10.0KCCT-ND
- renumbered RV1 to 500K1
Connections:
- net at C1.1, P1.1, P3.2 (PM): now also P5.1, R4.1; no longer JP1.2, L1.3, U1.7 (Vin)
- net at C4.2, L1.1, U1.5 (Vsw): now also P10.1, R5.1; no longer C5.1, P7.2 (PM), P8.1
- new net: C5.1, P11.1, P7.2 (PM), P8.1, R5.2
- new net: JP1.2, L1.3, P6.1, R4.2, U1.7 (Vin)
Other:
- note added: "Replace 0R\nresistor with\nshunt resistor\nfor external\npower meas."
- moved on the sheet: 500K1, C1, C2, C3, C4, C5, D1, JP1, L1A, L1B, P1, P2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

Commit message: working on sepic
Parts:
- removed P7: JST_Out, frep:JST-PH-2-THM, symbol CONN_2
- added P12, P13, P14, P15, P16, P7: NC, frep:Pin_Proto_Straight_1x01, symbol CONN_1
- P3: footprint frep:JST-PH-2-THM -> frep:JST-PH-2-THM-RA
Connections:
- net at C4.2, L1.1, P10.1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: now also C5.1
- net at P11.1, P8.1, R5.2: no longer C5.1
- no-connect marks 2 -> 8
Other:
- moved on the sheet: P10, P11, P8, P9, R5
Changed lines of the file:
@@
 F 0 "P3" V 2400 3600 40  0000 C CNN
 F 1 "JST_In" V 2500 3600 40  0000 C CNN
-F 2 "frep:JST-PH-2-THM" H 2450 3600 60  0001 C CNN
+F 2 "frep:JST-PH-2-THM-RA" H 2450 3600 60  0001 C CNN
 F 3 "" H 2450 3600 60  0000 C CNN
 F 4 "455-1704-ND" V 2450 3600 60  0001 C CNN "DK"
 	1    2450 3600
 	-1   0    0    1
-$EndComp
-$Comp
-L CONN_2 P7
-U 1 1 55E5C5EC
-P 8950 3600
-F 0 "P7" V 8900 3600 40  0000 C CNN
-F 1 "JST_Out" V 9000 3600 40  0000 C CNN
-F 2 "frep:JST-PH-2-THM" H 8950 3600 60  0001 C CNN
-F 3 "" H 8950 3600 60  0000 C CNN
-F 4 "455-1704-ND" V 8950 3600 60  0001 C CNN "DK"
-	1    8950 3600
-	1    0    0    1
 $EndComp
 $Comp
@@
 Wire Wire Line
 	8300 3800 8300 5200
-Wire Wire Line
-	8600 3500 8600 3350
-Wire Wire Line
-	8600 3350 8300 3350
-Connection ~ 8300 3350
-Wire Wire Line
-	8600 3700 8600 3850
-Wire Wire Line
-	8600 3850 8300 3850
-Connection ~ 8300 3850
 $Comp
 L CONN_1 P8
 U 1 1 55E875C6
-P 9050 2750
-F 0 "P8" H 9130 2750 40  0000 L CNN
-F 1 "V_out+" H 9050 2650 60  0000 C CNN
-F 2 "frep:Pin_Proto_Straight_1x01" H 9050 2750 60  0001 C CNN
-F 3 "" H 9050 2750 60  0000 C CNN
-	1    9050 2750
+P 9450 2750
+F 0 "P8" H 9530 2750 40  0000 L CNN
+F 1 "V_out+" H 9450 2650 60  0000 C CNN
+F 2 "frep:Pin_Proto_Straight_1x01" H 9450 2750 60  0001 C CNN
+F 3 "" H 9450 2750 60  0000 C CNN
+	1    9450 2750
 	1    0    0    -1
 $EndComp
@@
 L CONN_1 P9
 U 1 1 55E87638
-P 9050 5000
-F 0 "P9" H 9130 5000 40  0000 L CNN
-F 1 "GND" H 9050 4900 60  0000 C CNN
-F 2 "frep:Pin_Proto_Straight_1x01" H 9050 5000 60  0001 C CNN
-F 3 "" H 9050 5000 60  0000 C CNN
-	1    9050 5000
-	1    0    0    -1
-$EndComp
-Wire Wire Line
-	8900 5000 8300 5000
+P 9450 5000
+F 0 "P9" H 9530 5000 40  0000 L CNN
+F 1 "GND" H 9450 4900 60  0000 C CNN
+F 2 "frep:Pin_Proto_Straight_1x01" H 9450 5000 60  0001 C CNN
+F 3 "" H 9450 5000 60  0000 C CNN
+	1    9450 5000
+	1    0    0    -1
+$EndComp
 Connection ~ 8300 5000
 Connection ~ 8300 2750
@@
 L R R5
 U 1 1 55EAD0BA
-P 7150 2750
-F 0 "R5" V 7230 2750 40  0000 C CNN
-F 1 "0R" V 7157 2751 40  0000 C CNN
-F 2 "frep:R1206" V 7080 2750 30  0001 C CNN
-F 3 "" H 7150 2750 30  0000 C CNN
-F 4 "541-0.0UBCT-ND" V 7150 2750 60  0001 C CNN "DK"
-	1    7150 2750
+P 8750 2750
+F 0 "R5" V 8830 2750 40  0000 C CNN
+F 1 "0R" V 8757 2751 40  0000 C CNN
+F 2 "frep:R1206" V 8680 2750 30  0001 C CNN
+F 3 "" H 8750 2750 30  0000 C CNN
+F 4 "541-0.0UBCT-ND" V 8750 2750 60  0001 C CNN "DK"
+	1    8750 2750
 	0    -1   -1   0
 $EndComp
@@
 L CONN_1 P10
 U 1 1 55EAD60A
-P 6900 2600
-F 0 "P10" H 6980 2600 40  0000 L CNN
-F 1 "V_out+" H 7000 2700 60  0000 C CNN
-F 2 "frep:Pin_Proto_Straight_1x01" H 6900 2600 60  0001 C CNN
-F 3 "" H 6900 2600 60  0000 C CNN
-	1    6900 2600
+P 8500 2600
+F 0 "P10" H 8580 2600 40  0000 L CNN
+F 1 "V_out+" H 8600 2700 60  0000 C CNN
+F 2 "frep:Pin_Proto_Straight_1x01" H 8500 2600 60  0001 C CNN
+F 3 "" H 8500 2600 60  0000 C CNN
+	1    8500 2600
 	0    -1   -1   0
 $EndComp
@@
 L CONN_1 P11
 U 1 1 55EAD688
-P 7400 2600
-F 0 "P11" H 7480 2600 40  0000 L CNN
-F 1 "V_out-" H 7500 2500 60  0000 C CNN
-F 2 "frep:Pin_Proto_Straight_1x01" H 7400 2600 60  0001 C CNN
-F 3 "" H 7400 2600 60  0000 C CNN
-	1    7400 2600
-	0    -1   -1   0
-$EndComp
-Wire Wire Line
-	6900 2750 6300 2750
-Wire Wire Line
-	7400 2750 8900 2750
+P 9000 2600
+F 0 "P11" H 9080 2600 40  0000 L CNN
+F 1 "V_out-" H 9100 2500 60  0000 C CNN
+F 2 "frep:Pin_Proto_Straight_1x01" H 9000 2600 60  0001 C CNN
+F 3 "" H 9000 2600 60  0000 C CNN
+	1    9000 2600
+	0    -1   -1   0
+$EndComp
 Connection ~ 3300 2750
 Connection ~ 3800 2750
-Connection ~ 6900 2750
-Connection ~ 7400 2750
+Connection ~ 8500 2750
+Connection ~ 9000 2750
 Wire Notes Line
 	3150 2300 3150 2850
@@
 Text Notes 3250 2250 0    60   ~ 0
 Replace 0R\nresistor with\nshunt resistor\nfor external\npower meas.
-Text Notes 6850 2250 0    60   ~ 0
+Text Notes 8450 2250 0    60   ~ 0
 Replace 0R\nresistor with\nshunt resistor\nfor external\npower meas.
 Wire Notes Line
-	6700 2300 6700 2850
-Wire Notes Line
-	6700 2850 7600 2850
-Wire Notes Line
-	7600 2850 7600 2300
-Wire Notes Line
-	7600 2300 6700 2300
+	8300 2300 8300 2850
+Wire Notes Line
+	8300 2850 9200 2850
+Wire Notes Line
+	9200 2850 9200 2300
+Wire Notes Line
+	9200 2300 8300 2300
+$Comp
+L CONN_1 P13
+U 1 1 55EC9B0A
+P 5000 2150
+F 0 "P13" H 5080 2150 40  0000 L CNN
+F 1 "NC" H 5000 2250 60  0000 C CNN
+F 2 "frep:Pin_Proto_Straight_1x01" H 5000 2150 60  0001 C CNN
+F 3 "" H 5000 2150 60  0000 C CNN
+	1    5000 2150
+	0    -1   -1   0
+$EndComp
+$Comp
+L CONN_1 P14
+U 1 1 55EC9B9E
+P 5200 2150
+F 0 "P14" H 5280 2150 40  0000 L CNN
+F 1 "NC" H 5200 2250 60  0000 C CNN
+F 2 "frep:Pin_Proto_Straight_1x01" H 5200 2150 60  0001 C CNN
+F 3 "" H 5200 2150 60  0000 C CNN
+	1    5200 2150
+	0    -1   -1   0
+$EndComp
+$Comp
+L CONN_1 P15
+U 1 1 55EC9C0F
+P 5400 2150
+F 0 "P15" H 5480 2150 40  0000 L CNN
+F 1 "NC" H 5400 2250 60  0000 C CNN
+F 2 "frep:Pin_Proto_Straight_1x01" H 5400 2150 60  0001 C CNN
+F 3 "" H 5400 2150 60  0000 C CNN
+	1    5400 2150
+	0    -1   -1   0
+$EndComp
+$Comp
+L CONN_1 P16
+U 1 1 55EC9C81
+P 5600 2150
+F 0 "P16" H 5680 2150 40  0000 L CNN
+F 1 "NC" H 5600 2250 60  0000 C CNN
+F 2 "frep:Pin_Proto_Straight_1x01" H 5600 2150 60  0001 C CNN
+F 3 "" H 5600 2150 60  0000 C CNN
+	1    5600 2150
+	0    -1   -1   0
+$EndComp
+NoConn ~ 5000 2300
+NoConn ~ 5200 2300
+NoConn ~ 5400 2300
+NoConn ~ 5600 2300
+Wire Wire Line
+	8300 5000 9300 5000
+$Comp
+L CONN_1 P7
+U 1 1 55EF15C1
+P 4800 2150
+F 0 "P7" H 4880 2150 40  0000 L CNN
+F 1 "NC" H 4800 2250 60  0000 C CNN
+F 2 "frep:Pin_Proto_Straight_1x01" H 4800 2150 60  0001 C CNN
+F 3 "" H 4800 2150 60  0000 C CNN
+	1    4800 2150
+	0    -1   -1   0
+$EndComp
+$Comp
+L CONN_1 P12
+U 1 1 55EF1630
+P 5800 2150
+F 0 "P12" H 5880 2150 40  0000 L CNN
+F 1 "NC" H 5800 2250 60  0000 C CNN
+F 2 "frep:Pin_Proto_Straight_1x01" H 5800 2150 60  0001 C CNN
+F 3 "" H 5800 2150 60  0000 C CNN
+	1    5800 2150
+	0    -1   -1   0
+$EndComp
+NoConn ~ 5800 2300
+NoConn ~ 4800 2300
+Wire Wire Line
+	9300 2750 9000 2750
+Wire Wire Line
+	6300 2750 8500 2750
 $EndSCHEMATC

Commit message: working on sepic
Parts:
- removed JP1: JUMPER, bytelabs:S_JUMPER_2, symbol JUMPER
- removed R4, R5: 0R, frep:R1206, symbol R
- added 500K2: POT, frep:Trimmer, symbol POT
- added CON1: USB-MICRO-LOAD, frep:USB_Micro_Load, symbol USB-MICRO-LOAD
- added JP1, JP2: JUMPER3, frep:Pin_Proto_Straight_1x03, symbol JUMPER3
- added P17, P24, P25, P28, P29: GND, frep:Pin_Proto_Straight_1x01, symbol CONN_1
- added P18: V_in+, frep:Pin_Proto_Straight_1x01, symbol CONN_1
- added P19: V_in-, frep:Pin_Proto_Straight_1x01, symbol CONN_1
- added P20, P22, P23, P26, P27: V_out+, frep:Pin_Proto_Straight_1x01, symbol CONN_1
- added P21: V_out-, frep:Pin_Proto_Straight_1x01, symbol CONN_1
- added P30, P31: CONN_3X2, frep:Pin_Proto_Straight_2x03, symbol CONN_3X2
- added P32, P33: CONN_2, frep:Pin_Proto_Straight_1x02, symbol CONN_2
- P1, P8, P9: footprint frep:Pin_Proto_Straight_1x01 -> frep:SMD_SOLDERPOINT
- P12, P13: value NC -> GND
- P14: value NC -> GND; footprint frep:Pin_Proto_Straight_1x01 -> frep:SMD_SOLDERPOINT
- P15, P16, P7: value NC -> V_in+
- P4: value En -> V_in+
Connections:
- net GND: now also P12.1, P13.1, P14.1, CON1.2 (GND), CON1.3 (SHELL1), CON1.4 (SHELL2), CON1.5 (SHELL3), CON1.6 (SHELL4), P17.1, P24.1, P25.1, P28.1, P29.1
- net at C1.1, P1.1, P3.2 (PM)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: now also P15.1, P16.1, P4.1, P7.1, CON1.1 (VBUS), P18.1
- net at C4.2, C5.1, L1.1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: now also P20.1
- net at 500K1.1, D1.2 (K), R2.1: now also 500K2.1
- net at 500K1.2, R2.2, R3.1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: now also 500K2.2
- net at L1.3, P6.1, U1.7 (Vin): now also JP1.3, JP2.3, P19.1
- net at U1.3 (S/S): now also JP1.2, JP2.2; no longer P4.1
- net at P11.1, P8.1: now also P21.1, P22.1, P23.1, P26.1, P27.1
- no-connect marks 8 -> 21
Other:
- moved on the sheet: P2, P8, P9
