File: projects/EspDevBoard/EspDevBoard.sch (KiCad schematic (older format))
At the start: 53 parts, among them CON1 USB-MICRO, P1 CONN_3X2, P2 CONN_3X2, P3 CONN_10X2, P4 CONN_13X2, U1 ESP-12E, U2 NODE_MCU, U3 AP1117, U4 AD5274, U5 ATMEGA32U4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

Commit message: work on footprints and netlist
Parts:
- removed U3: AP1117, symbol AP1117
- added U3: AZ1117, frep:SOT223, symbol AZ1117
- C1, C10, C11, C12, C13, C2, C3, C4, C5, C6, C7, C8, C9, L1: footprint (none) -> frep:C0805
- F1: footprint (none) -> frep:C1812
- JP1, JP2: footprint (none) -> frep:Pin_Proto_Straight_1x03
- P1: value CONN_3X2 -> ICSP; footprint (none) -> frep:Pin_Proto_Straight_2x03
- P2: value CONN_3X2 -> ICSP_P; footprint (none) -> frep:Pin_Proto_Straight_2x03
- P3: value CONN_10X2 -> Display; footprint (none) -> frep:Pin_Proto_Straight_2x10
- P4: value CONN_13X2 -> Sepic_TH; footprint (none) -> frep:Sepic_TH
- R17, R18: footprint (none) -> frep:R1206
- U2: footprint (none) -> frep:NodeMcu
- U4: footprint (none) -> frep:MSOP10
- X1: footprint (none) -> frep:Resonator
Connections:
- net +3.3V: now also P3.1 (P1), U3.2 (VO), U3.4 (VO); no longer P3.2 (P2)
- net CS: now also P3.18 (P18); no longer P3.17 (P17)
- net GND: now also P3.16 (P16), P3.17 (P17), P3.2 (P2), P3.20 (P20), U3.1 (GND); no longer P3.1 (P1), P3.15 (P15), P3.18 (P18), P3.19 (P19)
- net MOSI: now also P3.14 (P14); no longer P3.13 (P13)
- net RES: now also P3.15 (P15); no longer P3.16 (P16)
- net RS: now also P3.3 (P3); no longer P3.4 (P4)
- net SCLK: now also P3.13 (P13); no longer P3.14 (P14)
- net at C1.1, JP1.2, JP2.2: now also U3.3 (VI)
Changed lines of the file:
@@
 LIBS:frep
 LIBS:ESP8266
+LIBS:EspDevBoard-cache
 EELAYER 25 0
 EELAYER END
@@
 P 3750 2950
 F 0 "P3" H 3750 3500 60  0000 C CNN
-F 1 "CONN_10X2" V 3750 2850 50  0000 C CNN
-F 2 "" H 3750 2950 60  0001 C CNN
+F 1 "Display" V 3750 2950 50  0000 C CNN
+F 2 "frep:Pin_Proto_Straight_2x10" H 3750 2950 60  0001 C CNN
 F 3 "" H 3750 2950 60  0000 C CNN
 	1    3750 2950
-	-1   0    0    -1
+	1    0    0    -1
 $EndComp
 Text Notes 3600 2300 0    60   ~ 0
@@
 F 0 "U2" H 1650 3600 60  0000 C CNN
 F 1 "NODE_MCU" V 1650 2800 50  0000 C CNN
-F 2 "" H 1650 2800 60  0001 C CNN
+F 2 "frep:NodeMcu" H 1650 2800 60  0001 C CNN
 F 3 "" H 1650 2800 60  0000 C CNN
 	1    1650 2800
@@
 P 1650 4200
 F 0 "P1" H 1650 4450 50  0000 C CNN
-F 1 "CONN_3X2" V 1650 4250 40  0000 C CNN
-F 2 "" H 1650 4200 60  0001 C CNN
+F 1 "ICSP" V 1650 4250 40  0000 C CNN
+F 2 "frep:Pin_Proto_Straight_2x03" H 1650 4200 60  0001 C CNN
 F 3 "" H 1650 4200 60  0000 C CNN
 	1    1650 4200
@@
 P 3750 5000
 F 0 "P4" H 3750 5700 60  0000 C CNN
-F 1 "CONN_13X2" V 3750 5000 50  0000 C CNN
-F 2 "" H 3750 5000 60  0001 C CNN
+F 1 "Sepic_TH" V 3750 5000 50  0000 C CNN
+F 2 "frep:Sepic_TH" H 3750 5000 60  0001 C CNN
 F 3 "" H 3750 5000 60  0000 C CNN
 	1    3750 5000
@@
 F 0 "U4" H 6300 5375 60  0000 C CNN
 F 1 "AD5274" H 6300 4625 60  0000 C CNN
-F 2 "" H 6300 4875 60  0001 C CNN
+F 2 "frep:MSOP10" H 6300 4875 60  0001 C CNN
 F 3 "" H 6300 4875 60  0000 C CNN
 	1    6300 5000
@@
 F 0 "JP1" H 1200 7000 40  0000 L CNN
 F 1 "JUMPER3" H 1150 7200 40  0000 C CNN
-F 2 "" H 1150 7100 60  0001 C CNN
+F 2 "frep:Pin_Proto_Straight_1x03" H 1150 7100 60  0001 C CNN
 F 3 "" H 1150 7100 60  0000 C CNN
 	1    1150 7100
@@
 F 0 "C8" H 5600 5500 40  0000 L CNN
 F 1 "1uF" H 5606 5315 40  0000 L CNN
-F 2 "" H 5638 5250 30  0001 C CNN
+F 2 "frep:C0805" H 5638 5250 30  0001 C CNN
 F 3 "" H 5600 5400 60  0000 C CNN
 	1    5600 5400
@@
 F 0 "C5" H 4850 5100 40  0000 L CNN
 F 1 "10uF" H 4856 4915 40  0000 L CNN
-F 2 "" H 4888 4850 30  0001 C CNN
+F 2 "frep:C0805" H 4888 4850 30  0001 C CNN
 F 3 "" H 4850 5000 60  0000 C CNN
 	1    4850 5000
@@
 F 0 "C7" H 5150 5100 40  0000 L CNN
 F 1 "100nF" H 5156 4915 40  0000 L CNN
-F 2 "" H 5188 4850 30  0001 C CNN
+F 2 "frep:C0805" H 5188 4850 30  0001 C CNN
 F 3 "" H 5150 5000 60  0000 C CNN
 	1    5150 5000
@@
 P 1650 4750
 F 0 "P2" H 1650 5000 50  0000 C CNN
-F 1 "CONN_3X2" V 1650 4800 40  0000 C CNN
-F 2 "" H 1650 4750 60  0001 C CNN
+F 1 "ICSP_P" V 1650 4800 40  0000 C CNN
+F 2 "frep:Pin_Proto_Straight_2x03" H 1650 4750 60  0001 C CNN
 F 3 "" H 1650 4750 60  0000 C CNN
 	1    1650 4750
@@
 F 0 "F1" H 2200 5450 40  0000 C CNN
 F 1 "FUSE" H 2000 5350 40  0000 C CNN
-F 2 "" H 2100 5400 60  0001 C CNN
+F 2 "frep:C1812" H 2100 5400 60  0001 C CNN
 F 3 "" H 2100 5400 60  0000 C CNN
 	1    2100 5400
@@
 F 0 "C3" H 4250 7400 40  0000 L CNN
 F 1 "100nF" H 4256 7215 40  0000 L CNN
-F 2 "" H 4288 7150 30  0001 C CNN
+F 2 "frep:C0805" H 4288 7150 30  0001 C CNN
 F 3 "" H 4250 7300 60  0000 C CNN
 	1    4250 7300
@@
 F 0 "C4" H 4700 7400 50  0000 L CNN
 F 1 "4u7F" H 4700 7200 50  0000 L CNN
-F 2 "" H 4650 7300 60  0001 C CNN
+F 2 "frep:C0805" H 4650 7300 60  0001 C CNN
 F 3 "" H 4650 7300 60  0000 C CNN
 	1    4650 7300
@@
 F 0 "C9" H 5750 2150 40  0000 L CNN
 F 1 "100nF" H 5756 1965 40  0000 L CNN
-F 2 "" H 5788 1900 30  0001 C CNN
+F 2 "frep:C0805" H 5788 1900 30  0001 C CNN
 F 3 "" H 5750 2050 60  0000 C CNN
 	1    5750 2050
@@
 F 0 "C10" H 9750 1650 40  0000 L CNN
 F 1 "100nF" H 9756 1465 40  0000 L CNN
-F 2 "" H 9788 1400 30  0001 C CNN
+F 2 "frep:C0805" H 9788 1400 30  0001 C CNN
 F 3 "" H 9750 1550 60  0000 C CNN
 	1    9750 1550
@@
 F 0 "L1" V 10350 1150 40  0000 C CNN
 F 1 "INDUCTOR" V 10500 1150 40  0000 C CNN
-F 2 "" H 10400 1150 60  0001 C CNN
+F 2 "frep:C0805" H 10400 1150 60  0001 C CNN
 F 3 "" H 10400 1150 60  0000 C CNN
 	1    10400 1150
@@
 F 0 "C11" H 10100 1450 40  0000 L CNN
 F 1 "1uF" H 10106 1265 40  0000 L CNN
-F 2 "" H 10138 1200 30  0001 C CNN
+F 2 "frep:C0805" H 10138 1200 30  0001 C CNN
 F 3 "" H 10100 1350 60  0000 C CNN
 	1    10100 1350
@@
 F 0 "R17" V 10480 4400 40  0000 C CNN
 F 1 "0.1R 1%" V 10407 4401 40  0000 C CNN
-F 2 "" V 10330 4400 30  0001 C CNN
+F 2 "frep:R1206" V 10330 4400 30  0001 C CNN
 F 3 "" H 10400 4400 30  0000 C CNN
 	1    10400 4400
@@
 F 0 "C12" H 10100 4500 40  0000 L CNN
 F 1 "100nF" H 10106 4315 40  0000 L CNN
-F 2 "" H 10138 4250 30  0001 C CNN
+F 2 "frep:C0805" H 10138 4250 30  0001 C CNN
 F 3 "" H 10100 4400 60  0000 C CNN
 	1    10100 4400
@@
 F 0 "R18" V 10480 5600 40  0000 C CNN
 F 1 "0.1R 1%" V 10407 5601 40  0000 C CNN
-F 2 "" V 10330 5600 30  0001 C CNN
+F 2 "frep:R1206" V 10330 5600 30  0001 C CNN
 F 3 "" H 10400 5600 30  0000 C CNN
 	1    10400 5600
@@
 F 0 "C13" H 10100 5700 40  0000 L CNN
 F 1 "100nF" H 10106 5515 40  0000 L CNN
-F 2 "" H 10138 5450 30  0001 C CNN
+F 2 "frep:C0805" H 10138 5450 30  0001 C CNN
 F 3 "" H 10100 5600 60  0000 C CNN
 	1    10100 5600
@@
 	9400 4250 9200 4250
 $Comp
-L AP1117 U3
-U 1 1 569EA288
-P 2500 7150
-F 0 "U3" H 2650 6954 60  0000 C CNN
-F 1 "AP1117" H 2500 7350 60  0000 C CNN
-F 2 "" H 2500 7150 60  0001 C CNN
-F 3 "" H 2500 7150 60  0000 C CNN
-	1    2500 7150
-	1    0    0    -1
-$EndComp
-$Comp
 L GND #PWR049
 U 1 1 569EA6B8
@@
 F 0 "X1" H 5375 2925 60  0000 C CNN
 F 1 "Resonator" H 5350 2850 60  0000 C CNN
-F 2 "" H 5350 2450 60  0001 C CNN
+F 2 "frep:Resonator" H 5350 2450 60  0001 C CNN
 F 3 "" H 5350 2450 60  0000 C CNN
 	1    5350 2700
@@
 F 0 "C6" H 5150 1150 40  0000 L CNN
 F 1 "100nF" H 5156 965 40  0000 L CNN
-F 2 "" H 5188 900 30  0001 C CNN
+F 2 "frep:C0805" H 5188 900 30  0001 C CNN
 F 3 "" H 5150 1050 60  0000 C CNN
 	1    5150 1050
@@
 F 0 "C1" H 1900 7400 40  0000 L CNN
 F 1 "4u7F" H 1906 7215 40  0000 L CNN
-F 2 "" H 1938 7150 30  0001 C CNN
+F 2 "frep:C0805" H 1938 7150 30  0001 C CNN
 F 3 "" H 1900 7300 60  0000 C CNN
 	1    1900 7300
@@
 F 0 "C2" H 3100 7400 40  0000 L CNN
 F 1 "4u7F" H 3106 7215 40  0000 L CNN
-F 2 "" H 3138 7150 30  0001 C CNN
+F 2 "frep:C0805" H 3138 7150 30  0001 C CNN
 F 3 "" H 3100 7300 60  0000 C CNN
 	1    3100 7300
@@
 F 0 "JP2" H 1500 7000 40  0000 L CNN
 F 1 "JUMPER3" H 1450 7200 40  0000 C CNN
-F 2 "" H 1450 7100 60  0001 C CNN
+F 2 "frep:Pin_Proto_Straight_1x03" H 1450 7100 60  0001 C CNN
 F 3 "" H 1450 7100 60  0000 C CNN
 	1    1450 7100
@@
 NoConn ~ 3500 2000
 NoConn ~ 3600 2000
+$Comp
+L AZ1117 U3
+U 1 1 56ACEE26
+P 2500 7150
+F 0 "U3" H 2650 6954 60  0000 C CNN
+F 1 "AZ1117" H 2500 7350 60  0000 C CNN
+F 2 "frep:SOT223" H 2500 7150 60  0001 C CNN
+F 3 "" H 2500 7150 60  0000 C CNN
+	1    2500 7150
+	1    0    0    -1
+$EndComp
+Wire Wire Line
+	2900 7200 2900 7100
 $EndSCHEMATC
