File: projects/EspDevBoard/EspDevBoard.sch (KiCad schematic (older format))
At the start: 53 parts, among them CON1 USB-MICRO, P1 ICSP, P2 ICSP_P, P3 Display, P4 Sepic_TH, U1 ESP-12E, U2 NODE_MCU, U3 AZ1117, U4 AD5274, U5 ATMEGA32U4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

Commit message: start with pcb
Connections:
- net R2+: now also U4.2 (A); no longer U4.3 (W)
- net R2-: now also U4.3 (W); no longer U4.2 (A)
Changed lines of the file:
@@
 	0    -1   -1   0
 $EndComp
+Text GLabel 5600 4900 0    40   Input ~ 0
+R2+
 Text GLabel 5600 5000 0    40   Input ~ 0
-R2+
-Text GLabel 5600 4900 0    40   Input ~ 0
 R2-
 $Comp

Commit message: work in progress
Parts:
- added P5, P6, P7, P8: CONN_1, frep:MountingHole_3mm, symbol CONN_1
Connections:
- no-connect marks 39 -> 43
Changed lines of the file:
@@
 Wire Wire Line
 	2900 7200 2900 7100
+$Comp
+L CONN_1 P5
+U 1 1 56D2DBEF
+P 5550 7200
+F 0 "P5" H 5630 7200 40  0000 L CNN
+F 1 "CONN_1" H 5550 7255 30  0001 C CNN
+F 2 "frep:MountingHole_3mm" H 5550 7200 60  0001 C CNN
+F 3 "" H 5550 7200 60  0000 C CNN
+	1    5550 7200
+	1    0    0    -1
+$EndComp
+$Comp
+L CONN_1 P6
+U 1 1 56D2DE23
+P 5550 7300
+F 0 "P6" H 5630 7300 40  0000 L CNN
+F 1 "CONN_1" H 5550 7355 30  0001 C CNN
+F 2 "frep:MountingHole_3mm" H 5550 7300 60  0001 C CNN
+F 3 "" H 5550 7300 60  0000 C CNN
+	1    5550 7300
+	1    0    0    -1
+$EndComp
+$Comp
+L CONN_1 P7
+U 1 1 56D2DED8
+P 5550 7400
+F 0 "P7" H 5630 7400 40  0000 L CNN
+F 1 "CONN_1" H 5550 7455 30  0001 C CNN
+F 2 "frep:MountingHole_3mm" H 5550 7400 60  0001 C CNN
+F 3 "" H 5550 7400 60  0000 C CNN
+	1    5550 7400
+	1    0    0    -1
+$EndComp
+$Comp
+L CONN_1 P8
+U 1 1 56D2DF92
+P 5550 7500
+F 0 "P8" H 5630 7500 40  0000 L CNN
+F 1 "CONN_1" H 5550 7555 30  0001 C CNN
+F 2 "frep:MountingHole_3mm" H 5550 7500 60  0001 C CNN
+F 3 "" H 5550 7500 60  0000 C CNN
+	1    5550 7500
+	1    0    0    -1
+$EndComp
+NoConn ~ 5400 7200
+NoConn ~ 5400 7300
+NoConn ~ 5400 7400
+NoConn ~ 5400 7500
 $EndSCHEMATC
