File: projects/LabBenchPsu/RevB/frontpanel/frontpanel.kicad_pcb (KiCad board)
At the start: 2 copper layers, 0 parts

Commit message: start with pcb
Parts:
- added C1: 4u7F, frep:C0805, F.Cu at (125.0, 155.0)
- added C10: 10nF, frep:C0805, B.Cu at (180.0, 110.0)
- added C11: 10nF, frep:C0805, B.Cu at (170.0, 115.0)
- added C2: 4u7F, frep:C0805, F.Cu at (125.0, 160.0)
- added C3: 1uF, frep:C0805, F.Cu at (50.0, 130.0)
- added C4: 1uF, frep:C0805, F.Cu at (50.0, 135.0)
- added C5: 1uF, frep:C0805, F.Cu at (50.0, 140.0)
- added C6: 10uF, frep:C0805, F.Cu at (50.0, 145.0)
- added C7: 100nF, frep:C0805, F.Cu at (50.0, 150.0)
- added C8: 10nF, frep:C0805, B.Cu at (105.0, 105.0)
- added C9: 10nF, frep:C0805, B.Cu at (105.0, 110.0)
- added CON1: USB-A-stacked, frep:USB-A-Stacked, F.Cu at (200.0, 30.0)
- added CON2: USB-A-stacked, frep:USB-A-Stacked, F.Cu at (225.0, 30.0)
- added CON3: USB-A-stacked, frep:USB-A-Stacked, F.Cu at (250.0, 30.0)
- added D1: PowerGood, frep:LED-0805, F.Cu at (65.0, 60.0)
- added D2: MainsOn, frep:LED-0805, F.Cu at (65.0, 65.0)
- added D3: LoadOn, frep:LED-0805, F.Cu at (200.0, 95.0)
- added D4: Charge complete, frep:LED-0805, F.Cu at (40.0, 140.0)
- added D5: Charging, frep:LED-0805, F.Cu at (40.0, 145.0)
- added ENC1: RotaryEncoder, frep:RotaryEncoder, F.Cu at (130.0, 110.0)
- added ENC2: RotaryEncoder, frep:RotaryEncoder, F.Cu at (155.0, 110.0)
- added F1: FUSE, frep:C1812, B.Cu at (115.0, 125.0)
- added F2: FUSE, frep:C1812, B.Cu at (130.0, 125.0)
- added F3: FUSE, frep:C1812, B.Cu at (145.0, 125.0)
- added JP1: JUMPER3, frep:Pin_Proto_Straight_1x03, F.Cu at (50.0, 95.0)
- added JP2: JUMPER, frep:Pin_Proto_Straight_1x02, F.Cu at (50.0, 100.0)
- added K1: TERMINAL, frep:terminal_3p5mm_3pin, B.Cu at (50.0, 85.0)
- added P1: INPUT_TERMINAL, frep:terminal_3p5mm_8pin, B.Cu at (100.0, 35.0)
- added P10: BindingPost, frep:BindingPost, B.Cu at (175.0, 135.0)
- added P11: LoadSwitch, frep:LoadSwitch, F.Cu at (190.0, 90.0)
- added P12: CONN_2, frep:Pin_Proto_Straight_1x02, F.Cu at (50.0, 115.0)
- added P13: BindingPost, frep:BindingPost, B.Cu at (130.0, 135.0)
- added P14: BindingPost, frep:BindingPost, B.Cu at (145.0, 135.0)
- added P15: BindingPost, frep:BindingPost, B.Cu at (160.0, 135.0)
- added P16: CONN_2, frep:JST-PH-2-THM, F.Cu at (30.0, 140.0)
- added P17: NHD-1.69-160128UGC3, frep:NHD-1.69-160128UGC3, F.Cu at (145.0, 75.0)
- added P2: MH, frep:MountingHole_3mm, F.Cu at (75.0, 140.0)
- added P3: MH, frep:MountingHole_3mm, F.Cu at (215.0, 140.0)
- added P4: MH, frep:MountingHole_3mm, F.Cu at (75.0, 50.0)
- added P5: MH, frep:MountingHole_3mm, F.Cu at (215.0, 50.0)
- added P6: CONN_2, frep:Pin_Proto_Straight_1x02, F.Cu at (50.0, 110.0)
- added P7: CONN_2, frep:Pin_Proto_Straight_1x02, F.Cu at (50.0, 105.0)
- added P8: BindingPost, frep:BindingPost, B.Cu at (115.0, 135.0)
- added P9: OnOffSwitch, frep:RockerSwitch, F.Cu at (95.0, 60.0)
- added R1: 1K, frep:R0805, B.Cu at (75.0, 60.0)
- added R10: 10K, frep:R0805, B.Cu at (115.0, 60.0)
- added R11: 10K, frep:R0805, B.Cu at (115.0, 90.0)
- added R12: 10K, frep:R0805, B.Cu at (175.0, 60.0)
- added R13: 10K, frep:R0805, B.Cu at (175.0, 90.0)
- added R14: 10K, frep:R0805, B.Cu at (115.0, 110.0)
- added R15: 10K, frep:R0805, B.Cu at (115.0, 115.0)
- added R16: 10K, frep:R0805, B.Cu at (180.0, 105.0)
- added R17: 10K, frep:R0805, B.Cu at (175.0, 105.0)
- added R18: 1K, frep:R0805, F.Cu at (200.0, 90.0)
- added R19: 10K, frep:R0805, B.Cu at (110.0, 110.0)
- added R2: 1K, frep:R0805, B.Cu at (75.0, 65.0)
- added R20: 10K, frep:R0805, B.Cu at (110.0, 105.0)
- added R21: 10K, frep:R0805, B.Cu at (170.0, 110.0)
- added R22: 10K, frep:R0805, B.Cu at (175.0, 110.0)
- added R3: 10R 10W, frep:R_ceramic_48x9p5x9mm, B.Cu at (90.0, 110.0)
- added R4: 270, frep:R0805, F.Cu at (60.0, 130.0)
- added R5: 270, frep:R0805, F.Cu at (60.0, 135.0)
- added R6: 1K, frep:R0805, F.Cu at (60.0, 140.0)
- added R7: 10K, frep:R0805, F.Cu at (60.0, 145.0)
- added R8: 10K, frep:R0805, B.Cu at (115.0, 105.0)
- added R9: 10K, frep:R0805, B.Cu at (170.0, 105.0)
- added S1: TAC_SWITCH, frep:TACTILE-PTH, F.Cu at (115.0, 60.0)
- added S2: TAC_SWITCH, frep:TACTILE-PTH, F.Cu at (115.0, 90.0)
- added S3: TAC_SWITCH, frep:TACTILE-PTH, F.Cu at (175.0, 60.0)
- added S4: TAC_SWITCH, frep:TACTILE-PTH, F.Cu at (175.0, 90.0)
- added U1: TPS2513, frep:SOT23-6, B.Cu at (200.0, 30.0)
- added U2: TPS2513, frep:SOT23-6, B.Cu at (225.0, 30.0)
- added U3: TPS2513, frep:SOT23-6, B.Cu at (250.0, 30.0)
- added U4: AZ1117, frep:SOT223, F.Cu at (115.0, 155.0)
- added U5: esp8266Feather, frep:featherEsp, B.Cu at (235.0, 110.0)
- added U6: MCP73833, frep:MSOP10, F.Cu at (20.0, 135.0)
- added U7: AD5274, frep:MSOP10, F.Cu at (20.0, 145.0)
- added U8: MCP23017, frep:SOIC28W, F.Cu at (25.0, 75.1)
Other:
- board outline added: 150 x 100 mm

Commit message: work on pcb
Parts:
- C1, C2, C3, C4, C5, C6, C7, JP2, P6, P7, R18, R4, R5, R6, R7, U4, U6, U7, U8: moved to B.Cu
- moved P6 164.3 mm to (203.0, 50.0)
- moved U8 160.1 mm to (182.5, 104.0), turned to 180 degrees
- moved P7 155.1 mm to (195.0, 50.0)
- moved JP2 144.7 mm to (192.0, 72.0), turned to 90 degrees
- moved P12 141.2 mm to (180.5, 61.0)
- moved K1 136.5 mm to (183.0, 54.5)
- moved CON3 99.7 mm to (207.0, 120.0)
- moved U3 98.4 mm to (207.0, 118.5)
- moved CON2 67.4 mm to (207.0, 95.0)
- moved U2 66.0 mm to (207.0, 93.5)
- moved P1 61.6 mm to (91.5, 96.0), turned to 90 degrees
- moved U6 60.1 mm to (77.0, 116.0)
- moved JP1 60.0 mm to (108.5, 108.5)
- moved U7 60.0 mm to (72.5, 116.0)
- moved P16 59.2 mm to (89.0, 135.0)
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Other:
- board text added: "-12V"
- board text added: "-5V"
- board text added: "12V"
- board text added: "3.3V"
- board text added: "5V"
- board text added: "5VSB"
- board text added: "ADJ"
- board text added: "BLACK"
- board text added: "BLUE"
- board text added: "GND"
- board text added: "GREY"
- board text added: "ORANGE"
- board text added: "PG"
- board text added: "PURPLE"
- board text added: "RED"
- board text added: "WHITE"
- board text added: "YELLOW"

Commit message: pcb in progress
Parts:
- moved K1 79.3 mm to (211.5, 128.5), turned to 90 degrees
- moved D3 73.7 mm to (183.0, 143.0)
- moved P12 67.1 mm to (197.0, 126.0), turned to 270 degrees
- moved P11 66.7 mm to (198.0, 135.0)
- moved R18 64.0 mm to (174.5, 130.5), turned to 270 degrees
- moved R4 21.5 mm to (94.5, 134.5), turned to 270 degrees
- moved D4 20.7 mm to (94.5, 134.5), turned to 90 degrees
- moved JP2 18.3 mm to (186.5, 54.5), turned to 180 degrees
- moved U7 18.3 mm to (89.0, 124.0), turned to 90 degrees
- moved U6 17.7 mm to (89.0, 129.0), turned to 90 degrees
- moved R5 17.7 mm to (82.5, 134.5), turned to 270 degrees
- moved C3 17.5 mm to (83.0, 131.0), turned to 180 degrees
- moved C2 15.7 mm to (112.5, 117.0), turned to 270 degrees
- moved C5 10.8 mm to (89.0, 132.5), turned to 180 degrees
- moved P7 10.1 mm to (204.0, 54.5)
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Routing:
- net 3.3V: track 0.00 -> 28.7 mm
- net 5V: track 0.00 -> 28.0 mm
- net 12V: track 0.00 -> 26.0 mm
- net Net-(F3-Pad2): track 0.00 -> 11.9 mm
- net Net-(F2-Pad2): track 0.00 -> 11.9 mm
- net Net-(F1-Pad2): track 0.00 -> 11.9 mm
- net 3V3Reg: track 0.00 -> 8.25 mm
- net ADJ: track 0.00 -> 7.41 mm
- net Net-(ENC2-Pad3): track 0.00 -> 7.23 mm
- net Net-(ENC2-Pad1): track 0.00 -> 7.12 mm
- net Net-(ENC1-Pad3): track 0.00 -> 7.12 mm
- net Net-(ENC1-Pad1): track 0.00 -> 7.12 mm
- net Net-(CON2-Pad7): track 0.00 -> 3.59 mm
- net Net-(CON2-Pad6): track 0.00 -> 3.59 mm
- net Net-(CON2-Pad3): track 0.00 -> 3.25 mm
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- added copper zone on F.Cu, net GND
Other:
- net class 0805 added: clearance 0.2, trace_width 1, via_dia 0.6, via_drill 0.4
- net class 1812 added: clearance 0.2, trace_width 1.8, via_dia 0.6, via_drill 0.4
- net class Default: trace_width 0.25 -> 0.5
- net class default2 added: clearance 0.2, trace_width 0.25, via_dia 0.6, via_drill 0.4
- board text added: "Ext. V"
- board text added: "Rx"
- board text added: "SCL"
- board text added: "SDA"
- board text added: "Tx"
- board text added: "i2c"
- board text added: "serial"
