File: projects/LabBenchPsu/RevB/labpsu/Preregulation.sch (KiCad schematic (older format))
At the start: 17 parts

Commit message: working on schematic
Parts:
- gave numbers to parts that had none: 16
Changed lines of the file:
@@
 encoding utf-8
 Sheet 2 3
-Title "Lab Psu"
+Title "Lab Psu (0-20V 0-2A)"
 Date ""
 Rev "B"
 Comp ""
-Comment1 "- based on David Jones' uSupply project"
-Comment2 "- Preregulation with SEPIC converter "
-Comment3 "- Powered from standard pc psu (12V)"
-Comment4 "- 2 pcb concept. To be used together with frontpanel pcb"
+Comment1 ""
+Comment2 "- Powered from standard pc psu (12V)"
+Comment3 "- SEPIC converter"
+Comment4 "- Switching pre regulator"
 $EndDescr
 $Comp
-L CP1 C?
+L CP1 C10
 U 1 1 57DD4052
 P 2100 3150
-F 0 "C?" H 2150 3250 50  0000 L CNN
+F 0 "C10" H 2150 3250 50  0000 L CNN
 F 1 "100uF" H 2150 3050 50  0000 L CNN
 F 2 "" H 2100 3150 60  0000 C CNN
@@
 $EndComp
 $Comp
-L CP1 C?
+L CP1 C15
 U 1 1 57DD4059
 P 8900 3150
-F 0 "C?" H 8950 3250 50  0000 L CNN
+F 0 "C15" H 8950 3250 50  0000 L CNN
 F 1 "100uF" H 8950 3050 50  0000 L CNN
 F 2 "" H 8900 3150 60  0000 C CNN
@@
 $EndComp
 $Comp
-L LT1370 U?
+L LT1370 U7
 U 1 1 57DD4060
 P 3650 3400
-F 0 "U?" H 3775 3875 60  0000 C CNN
+F 0 "U7" H 3775 3875 60  0000 C CNN
 F 1 "LT1370" H 3150 3900 60  0000 C CNN
 F 2 "" H 3650 3400 60  0000 C CNN
@@
 NoConn ~ 2650 3150
 $Comp
-L JUMPER3 JP?
+L JUMPER3 JP2
 U 1 1 57DD4068
 P 2550 3650
-F 0 "JP?" H 2600 3550 40  0000 L CNN
+F 0 "JP2" H 2600 3550 40  0000 L CNN
 F 1 "JUMPER3" H 2550 3750 40  0000 C CNN
 F 2 "" H 2550 3650 60  0000 C CNN
@@
 	1900 2700 3850 2700
 $Comp
-L GND #PWR?
+L GND #PWR025
 U 1 1 57DD4073
 P 2100 3350
-F 0 "#PWR?" H 2100 3350 30  0001 C CNN
+F 0 "#PWR025" H 2100 3350 30  0001 C CNN
 F 1 "GND" H 2100 3280 30  0001 C CNN
 F 2 "" H 2100 3350 60  0000 C CNN
@@
 $EndComp
 $Comp
-L GND #PWR?
+L GND #PWR026
 U 1 1 57DD4079
 P 3400 4200
-F 0 "#PWR?" H 3400 4200 30  0001 C CNN
+F 0 "#PWR026" H 3400 4200 30  0001 C CNN
 F 1 "GND" H 3400 4130 30  0001 C CNN
 F 2 "" H 3400 4200 60  0000 C CNN
@@
 	2550 4050 2550 3900
 $Comp
-L R R?
+L R R15
 U 1 1 57DD4D23
 P 3900 4350
-F 0 "R?" V 3980 4350 40  0000 C CNN
+F 0 "R15" V 3980 4350 40  0000 C CNN
 F 1 "2K" V 3907 4351 40  0000 C CNN
 F 2 "" V 3830 4350 30  0000 C CNN
@@
 $EndComp
 $Comp
-L C C?
+L C C11
 U 1 1 57DD4D5A
 P 3900 4800
-F 0 "C?" H 3900 4900 40  0000 L CNN
+F 0 "C11" H 3900 4900 40  0000 L CNN
 F 1 "470nF" H 3906 4715 40  0000 L CNN
 F 2 "" H 3938 4650 30  0000 C CNN
@@
 $EndComp
 $Comp
-L C C?
+L C C12
 U 1 1 57DD4DBC
 P 4150 4800
-F 0 "C?" H 4150 4900 40  0000 L CNN
+F 0 "C12" H 4150 4900 40  0000 L CNN
 F 1 "4n7F" H 4156 4715 40  0000 L CNN
 F 2 "" H 4188 4650 30  0000 C CNN
@@
 $EndComp
 $Comp
-L GND #PWR?
+L GND #PWR027
 U 1 1 57DD4E4B
 P 3650 4200
-F 0 "#PWR?" H 3650 4200 30  0001 C CNN
+F 0 "#PWR027" H 3650 4200 30  0001 C CNN
 F 1 "GND" H 3650 4130 30  0001 C CNN
 F 2 "" H 3650 4200 60  0000 C CNN
@@
 	3650 4100 3650 4200
 $Comp
-L GND #PWR?
+L GND #PWR028
 U 1 1 57DD4EED
 P 3900 5000
-F 0 "#PWR?" H 3900 5000 30  0001 C CNN
+F 0 "#PWR028" H 3900 5000 30  0001 C CNN
 F 1 "GND" H 3900 4930 30  0001 C CNN
 F 2 "" H 3900 5000 60  0000 C CNN
@@
 $EndComp
 $Comp
-L GND #PWR?
+L GND #PWR029
 U 1 1 57DD4F0D
 P 4150 5000
-F 0 "#PWR?" H 4150 5000 30  0001 C CNN
+F 0 "#PWR029" H 4150 5000 30  0001 C CNN
 F 1 "GND" H 4150 4930 30  0001 C CNN
 F 2 "" H 4150 5000 60  0000 C CNN
@@
 Connection ~ 3900 4100
 $Comp
-L InductorsCoupled L?
+L InductorsCoupled L1
 U 1 1 57DD5172
 P 4250 2700
-F 0 "L?" H 4250 2600 60  0000 C CNN
+F 0 "L1" H 4250 2600 60  0000 C CNN
 F 1 "22uH" H 4250 2825 60  0000 C CNN
 F 2 "" H 4250 2700 60  0000 C CNN
@@
 $EndComp
 $Comp
-L InductorsCoupled L?
+L InductorsCoupled L1
 U 2 1 57DD51B0
 P 5050 3100
-F 0 "L?" H 5050 3000 60  0000 C CNN
+F 0 "L1" H 5050 3000 60  0000 C CNN
 F 1 "22uH" H 5050 3225 60  0000 C CNN
 F 2 "" H 5050 3100 60  0000 C CNN
@@
 	4650 2700 4650 3150
 $Comp
-L C C?
+L C C13
 U 1 1 57DD5296
 P 4850 2700
-F 0 "C?" H 4850 2800 40  0000 L CNN
+F 0 "C13" H 4850 2800 40  0000 L CNN
 F 1 "4u7F" H 4856 2615 40  0000 L CNN
 F 2 "" H 4888 2550 30  0000 C CNN
@@
 $EndComp
 $Comp
-L GND #PWR?
+L GND #PWR030
 U 1 1 57DD5424
 P 5050 3500
-F 0 "#PWR?" H 5050 3500 30  0001 C CNN
+F 0 "#PWR030" H 5050 3500 30  0001 C CNN
 F 1 "GND" H 5050 3430 30  0001 C CNN
 F 2 "" H 5050 3500 60  0000 C CNN
@@
 $EndComp
 $Comp
-L DIODESCH D?
+L DIODESCH D3
 U 1 1 57DD5445
 P 5400 2700
-F 0 "D?" H 5400 2800 40  0000 C CNN
+F 0 "D3" H 5400 2800 40  0000 C CNN
 F 1 "V8PAN50-M3" H 5400 2600 40  0000 C CNN
 F 2 "" H 5400 2700 60  0000 C CNN
@@
 	5200 2700 5050 2700
 $Comp
-L R R?
+L R R16
 U 1 1 57DD5648
 P 5750 2950
-F 0 "R?" V 5830 2950 40  0000 C CNN
+F 0 "R16" V 5830 2950 40  0000 C CNN
 F 1 "10K" V 5757 2951 40  0000 C CNN
 F 2 "" V 5680 2950 30  0000 C CNN
@@
 $EndComp
 $Comp
-L R R?
+L R R17
 U 1 1 57DD56C7
 P 5750 4000
-F 0 "R?" V 5830 4000 40  0000 C CNN
+F 0 "R17" V 5830 4000 40  0000 C CNN
 F 1 "10K" V 5757 4001 40  0000 C CNN
 F 2 "" V 5680 4000 30  0000 C CNN
@@
 $EndComp
 $Comp
-L R R?
+L R R18
 U 1 1 57DD5713
 P 5750 4650
-F 0 "R?" V 5830 4650 40  0000 C CNN
+F 0 "R18" V 5830 4650 40  0000 C CNN
 F 1 "10K" V 5757 4651 40  0000 C CNN
 F 2 "" V 5680 4650 30  0000 C CNN
@@
 	4650 3650 5900 3650
 $Comp
-L GND #PWR?
+L GND #PWR031
 U 1 1 57DD5B21
 P 5750 5000
-F 0 "#PWR?" H 5750 5000 30  0001 C CNN
+F 0 "#PWR031" H 5750 5000 30  0001 C CNN
 F 1 "GND" H 5750 4930 30  0001 C CNN
 F 2 "" H 5750 5000 60  0000 C CNN
@@
 	5750 4900 5750 5000
 $Comp
-L R R?
+L R R19
 U 1 1 57DD5CA4
 P 6150 3650
-F 0 "R?" V 6230 3650 40  0000 C CNN
+F 0 "R19" V 6230 3650 40  0000 C CNN
 F 1 "330R" V 6157 3651 40  0000 C CNN
 F 2 "" V 6080 3650 30  0000 C CNN
@@
 $EndComp
 $Comp
-L AD5274 U?
+L AD5274 U8
 U 1 1 57DD5DF2
 P 7250 3750
-F 0 "U?" H 7250 4125 60  0000 C CNN
+F 0 "U8" H 7250 4125 60  0000 C CNN
 F 1 "AD5274" H 7250 3375 60  0000 C CNN
 F 2 "" H 7250 3625 60  0000 C CNN
@@
 3V3Reg
 $Comp
-L C C?
+L C C14
 U 1 1 57DD6B53
 P 6550 4150
-F 0 "C?" H 6550 4250 40  0000 L CNN
+F 0 "C14" H 6550 4250 40  0000 L CNN
 F 1 "1uF" H 6556 4065 40  0000 L CNN
 F 2 "" H 6588 4000 30  0000 C CNN
@@
 $EndComp
 $Comp
-L GND #PWR?
+L GND #PWR032
 U 1 1 57DD6BEC
 P 6550 3850
-F 0 "#PWR?" H 6550 3850 30  0001 C CNN
+F 0 "#PWR032" H 6550 3850 30  0001 C CNN
 F 1 "GND" H 6550 3780 30  0001 C CNN
 F 2 "" H 6550 3850 60  0000 C CNN
@@
 $EndComp
 $Comp
-L GND #PWR?
+L GND #PWR033
 U 1 1 57DD6D24
 P 6550 4350
-F 0 "#PWR?" H 6550 4350 30  0001 C CNN
+F 0 "#PWR033" H 6550 4350 30  0001 C CNN
 F 1 "GND" H 6550 4280 30  0001 C CNN
 F 2 "" H 6550 4350 60  0000 C CNN
@@
 Connection ~ 5750 4900
 $Comp
-L GND #PWR?
+L GND #PWR034
 U 1 1 57DD6F45
 P 7950 3950
-F 0 "#PWR?" H 7950 3950 30  0001 C CNN
+F 0 "#PWR034" H 7950 3950 30  0001 C CNN
 F 1 "GND" H 7950 3880 30  0001 C CNN
 F 2 "" H 7950 3950 60  0000 C CNN
@@
 $EndComp
 $Comp
-L GND #PWR?
+L GND #PWR035
 U 1 1 57DD6F83
 P 7950 3550
-F 0 "#PWR?" H 7950 3550 30  0001 C CNN
+F 0 "#PWR035" H 7950 3550 30  0001 C CNN
 F 1 "GND" H 7950 3480 30  0001 C CNN
 F 2 "" H 7950 3550 60  0000 C CNN
@@
 Connection ~ 5750 2700
 $Comp
-L GND #PWR?
+L GND #PWR036
 U 1 1 57DD7647
 P 8900 3350
-F 0 "#PWR?" H 8900 3350 30  0001 C CNN
+F 0 "#PWR036" H 8900 3350 30  0001 C CNN
 F 1 "GND" H 8900 3280 30  0001 C CNN
 F 2 "" H 8900 3350 60  0000 C CNN

Commit message: redraw schematic
Parts:
- renumbered R15 to R17, R16 to R18, R17 to R19, R18 to R20, R19 to R21
Changed lines of the file:
@@
 $Descr A4 11693 8268
 encoding utf-8
-Sheet 2 3
+Sheet 3 3
 Title "Lab Psu (0-20V 0-2A)"
 Date ""
@@
 	1900 2700 3850 2700
 $Comp
-L GND #PWR025
+L GND #PWR033
 U 1 1 57DD4073
 P 2100 3350
-F 0 "#PWR025" H 2100 3350 30  0001 C CNN
+F 0 "#PWR033" H 2100 3350 30  0001 C CNN
 F 1 "GND" H 2100 3280 30  0001 C CNN
 F 2 "" H 2100 3350 60  0000 C CNN
@@
 $EndComp
 $Comp
-L GND #PWR026
+L GND #PWR034
 U 1 1 57DD4079
 P 3400 4200
-F 0 "#PWR026" H 3400 4200 30  0001 C CNN
+F 0 "#PWR034" H 3400 4200 30  0001 C CNN
 F 1 "GND" H 3400 4130 30  0001 C CNN
 F 2 "" H 3400 4200 60  0000 C CNN
@@
 	2550 4050 2550 3900
 $Comp
-L R R15
+L R R17
 U 1 1 57DD4D23
 P 3900 4350
-F 0 "R15" V 3980 4350 40  0000 C CNN
+F 0 "R17" V 3980 4350 40  0000 C CNN
 F 1 "2K" V 3907 4351 40  0000 C CNN
 F 2 "" V 3830 4350 30  0000 C CNN
@@
 $EndComp
 $Comp
-L GND #PWR027
+L GND #PWR035
 U 1 1 57DD4E4B
 P 3650 4200
-F 0 "#PWR027" H 3650 4200 30  0001 C CNN
+F 0 "#PWR035" H 3650 4200 30  0001 C CNN
 F 1 "GND" H 3650 4130 30  0001 C CNN
 F 2 "" H 3650 4200 60  0000 C CNN
@@
 	3650 4100 3650 4200
 $Comp
-L GND #PWR028
+L GND #PWR036
 U 1 1 57DD4EED
 P 3900 5000
-F 0 "#PWR028" H 3900 5000 30  0001 C CNN
+F 0 "#PWR036" H 3900 5000 30  0001 C CNN
 F 1 "GND" H 3900 4930 30  0001 C CNN
 F 2 "" H 3900 5000 60  0000 C CNN
@@
 $EndComp
 $Comp
-L GND #PWR029
+L GND #PWR037
 U 1 1 57DD4F0D
 P 4150 5000
-F 0 "#PWR029" H 4150 5000 30  0001 C CNN
+F 0 "#PWR037" H 4150 5000 30  0001 C CNN
 F 1 "GND" H 4150 4930 30  0001 C CNN
 F 2 "" H 4150 5000 60  0000 C CNN
@@
 $EndComp
 $Comp
-L GND #PWR030
+L GND #PWR038
 U 1 1 57DD5424
 P 5050 3500
-F 0 "#PWR030" H 5050 3500 30  0001 C CNN
+F 0 "#PWR038" H 5050 3500 30  0001 C CNN
 F 1 "GND" H 5050 3430 30  0001 C CNN
 F 2 "" H 5050 3500 60  0000 C CNN
@@
 	5200 2700 5050 2700
 $Comp
-L R R16
+L R R18
 U 1 1 57DD5648
 P 5750 2950
-F 0 "R16" V 5830 2950 40  0000 C CNN
+F 0 "R18" V 5830 2950 40  0000 C CNN
 F 1 "10K" V 5757 2951 40  0000 C CNN
 F 2 "" V 5680 2950 30  0000 C CNN
@@
 $EndComp
 $Comp
-L R R17
+L R R19
 U 1 1 57DD56C7
 P 5750 4000
-F 0 "R17" V 5830 4000 40  0000 C CNN
+F 0 "R19" V 5830 4000 40  0000 C CNN
 F 1 "10K" V 5757 4001 40  0000 C CNN
 F 2 "" V 5680 4000 30  0000 C CNN
@@
 $EndComp
 $Comp
-L R R18
+L R R20
 U 1 1 57DD5713
 P 5750 4650
-F 0 "R18" V 5830 4650 40  0000 C CNN
+F 0 "R20" V 5830 4650 40  0000 C CNN
 F 1 "10K" V 5757 4651 40  0000 C CNN
 F 2 "" V 5680 4650 30  0000 C CNN
@@
 	4650 3650 5900 3650
 $Comp
-L GND #PWR031
+L GND #PWR039
 U 1 1 57DD5B21
 P 5750 5000
-F 0 "#PWR031" H 5750 5000 30  0001 C CNN
+F 0 "#PWR039" H 5750 5000 30  0001 C CNN
 F 1 "GND" H 5750 4930 30  0001 C CNN
 F 2 "" H 5750 5000 60  0000 C CNN
@@
 	5750 4900 5750 5000
 $Comp
-L R R19
+L R R21
 U 1 1 57DD5CA4
 P 6150 3650
-F 0 "R19" V 6230 3650 40  0000 C CNN
+F 0 "R21" V 6230 3650 40  0000 C CNN
 F 1 "330R" V 6157 3651 40  0000 C CNN
 F 2 "" V 6080 3650 30  0000 C CNN
@@
 $EndComp
 $Comp
-L GND #PWR032
+L GND #PWR040
 U 1 1 57DD6BEC
 P 6550 3850
-F 0 "#PWR032" H 6550 3850 30  0001 C CNN
+F 0 "#PWR040" H 6550 3850 30  0001 C CNN
 F 1 "GND" H 6550 3780 30  0001 C CNN
 F 2 "" H 6550 3850 60  0000 C CNN
@@
 $EndComp
 $Comp
-L GND #PWR033
+L GND #PWR041
 U 1 1 57DD6D24
 P 6550 4350
-F 0 "#PWR033" H 6550 4350 30  0001 C CNN
+F 0 "#PWR041" H 6550 4350 30  0001 C CNN
 F 1 "GND" H 6550 4280 30  0001 C CNN
 F 2 "" H 6550 4350 60  0000 C CNN
@@
 Connection ~ 5750 4900
 $Comp
-L GND #PWR034
+L GND #PWR042
 U 1 1 57DD6F45
 P 7950 3950
-F 0 "#PWR034" H 7950 3950 30  0001 C CNN
+F 0 "#PWR042" H 7950 3950 30  0001 C CNN
 F 1 "GND" H 7950 3880 30  0001 C CNN
 F 2 "" H 7950 3950 60  0000 C CNN
@@
 $EndComp
 $Comp
-L GND #PWR035
+L GND #PWR043
 U 1 1 57DD6F83
 P 7950 3550
-F 0 "#PWR035" H 7950 3550 30  0001 C CNN
+F 0 "#PWR043" H 7950 3550 30  0001 C CNN
 F 1 "GND" H 7950 3480 30  0001 C CNN
 F 2 "" H 7950 3550 60  0000 C CNN
@@
 Connection ~ 5750 2700
 $Comp
-L GND #PWR036
+L GND #PWR044
 U 1 1 57DD7647
 P 8900 3350
-F 0 "#PWR036" H 8900 3350 30  0001 C CNN
+F 0 "#PWR044" H 8900 3350 30  0001 C CNN
 F 1 "GND" H 8900 3280 30  0001 C CNN
 F 2 "" H 8900 3350 60  0000 C CNN

Commit message: schematic more or less done
Parts:
- renumbered C10 to C13, C11 to C14, C12 to C15, C13 to C16, C14 to C17, C15 to C18, D3 to D1, R17 to R26, R18 to R27, R19 to R28, R20 to R29, R21 to R30, U7 to U6, U8 to U7
Changed lines of the file:
@@
 $EndDescr
 $Comp
-L CP1 C10
+L CP1 C13
 U 1 1 57DD4052
 P 2100 3150
-F 0 "C10" H 2150 3250 50  0000 L CNN
+F 0 "C13" H 2150 3250 50  0000 L CNN
 F 1 "100uF" H 2150 3050 50  0000 L CNN
-F 2 "" H 2100 3150 60  0000 C CNN
+F 2 "" H 2100 3150 60  0001 C CNN
 F 3 "" H 2100 3150 60  0000 C CNN
 	1    2100 3150
@@
 $EndComp
 $Comp
-L CP1 C15
+L CP1 C18
 U 1 1 57DD4059
 P 8900 3150
-F 0 "C15" H 8950 3250 50  0000 L CNN
+F 0 "C18" H 8950 3250 50  0000 L CNN
 F 1 "100uF" H 8950 3050 50  0000 L CNN
-F 2 "" H 8900 3150 60  0000 C CNN
+F 2 "" H 8900 3150 60  0001 C CNN
 F 3 "" H 8900 3150 60  0000 C CNN
 	1    8900 3150
@@
 $EndComp
 $Comp
-L LT1370 U7
+L LT1370 U6
 U 1 1 57DD4060
 P 3650 3400
-F 0 "U7" H 3775 3875 60  0000 C CNN
+F 0 "U6" H 3775 3875 60  0000 C CNN
 F 1 "LT1370" H 3150 3900 60  0000 C CNN
-F 2 "" H 3650 3400 60  0000 C CNN
+F 2 "" H 3650 3400 60  0001 C CNN
 F 3 "" H 3650 3400 60  0000 C CNN
 	1    3650 3400
@@
 F 0 "JP2" H 2600 3550 40  0000 L CNN
 F 1 "JUMPER3" H 2550 3750 40  0000 C CNN
-F 2 "" H 2550 3650 60  0000 C CNN
+F 2 "" H 2550 3650 60  0001 C CNN
 F 3 "" H 2550 3650 60  0000 C CNN
 	1    2550 3650
@@
 	1900 2700 3850 2700
 $Comp
-L GND #PWR033
+L GND #PWR034
 U 1 1 57DD4073
 P 2100 3350
-F 0 "#PWR033" H 2100 3350 30  0001 C CNN
+F 0 "#PWR034" H 2100 3350 30  0001 C CNN
 F 1 "GND" H 2100 3280 30  0001 C CNN
 F 2 "" H 2100 3350 60  0000 C CNN
@@
 $EndComp
 $Comp
-L GND #PWR034
+L GND #PWR035
 U 1 1 57DD4079
 P 3400 4200
-F 0 "#PWR034" H 3400 4200 30  0001 C CNN
+F 0 "#PWR035" H 3400 4200 30  0001 C CNN
 F 1 "GND" H 3400 4130 30  0001 C CNN
 F 2 "" H 3400 4200 60  0000 C CNN
@@
 	2550 4050 2550 3900
 $Comp
-L R R17
+L R R26
 U 1 1 57DD4D23
 P 3900 4350
-F 0 "R17" V 3980 4350 40  0000 C CNN
+F 0 "R26" V 3980 4350 40  0000 C CNN
 F 1 "2K" V 3907 4351 40  0000 C CNN
-F 2 "" V 3830 4350 30  0000 C CNN
+F 2 "" V 3830 4350 30  0001 C CNN
 F 3 "" H 3900 4350 30  0000 C CNN
 	1    3900 4350
@@
 $EndComp
 $Comp
-L C C11
+L C C14
 U 1 1 57DD4D5A
 P 3900 4800
-F 0 "C11" H 3900 4900 40  0000 L CNN
+F 0 "C14" H 3900 4900 40  0000 L CNN
 F 1 "470nF" H 3906 4715 40  0000 L CNN
-F 2 "" H 3938 4650 30  0000 C CNN
+F 2 "" H 3938 4650 30  0001 C CNN
 F 3 "" H 3900 4800 60  0000 C CNN
 	1    3900 4800
@@
 $EndComp
 $Comp
-L C C12
+L C C15
 U 1 1 57DD4DBC
 P 4150 4800
-F 0 "C12" H 4150 4900 40  0000 L CNN
+F 0 "C15" H 4150 4900 40  0000 L CNN
 F 1 "4n7F" H 4156 4715 40  0000 L CNN
-F 2 "" H 4188 4650 30  0000 C CNN
+F 2 "" H 4188 4650 30  0001 C CNN
 F 3 "" H 4150 4800 60  0000 C CNN
 	1    4150 4800
@@
 $EndComp
 $Comp
-L GND #PWR035
+L GND #PWR036
 U 1 1 57DD4E4B
 P 3650 4200
-F 0 "#PWR035" H 3650 4200 30  0001 C CNN
+F 0 "#PWR036" H 3650 4200 30  0001 C CNN
 F 1 "GND" H 3650 4130 30  0001 C CNN
 F 2 "" H 3650 4200 60  0000 C CNN
@@
 	3650 4100 3650 4200
 $Comp
-L GND #PWR036
+L GND #PWR037
 U 1 1 57DD4EED
 P 3900 5000
-F 0 "#PWR036" H 3900 5000 30  0001 C CNN
+F 0 "#PWR037" H 3900 5000 30  0001 C CNN
 F 1 "GND" H 3900 4930 30  0001 C CNN
 F 2 "" H 3900 5000 60  0000 C CNN
@@
 $EndComp
 $Comp
-L GND #PWR037
+L GND #PWR038
 U 1 1 57DD4F0D
 P 4150 5000
-F 0 "#PWR037" H 4150 5000 30  0001 C CNN
+F 0 "#PWR038" H 4150 5000 30  0001 C CNN
 F 1 "GND" H 4150 4930 30  0001 C CNN
 F 2 "" H 4150 5000 60  0000 C CNN
@@
 F 0 "L1" H 4250 2600 60  0000 C CNN
 F 1 "22uH" H 4250 2825 60  0000 C CNN
-F 2 "" H 4250 2700 60  0000 C CNN
+F 2 "" H 4250 2700 60  0001 C CNN
 F 3 "" H 4250 2700 60  0000 C CNN
 	1    4250 2700
@@
 F 0 "L1" H 5050 3000 60  0000 C CNN
 F 1 "22uH" H 5050 3225 60  0000 C CNN
-F 2 "" H 5050 3100 60  0000 C CNN
+F 2 "" H 5050 3100 60  0001 C CNN
 F 3 "" H 5050 3100 60  0000 C CNN
 	2    5050 3100
@@
 	4650 2700 4650 3150
 $Comp
-L C C13
+L C C16
 U 1 1 57DD5296
 P 4850 2700
-F 0 "C13" H 4850 2800 40  0000 L CNN
+F 0 "C16" H 4850 2800 40  0000 L CNN
 F 1 "4u7F" H 4856 2615 40  0000 L CNN
-F 2 "" H 4888 2550 30  0000 C CNN
+F 2 "" H 4888 2550 30  0001 C CNN
 F 3 "" H 4850 2700 60  0000 C CNN
 	1    4850 2700
@@
 $EndComp
 $Comp
-L GND #PWR038
+L GND #PWR039
 U 1 1 57DD5424
 P 5050 3500
-F 0 "#PWR038" H 5050 3500 30  0001 C CNN
+F 0 "#PWR039" H 5050 3500 30  0001 C CNN
 F 1 "GND" H 5050 3430 30  0001 C CNN
 F 2 "" H 5050 3500 60  0000 C CNN
@@
 $EndComp
 $Comp
-L DIODESCH D3
+L DIODESCH D1
 U 1 1 57DD5445
 P 5400 2700
-F 0 "D3" H 5400 2800 40  0000 C CNN
+F 0 "D1" H 5400 2800 40  0000 C CNN
 F 1 "V8PAN50-M3" H 5400 2600 40  0000 C CNN
-F 2 "" H 5400 2700 60  0000 C CNN
+F 2 "" H 5400 2700 60  0001 C CNN
 F 3 "" H 5400 2700 60  0000 C CNN
 	1    5400 2700
@@
 	5200 2700 5050 2700
 $Comp
-L R R18
+L R R27
 U 1 1 57DD5648
 P 5750 2950
-F 0 "R18" V 5830 2950 40  0000 C CNN
+F 0 "R27" V 5830 2950 40  0000 C CNN
 F 1 "10K" V 5757 2951 40  0000 C CNN
-F 2 "" V 5680 2950 30  0000 C CNN
+F 2 "" V 5680 2950 30  0001 C CNN
 F 3 "" H 5750 2950 30  0000 C CNN
 	1    5750 2950
@@
 $EndComp
 $Comp
-L R R19
+L R R28
 U 1 1 57DD56C7
 P 5750 4000
-F 0 "R19" V 5830 4000 40  0000 C CNN
+F 0 "R28" V 5830 4000 40  0000 C CNN
 F 1 "10K" V 5757 4001 40  0000 C CNN
-F 2 "" V 5680 4000 30  0000 C CNN
+F 2 "" V 5680 4000 30  0001 C CNN
 F 3 "" H 5750 4000 30  0000 C CNN
 	1    5750 4000
@@
 $EndComp
 $Comp
-L R R20
+L R R29
 U 1 1 57DD5713
 P 5750 4650
-F 0 "R20" V 5830 4650 40  0000 C CNN
+F 0 "R29" V 5830 4650 40  0000 C CNN
 F 1 "10K" V 5757 4651 40  0000 C CNN
-F 2 "" V 5680 4650 30  0000 C CNN
+F 2 "" V 5680 4650 30  0001 C CNN
 F 3 "" H 5750 4650 30  0000 C CNN
 	1    5750 4650
@@
 	4650 3650 5900 3650
 $Comp
-L GND #PWR039
+L GND #PWR040
 U 1 1 57DD5B21
 P 5750 5000
-F 0 "#PWR039" H 5750 5000 30  0001 C CNN
+F 0 "#PWR040" H 5750 5000 30  0001 C CNN
 F 1 "GND" H 5750 4930 30  0001 C CNN
 F 2 "" H 5750 5000 60  0000 C CNN
@@
 	5750 4900 5750 5000
 $Comp
-L R R21
+L R R30
 U 1 1 57DD5CA4
 P 6150 3650
-F 0 "R21" V 6230 3650 40  0000 C CNN
+F 0 "R30" V 6230 3650 40  0000 C CNN
 F 1 "330R" V 6157 3651 40  0000 C CNN
-F 2 "" V 6080 3650 30  0000 C CNN
+F 2 "" V 6080 3650 30  0001 C CNN
 F 3 "" H 6150 3650 30  0000 C CNN
 	1    6150 3650
@@
 $EndComp
 $Comp
-L AD5274 U8
+L AD5274 U7
 U 1 1 57DD5DF2
 P 7250 3750
-F 0 "U8" H 7250 4125 60  0000 C CNN
+F 0 "U7" H 7250 4125 60  0000 C CNN
 F 1 "AD5274" H 7250 3375 60  0000 C CNN
-F 2 "" H 7250 3625 60  0000 C CNN
+F 2 "" H 7250 3625 60  0001 C CNN
 F 3 "" H 7250 3625 60  0000 C CNN
 	1    7250 3750
@@
 3V3Reg
 $Comp
-L C C14
+L C C17
 U 1 1 57DD6B53
 P 6550 4150
-F 0 "C14" H 6550 4250 40  0000 L CNN
+F 0 "C17" H 6550 4250 40  0000 L CNN
 F 1 "1uF" H 6556 4065 40  0000 L CNN
-F 2 "" H 6588 4000 30  0000 C CNN
+F 2 "" H 6588 4000 30  0001 C CNN
 F 3 "" H 6550 4150 60  0000 C CNN
 	1    6550 4150
@@
 $EndComp
 $Comp
-L GND #PWR040
+L GND #PWR041
 U 1 1 57DD6BEC
 P 6550 3850
-F 0 "#PWR040" H 6550 3850 30  0001 C CNN
+F 0 "#PWR041" H 6550 3850 30  0001 C CNN
 F 1 "GND" H 6550 3780 30  0001 C CNN
 F 2 "" H 6550 3850 60  0000 C CNN
@@
 $EndComp
 $Comp
-L GND #PWR041
+L GND #PWR042
 U 1 1 57DD6D24
 P 6550 4350
-F 0 "#PWR041" H 6550 4350 30  0001 C CNN
+F 0 "#PWR042" H 6550 4350 30  0001 C CNN
 F 1 "GND" H 6550 4280 30  0001 C CNN
 F 2 "" H 6550 4350 60  0000 C CNN
@@
 Connection ~ 5750 4900
 $Comp
-L GND #PWR042
+L GND #PWR043
 U 1 1 57DD6F45
 P 7950 3950
-F 0 "#PWR042" H 7950 3950 30  0001 C CNN
+F 0 "#PWR043" H 7950 3950 30  0001 C CNN
 F 1 "GND" H 7950 3880 30  0001 C CNN
 F 2 "" H 7950 3950 60  0000 C CNN
@@
 $EndComp
 $Comp
-L GND #PWR043
+L GND #PWR044
 U 1 1 57DD6F83
 P 7950 3550
-F 0 "#PWR043" H 7950 3550 30  0001 C CNN
+F 0 "#PWR044" H 7950 3550 30  0001 C CNN
 F 1 "GND" H 7950 3480 30  0001 C CNN
 F 2 "" H 7950 3550 60  0000 C CNN
@@
 Connection ~ 5750 2700
 $Comp
-L GND #PWR044
+L GND #PWR045
 U 1 1 57DD7647
 P 8900 3350
-F 0 "#PWR044" H 8900 3350 30  0001 C CNN
+F 0 "#PWR045" H 8900 3350 30  0001 C CNN
 F 1 "GND" H 8900 3280 30  0001 C CNN
 F 2 "" H 8900 3350 60  0000 C CNN

Commit message: schematic reviewed
Parts:
- R27: value 10K -> 18K
- R30: value 330R -> 0R
Changed lines of the file:
@@
 P 5750 2950
 F 0 "R27" V 5830 2950 40  0000 C CNN
-F 1 "10K" V 5757 2951 40  0000 C CNN
+F 1 "18K" V 5757 2951 40  0000 C CNN
 F 2 "" V 5680 2950 30  0001 C CNN
 F 3 "" H 5750 2950 30  0000 C CNN
@@
 P 6150 3650
 F 0 "R30" V 6230 3650 40  0000 C CNN
-F 1 "330R" V 6157 3651 40  0000 C CNN
+F 1 "0R" V 6157 3651 40  0000 C CNN
 F 2 "" V 6080 3650 30  0001 C CNN
 F 3 "" H 6150 3650 30  0000 C CNN

Commit message: schematic with new DAC
Parts:
- added P9: Heatsink, symbol CONN_2
Connections:
- no-connect marks 1 -> 3
Changed lines of the file:
@@
 Sheet 3 5
 Title "Lab Psu (0-20V 0-2A)"
-Date ""
+Date "2016-11-06"
 Rev "B"
 Comp ""
-Comment1 ""
-Comment2 "- Powered from standard pc psu (12V)"
-Comment3 "- SEPIC converter"
-Comment4 "- Switching pre regulator"
+Comment1 "- based on David Jones' uSupply project"
+Comment2 "- Preregulation with SEPIC converter "
+Comment3 "- Powered from standard pc psu (12V)"
+Comment4 "- 2 pcb concept. To be used together with frontpanel pcb"
 $EndDescr
 $Comp
@@
 $EndComp
 Connection ~ 8900 2700
+$Comp
+L CONN_2 P9
+U 1 1 581FF4E7
+P 3650 2025
+F 0 "P9" V 3600 2025 40  0000 C CNN
+F 1 "Heatsink" V 3700 2025 40  0000 C CNN
+F 2 "" H 3650 2025 60  0001 C CNN
+F 3 "" H 3650 2025 60  0000 C CNN
+	1    3650 2025
+	0    -1   -1   0
+$EndComp
+NoConn ~ 3750 2375
+NoConn ~ 3550 2375
 $EndSCHEMATC

Commit message: i2c addresses added
Other:
- note added: "i2c addr: 0101111 = 0x2F"
Changed lines of the file:
@@
 NoConn ~ 3750 2375
 NoConn ~ 3550 2375
+Text Notes 6875 4325 0    60   ~ 0
+i2c addr: 0101111 = 0x2F
 $EndSCHEMATC
