File: projects/LabBenchPsu/RevB/labpsu/Preregulation.sch (KiCad schematic (older format))
At the start: 17 parts, among them P9 Heatsink, U6 LT1370, U7 AD5274

Commit message: sepic calculations added
Parts:
- JP2: footprint (none) -> frep:Pin_Proto_Straight_1x03
Connections:
- net at R27.2, R28.1, U6.2 (FB+): now also R30.1; no longer R30.2
- net at U7.2 (A): now also R30.2; no longer R30.1
Other:
- note added: "AD5274 = 1K => V_out = 24.78"
- note added: "AD5274 = 20K => V_out = 3.49"
- note added: "R_tot = (R28+R29)*(R30+AD5274)/((R28+R29)+(R30+AD5274))"
- note added: "V_out = 1.245*(1+(R27/R_tot))"
- moved on the sheet: C17, C18, R27, R30, U7
Changed lines of the file:
@@
 L CP1 C18
 U 1 1 57DD4059
-P 8900 3150
-F 0 "C18" H 8950 3250 50  0000 L CNN
-F 1 "100uF" H 8950 3050 50  0000 L CNN
-F 2 "" H 8900 3150 60  0001 C CNN
-F 3 "" H 8900 3150 60  0000 C CNN
-	1    8900 3150
+P 8400 3150
+F 0 "C18" H 8450 3250 50  0000 L CNN
+F 1 "100uF" H 8450 3050 50  0000 L CNN
+F 2 "" H 8400 3150 60  0001 C CNN
+F 3 "" H 8400 3150 60  0000 C CNN
+	1    8400 3150
 	1    0    0    -1
 $EndComp
@@
 F 0 "JP2" H 2600 3550 40  0000 L CNN
 F 1 "JUMPER3" H 2550 3750 40  0000 C CNN
-F 2 "" H 2550 3650 60  0001 C CNN
+F 2 "frep:Pin_Proto_Straight_1x03" H 2550 3650 60  0001 C CNN
 F 3 "" H 2550 3650 60  0000 C CNN
 	1    2550 3650
@@
 Text HLabel 1900 2700 0    60   Input ~ 0
 V_IN
-Text HLabel 9200 2700 2    60   Output ~ 0
+Text HLabel 8700 2700 2    60   Output ~ 0
 V_OUT
-Text HLabel 8050 3650 2    60   Input ~ 0
+Text HLabel 8050 4250 2    60   Input ~ 0
 SCL
 Connection ~ 2100 2700
@@
 L GND #PWR037
 U 1 1 57DD4EED
-P 3900 5000
-F 0 "#PWR037" H 3900 5000 30  0001 C CNN
-F 1 "GND" H 3900 4930 30  0001 C CNN
-F 2 "" H 3900 5000 60  0000 C CNN
-F 3 "" H 3900 5000 60  0000 C CNN
-	1    3900 5000
+P 3900 5150
+F 0 "#PWR037" H 3900 5150 30  0001 C CNN
+F 1 "GND" H 3900 5080 30  0001 C CNN
+F 2 "" H 3900 5150 60  0000 C CNN
+F 3 "" H 3900 5150 60  0000 C CNN
+	1    3900 5150
 	1    0    0    -1
 $EndComp
@@
 L GND #PWR038
 U 1 1 57DD4F0D
-P 4150 5000
-F 0 "#PWR038" H 4150 5000 30  0001 C CNN
-F 1 "GND" H 4150 4930 30  0001 C CNN
-F 2 "" H 4150 5000 60  0000 C CNN
-F 3 "" H 4150 5000 60  0000 C CNN
-	1    4150 5000
+P 4150 5150
+F 0 "#PWR038" H 4150 5150 30  0001 C CNN
+F 1 "GND" H 4150 5080 30  0001 C CNN
+F 2 "" H 4150 5150 60  0000 C CNN
+F 3 "" H 4150 5150 60  0000 C CNN
+	1    4150 5150
 	1    0    0    -1
 $EndComp
@@
 L R R27
 U 1 1 57DD5648
-P 5750 2950
-F 0 "R27" V 5830 2950 40  0000 C CNN
-F 1 "18K" V 5757 2951 40  0000 C CNN
-F 2 "" V 5680 2950 30  0001 C CNN
-F 3 "" H 5750 2950 30  0000 C CNN
-	1    5750 2950
+P 5750 3150
+F 0 "R27" V 5830 3150 40  0000 C CNN
+F 1 "18K" V 5757 3151 40  0000 C CNN
+F 2 "" V 5680 3150 30  0001 C CNN
+F 3 "" H 5750 3150 30  0000 C CNN
+	1    5750 3150
 	1    0    0    -1
 $EndComp
@@
 $EndComp
 Wire Wire Line
-	5600 2700 9200 2700
-Wire Wire Line
-	5750 3200 5750 3750
-Wire Wire Line
-	4650 3650 5900 3650
+	4650 3650 6300 3650
 $Comp
 L GND #PWR040
 U 1 1 57DD5B21
-P 5750 5000
-F 0 "#PWR040" H 5750 5000 30  0001 C CNN
-F 1 "GND" H 5750 4930 30  0001 C CNN
-F 2 "" H 5750 5000 60  0000 C CNN
-F 3 "" H 5750 5000 60  0000 C CNN
-	1    5750 5000
+P 5750 5150
+F 0 "#PWR040" H 5750 5150 30  0001 C CNN
+F 1 "GND" H 5750 5080 30  0001 C CNN
+F 2 "" H 5750 5150 60  0000 C CNN
+F 3 "" H 5750 5150 60  0000 C CNN
+	1    5750 5150
 	1    0    0    -1
 $EndComp
@@
 	5750 4250 5750 4400
 Wire Wire Line
-	5750 4900 5750 5000
+	5750 4900 5750 5150
 $Comp
 L R R30
 U 1 1 57DD5CA4
-P 6150 3650
-F 0 "R30" V 6230 3650 40  0000 C CNN
-F 1 "0R" V 6157 3651 40  0000 C CNN
-F 2 "" V 6080 3650 30  0001 C CNN
-F 3 "" H 6150 3650 30  0000 C CNN
-	1    6150 3650
-	0    1    1    0
+P 6300 4000
+F 0 "R30" V 6380 4000 40  0000 C CNN
+F 1 "0R" V 6307 4001 40  0000 C CNN
+F 2 "" V 6230 4000 30  0001 C CNN
+F 3 "" H 6300 4000 30  0000 C CNN
+	1    6300 4000
+	1    0    0    -1
 $EndComp
 $Comp
 L AD5274 U7
 U 1 1 57DD5DF2
-P 7250 3750
-F 0 "U7" H 7250 4125 60  0000 C CNN
-F 1 "AD5274" H 7250 3375 60  0000 C CNN
-F 2 "" H 7250 3625 60  0001 C CNN
-F 3 "" H 7250 3625 60  0000 C CNN
-	1    7250 3750
-	1    0    0    -1
-$EndComp
-Text HLabel 6550 3200 1    60   Input ~ 0
+P 7250 4350
+F 0 "U7" H 7250 4725 60  0000 C CNN
+F 1 "AD5274" H 7250 3975 60  0000 C CNN
+F 2 "" H 7250 4225 60  0001 C CNN
+F 3 "" H 7250 4225 60  0000 C CNN
+	1    7250 4350
+	1    0    0    -1
+$EndComp
+Text HLabel 8700 3900 2    60   Input ~ 0
 3V3Reg
 $Comp
 L C C17
 U 1 1 57DD6B53
-P 6550 4150
-F 0 "C17" H 6550 4250 40  0000 L CNN
-F 1 "1uF" H 6556 4065 40  0000 L CNN
-F 2 "" H 6588 4000 30  0001 C CNN
-F 3 "" H 6550 4150 60  0000 C CNN
-	1    6550 4150
+P 6550 4750
+F 0 "C17" H 6550 4850 40  0000 L CNN
+F 1 "1uF" H 6556 4665 40  0000 L CNN
+F 2 "" H 6588 4600 30  0001 C CNN
+F 3 "" H 6550 4750 60  0000 C CNN
+	1    6550 4750
 	1    0    0    -1
 $EndComp
@@
 L GND #PWR041
 U 1 1 57DD6BEC
-P 6550 3850
-F 0 "#PWR041" H 6550 3850 30  0001 C CNN
-F 1 "GND" H 6550 3780 30  0001 C CNN
-F 2 "" H 6550 3850 60  0000 C CNN
-F 3 "" H 6550 3850 60  0000 C CNN
-	1    6550 3850
+P 6550 4450
+F 0 "#PWR041" H 6550 4450 30  0001 C CNN
+F 1 "GND" H 6550 4380 30  0001 C CNN
+F 2 "" H 6550 4450 60  0000 C CNN
+F 3 "" H 6550 4450 60  0000 C CNN
+	1    6550 4450
 	0    1    1    0
 $EndComp
@@
 L GND #PWR042
 U 1 1 57DD6D24
-P 6550 4350
-F 0 "#PWR042" H 6550 4350 30  0001 C CNN
-F 1 "GND" H 6550 4280 30  0001 C CNN
-F 2 "" H 6550 4350 60  0000 C CNN
-F 3 "" H 6550 4350 60  0000 C CNN
-	1    6550 4350
-	1    0    0    -1
-$EndComp
-Wire Wire Line
-	6550 3200 6550 3550
-Wire Wire Line
-	6400 3650 6550 3650
-Wire Wire Line
-	6550 3750 6300 3750
-Wire Wire Line
-	6300 3750 6300 4900
+P 6550 5150
+F 0 "#PWR042" H 6550 5150 30  0001 C CNN
+F 1 "GND" H 6550 5080 30  0001 C CNN
+F 2 "" H 6550 5150 60  0000 C CNN
+F 3 "" H 6550 5150 60  0000 C CNN
+	1    6550 5150
+	1    0    0    -1
+$EndComp
+Wire Wire Line
+	6300 4250 6550 4250
+Wire Wire Line
+	6550 4350 6300 4350
 Wire Wire Line
 	6300 4900 5750 4900
@@
 L GND #PWR043
 U 1 1 57DD6F45
-P 7950 3950
-F 0 "#PWR043" H 7950 3950 30  0001 C CNN
-F 1 "GND" H 7950 3880 30  0001 C CNN
-F 2 "" H 7950 3950 60  0000 C CNN
-F 3 "" H 7950 3950 60  0000 C CNN
-	1    7950 3950
+P 7950 4550
+F 0 "#PWR043" H 7950 4550 30  0001 C CNN
+F 1 "GND" H 7950 4480 30  0001 C CNN
+F 2 "" H 7950 4550 60  0000 C CNN
+F 3 "" H 7950 4550 60  0000 C CNN
+	1    7950 4550
 	0    -1   -1   0
 $EndComp
@@
 L GND #PWR044
 U 1 1 57DD6F83
-P 7950 3550
-F 0 "#PWR044" H 7950 3550 30  0001 C CNN
-F 1 "GND" H 7950 3480 30  0001 C CNN
-F 2 "" H 7950 3550 60  0000 C CNN
-F 3 "" H 7950 3550 60  0000 C CNN
-	1    7950 3550
+P 7950 4150
+F 0 "#PWR044" H 7950 4150 30  0001 C CNN
+F 1 "GND" H 7950 4080 30  0001 C CNN
+F 2 "" H 7950 4150 60  0000 C CNN
+F 3 "" H 7950 4150 60  0000 C CNN
+	1    7950 4150
 	0    -1   -1   0
 $EndComp
-Text HLabel 8050 3750 2    60   Input ~ 0
+Text HLabel 8050 4350 2    60   Input ~ 0
 SDA
 Wire Wire Line
-	7950 3850 8400 3850
-Wire Wire Line
-	8400 3850 8400 3300
-Wire Wire Line
-	8400 3300 6550 3300
-Connection ~ 6550 3300
-Wire Wire Line
-	8050 3650 7950 3650
-Wire Wire Line
-	8050 3750 7950 3750
+	7950 4450 8400 4450
+Wire Wire Line
+	8400 4450 8400 3900
+Wire Wire Line
+	6550 3900 8700 3900
+Wire Wire Line
+	8050 4250 7950 4250
+Wire Wire Line
+	8050 4350 7950 4350
 Wire Wire Line
 	2100 2950 2100 2700
 Wire Wire Line
-	8900 2700 8900 2950
+	8400 2700 8400 2950
 Connection ~ 5750 2700
 $Comp
 L GND #PWR045
 U 1 1 57DD7647
-P 8900 3350
-F 0 "#PWR045" H 8900 3350 30  0001 C CNN
-F 1 "GND" H 8900 3280 30  0001 C CNN
-F 2 "" H 8900 3350 60  0000 C CNN
-F 3 "" H 8900 3350 60  0000 C CNN
-	1    8900 3350
-	1    0    0    -1
-$EndComp
-Connection ~ 8900 2700
+P 8400 3350
+F 0 "#PWR045" H 8400 3350 30  0001 C CNN
+F 1 "GND" H 8400 3280 30  0001 C CNN
+F 2 "" H 8400 3350 60  0000 C CNN
+F 3 "" H 8400 3350 60  0000 C CNN
+	1    8400 3350
+	1    0    0    -1
+$EndComp
+Connection ~ 8400 2700
 $Comp
 L CONN_2 P9
@@
 NoConn ~ 3750 2375
 NoConn ~ 3550 2375
-Text Notes 6875 4325 0    60   ~ 0
+Text Notes 6875 4925 0    60   ~ 0
 i2c addr: 0101111 = 0x2F
+Wire Wire Line
+	6300 3650 6300 3750
+Wire Wire Line
+	6300 4350 6300 4900
+Connection ~ 8400 3900
+Wire Wire Line
+	6550 3900 6550 4150
+Wire Wire Line
+	5600 2700 8700 2700
+Wire Wire Line
+	3900 5000 3900 5150
+Wire Wire Line
+	4150 5000 4150 5150
+Wire Wire Line
+	6550 4950 6550 5150
+Wire Notes Line
+	5550 3750 5550 5050
+Wire Notes Line
+	5550 5050 8550 5050
+Wire Notes Line
+	8550 5050 8550 3750
+Wire Notes Line
+	8550 3750 5550 3750
+Wire Wire Line
+	5750 2900 5750 2700
+Wire Wire Line
+	5750 3400 5750 3750
+Text Notes 6875 5200 0    60   ~ 0
+R_tot = (R28+R29)*(R30+AD5274)/((R28+R29)+(R30+AD5274))
+Text Notes 6875 5400 0    60   ~ 0
+V_out = 1.245*(1+(R27/R_tot))
+Text Notes 6875 5625 0    60   ~ 0
+AD5274 = 20K   =>  V_out = 3.49
+Text Notes 6875 5700 0    60   ~ 0
+AD5274 = 1K    =>  V_out = 24.78
 $EndSCHEMATC
